File: kicad/cpu_mem/50pin_connector.sch (KiCad schematic (older format))
At the start: 1 part, among them P5 CONN_02X25

Commit message: update
Parts:
- P5: footprint (none) -> Pin_Headers:Pin_Header_Angled_2x25
Changed lines of the file:
@@
 F 0 "P5" H 5550 5050 50  0000 C CNN
 F 1 "CONN_02X25" V 5550 3750 50  0000 C CNN
-F 2 "" H 5550 3000 60  0000 C CNN
+F 2 "Pin_Headers:Pin_Header_Angled_2x25" H 5550 3000 60  0001 C CNN
 F 3 "" H 5550 3000 60  0000 C CNN
 	1    5550 3750
