File: kicad/cpu_mem/steckschwein.kicad_pcb (KiCad board)
At the start: 2 copper layers, 160 x 100.3 mm, 33 parts, among them P1 CONN_02X04, P3 CONN_01X03, P4 CONN_02X02, P5 CONN_02X25, SW1 SW_PUSH, U1 W65C02SP, U2 LM555N, U3 74HCT00, U4 74LS393, U5 GAL22V10, U6 28C256, U7 HM62256BLP-7, U8 HM62256BLP-7, U9 74LS139, X1 OSC

Commit message: new with new empty pcb
Parts:
- removed R8: 10k, Discret:R3
- added C12: 100n, Discret:C1, F.Cu at (137.7, 55.6)
- added C13: 100n, Discret:C1, F.Cu at (99.8, 55.4)
- added MH1: MountingHole_3mm_RevA_Date21Jun2010, Mounting_Holes:MountingHole_3mm, F.Cu at (68.6, 52.8)
- added MH2: MountingHole_3mm_RevA_Date21Jun2010, Mounting_Holes:MountingHole_3mm, F.Cu at (215.6, 52.6)
- added MH3: MountingHole_3mm_RevA_Date21Jun2010, Mounting_Holes:MountingHole_3mm, F.Cu at (215.6, 138.9)
- added MH4: MountingHole_3mm_RevA_Date21Jun2010, Mounting_Holes:MountingHole_3mm, F.Cu at (68.6, 138.9)
- added U10: 74LS244, Sockets_DIP:DIP-20__300_ELL, F.Cu at (89.7, 126.0)
- added U11: 74LS273, Sockets_DIP:DIP-20__300_ELL, F.Cu at (104.9, 126.0)
- U9: footprint Sockets_DIP:DIP-14__300_ELL -> Sockets_DIP:DIP-16__300_ELL
- moved X1 129.8 mm to (201.7, 129.5), turned to 90 degrees
- moved C8 106.5 mm to (107.4, 110.0)
- moved U4 104.0 mm to (188.0, 129.8)
- moved U6 101.1 mm to (93.5, 76.7)
- moved C9 94.1 mm to (92.2, 110.0)
- moved P1 91.0 mm to (178.8, 131.1), turned to 270 degrees
- moved C6 83.7 mm to (167.9, 117.6)
- moved P3 79.9 mm to (178.1, 122.2), turned to 180 degrees
- moved C3 79.0 mm to (158.2, 110.7)
- moved SW1 78.2 mm to (151.9, 135.1), turned to 180 degrees
- moved C2 77.5 mm to (158.2, 105.2), turned to 270 degrees
- moved R6 76.9 mm to (165.4, 100.3)
- moved R5 76.9 mm to (165.4, 103.1)
- moved U2 76.8 mm to (165.4, 110.2)
- moved C4 76.6 mm to (157.2, 99.3), turned to 180 degrees
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Connections:
- net /A10 renamed /decoder/A10
- net /A11 renamed /decoder/A11
- net /A12 renamed /decoder/A12
- net /A13 renamed /decoder/A13
- net /A14 renamed /decoder/A14
- net /A15 renamed /decoder/A15
- net /A6 renamed /decoder/A6
- net /A7 renamed /decoder/A7
- net /A8 renamed /decoder/A8
- net /A9 renamed /decoder/A9
- net /CS_HIRAM renamed /decoder//CS_HIRAM
- net /CS_LORAM renamed /decoder//CS_LORAM
- P1 pad 2: PH0-IN -> Net-(P1-Pad2)
- P1 pad 3: Net-(P1-Pad3) -> Net-(P1-Pad1)
- P1 pad 4: PH0-IN -> Net-(P1-Pad4)
- P1 pad 5: Net-(P1-Pad5) -> Net-(P1-Pad1)
- P1 pad 6: PH0-IN -> Net-(P1-Pad6)
- P1 pad 7: Net-(P1-Pad7) -> Net-(P1-Pad1)
- P1 pad 8: PH0-IN -> Net-(P1-Pad8)
- P3 pad 1: PH0-IN -> Net-(P1-Pad1)
- P4 pad 2: GND -> Net-(P4-Pad2)
- P4 pad 4: Net-(P4-Pad4) -> GND
- P5 pad 14: Net-(P5-Pad14) -> (no net)
- P5 pad 16: Net-(P5-Pad16) -> (no net)
- P5 pad 18: Net-(P5-Pad18) -> (no net)
- P5 pad 19: /CS_IO1 -> /CS_IO2
- P5 pad 20: /CS_IO0 -> /CS_IO1
- P5 pad 21: /CS_SND -> /CS_IO0
- P5 pad 36: Net-(P5-Pad36) -> (no net)
- P5 pad 37: Net-(P5-Pad37) -> (no net)
- P5 pad 38: Net-(P5-Pad38) -> (no net)
- P5 pad 39: Net-(P5-Pad39) -> (no net)
- P5 pad 40: Net-(P5-Pad40) -> (no net)
- P5 pad 41: Net-(P5-Pad41) -> (no net)
- P5 pad 42: Net-(P5-Pad42) -> (no net)
- P5 pad 5: /ROMOFF -> (no net)
- R4 pad 2: Net-(P4-Pad4) -> Net-(P4-Pad2)
- U1 pad 1: Net-(P4-Pad1) -> Net-(P4-Pad3)
- U1 pad 3: Net-(U1-Pad3) -> (no net)
- U1 pad 35: Net-(U1-Pad35) -> (no net)
- U1 pad 36: Net-(P4-Pad3) -> Net-(P4-Pad1)
- U1 pad 37: PH0-IN -> Net-(P1-Pad1)
- U1 pad 38: Net-(U1-Pad38) -> (no net)
- U1 pad 5: Net-(U1-Pad5) -> (no net)
- U1 pad 7: Net-(U1-Pad7) -> (no net)
- U4 pad 3: Net-(P1-Pad1) -> Net-(P1-Pad2)
- U4 pad 4: Net-(P1-Pad3) -> Net-(P1-Pad4)
- U4 pad 5: Net-(P1-Pad5) -> Net-(P1-Pad6)
- U4 pad 6: Net-(P1-Pad7) -> Net-(P1-Pad8)
- U5 pad 15: /ROMOFF -> Net-(U11-Pad2)
- U5 pad 16: /CS_ROM -> (no net)
- U5 pad 22: /CS_SND -> Net-(U10-Pad1)
- U5 pad 23: /CS_IO -> Net-(U5-Pad23)
- U6 pad 20: /CS_ROM -> (no net)
- U9 pad 1: /CS_IO -> (no net)
- U9 pad 10: (no net) -> /CS_IO2
- U9 pad 11: (no net) -> /CS_IO1
- U9 pad 12: (no net) -> /CS_IO0
- U9 pad 13: (no net) -> /Connector/A5
- U9 pad 14: (no net) -> /Connector/A4
- U9 pad 2: /Connector/A0 -> (no net)
- U9 pad 3: /Connector/A1 -> (no net)
- U9 pad 4: /CS_IO0 -> (no net)
- U9 pad 5: /CS_IO1 -> (no net)
- U9 pad 6: /CS_IO2 -> (no net)
- U9 pad 7: /CS_IO3 -> (no net)
- X1 pad 1: Net-(X1-Pad1) -> (no net)
Routing:
- net PHI2: track 156.6 -> 25.5 mm
- net VCC: track 227.1 -> 284.0 mm
- net PH0-IN: track 35.5 -> 0.00 mm
- net Net-(P4-Pad3): track 23.7 -> 0.00 mm
- net Net-(U2-Pad3): track 2.54 -> 24.5 mm
- net Net-(P1-Pad1): track 17.9 -> 39.8 mm
- net Net-(P4-Pad1): track 3.17 -> 22.9 mm
- net Net-(C2-Pad1): track 30.2 -> 45.4 mm
- net Net-(P1-Pad3): track 14.4 -> 0.00 mm
- net /RW: track 37.9 -> 51.2 mm, vias 1 -> 0
- net Net-(P3-Pad3): track 6.02 -> 18.1 mm
- net Net-(P1-Pad5): track 10.8 -> 0.00 mm
- net Net-(U3-Pad10): track 9.72 -> 0.00 mm
- net Net-(P4-Pad4): track 8.67 -> 0.00 mm
- net Net-(P1-Pad7): track 8.22 -> 0.00 mm
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
Commit message: update
Parts:
- added C14: 100n, Discret:C1, F.Cu at (81.8, 86.4)
- added C15: 100n, Discret:C1, F.Cu at (120.1, 124.7)
- added C16: CP2, Capacitors_Elko_ThroughHole:Elko_vert_11.2x7.5mm_RM2.5, F.Cu at (215.9, 130.3)
- added P2: CONN_01X08, Pin_Headers:Pin_Header_Straight_1x08, F.Cu at (67.6, 69.8)
- added U12: 74LS244, Sockets_DIP:DIP-20__300_ELL, F.Cu at (79.2, 69.8)
- U10: value 74LS244 -> 7400; footprint Sockets_DIP:DIP-20__300_ELL -> Sockets_DIP:DIP-14__300_ELL
- moved C5 887.0 mm to (1073.9, 37.8), turned to 90 degrees
- moved C9 109.5 mm to (196.6, 77.0)
- moved X1 109.2 mm to (92.5, 129.5)
- moved SW1 96.3 mm to (205.5, 55.1), turned to 270 degrees
- moved C8 89.3 mm to (196.6, 104.6)
- moved U3 87.3 mm to (105.7, 66.0)
- moved U4 77.5 mm to (110.5, 129.5)
- moved P4 76.3 mm to (120.7, 100.1)
- moved C6 76.1 mm to (127.5, 53.1)
- moved P1 75.9 mm to (102.9, 130.8)
- moved U2 74.9 mm to (92.5, 93.2)
- moved U5 73.9 mm to (194.1, 122.9)
- moved R4 73.5 mm to (128.3, 98.8)
- moved R6 70.4 mm to (95.2, 107.2), turned to 270 degrees
- moved R5 67.4 mm to (98.0, 107.2), turned to 90 degrees
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Connections:
- net Net-(U11-Pad2) renamed /decoder//ROMOFF
- U10 pad 10: GND -> Net-(U10-Pad10)
- U10 pad 11: /Connector/D4 -> Net-(U10-Pad11)
- U10 pad 12: Net-(U10-Pad12) -> Net-(U10-Pad10)
- U10 pad 13: /Connector/D5 -> Net-(U10-Pad13)
- U10 pad 14: Net-(U10-Pad14) -> VCC
- U10 pad 2: /Connector/D0 -> Net-(U10-Pad1)
- U10 pad 3: Net-(U10-Pad3) -> Net-(U10-Pad10)
- U10 pad 4: /Connector/D1 -> /RW
- U10 pad 5: Net-(U10-Pad5) -> /RW
- U10 pad 6: /Connector/D2 -> Net-(U10-Pad13)
- U10 pad 7: Net-(U10-Pad7) -> GND
- U10 pad 8: /Connector/D3 -> Net-(U10-Pad8)
- U10 pad 9: Net-(U10-Pad9) -> /RW
- U11 pad 11: Net-(U10-Pad1) -> Net-(U10-Pad8)
- U11 pad 12: (no net) -> Net-(P2-Pad5)
- U11 pad 13: Net-(U10-Pad9) -> /Connector/D4
- U11 pad 14: Net-(U10-Pad7) -> /Connector/D5
- U11 pad 15: (no net) -> Net-(P2-Pad6)
- U11 pad 16: (no net) -> Net-(P2-Pad7)
- U11 pad 17: Net-(U10-Pad5) -> /Connector/D6
- U11 pad 18: Net-(U10-Pad3) -> /Connector/D7
- U11 pad 19: (no net) -> Net-(P2-Pad8)
- U11 pad 3: Net-(U10-Pad18) -> /Connector/D0
- U11 pad 4: Net-(U10-Pad16) -> /Connector/D1
- U11 pad 5: (no net) -> /decoder/BANK1
- U11 pad 6: (no net) -> /decoder/BANK2
- U11 pad 7: Net-(U10-Pad14) -> /Connector/D2
- U11 pad 8: Net-(U10-Pad12) -> /Connector/D3
- U11 pad 9: (no net) -> Net-(P2-Pad4)
- U5 pad 16: (no net) -> /decoder//CS_ROM
- U6 pad 1: GND -> /decoder/BANK2
- U6 pad 20: (no net) -> /decoder//CS_ROM
- U6 pad 26: GND -> /decoder/BANK1
- U9 pad 1: (no net) -> Net-(U5-Pad23)
- U9 pad 10: /CS_IO2 -> (no net)
- U9 pad 11: /CS_IO1 -> (no net)
- U9 pad 12: /CS_IO0 -> (no net)
- U9 pad 13: /Connector/A5 -> (no net)
- U9 pad 14: /Connector/A4 -> (no net)
- U9 pad 15: Net-(U5-Pad23) -> (no net)
- U9 pad 2: (no net) -> /Connector/A4
- U9 pad 3: (no net) -> /Connector/A5
- U9 pad 4: (no net) -> /CS_IO0
- U9 pad 5: (no net) -> /CS_IO1
- U9 pad 6: (no net) -> /CS_IO2
Routing:
- net GND: track 340.4 -> 117.8 mm
- net /decoder/A7: track 0.00 -> 189.3 mm
- net /Connector/A4: track 0.00 -> 188.2 mm
- net /decoder/A6: track 0.00 -> 186.6 mm
- net /Connector/D5: track 0.00 -> 184.8 mm, vias 0 -> 1
- net /Connector/A5: track 0.00 -> 183.4 mm
- net /RW: track 51.2 -> 229.9 mm, vias 0 -> 2
- net /Connector/D4: track 0.00 -> 174.5 mm, vias 0 -> 1
- net /Connector/D3: track 0.00 -> 172.4 mm, vias 0 -> 2
- net /Connector/D0: track 0.00 -> 152.2 mm, vias 0 -> 1
- net /Connector/D1: track 0.00 -> 147.9 mm, vias 0 -> 1
- net VCC: track 284.0 -> 140.5 mm
- net /Connector/D2: track 0.00 -> 137.8 mm, vias 0 -> 1
- net /Connector/D7: track 0.00 -> 134.7 mm, vias 0 -> 1
- net /decoder/A8: track 0.00 -> 133.5 mm
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
Commit message: layout
Parts:
- removed C14, C15: 100n, Discret:C1
- removed U10: 7400, Sockets_DIP:DIP-14__300_ELL
- moved C5 874.1 mm to (201.9, 99.1), turned to 180 degrees
- moved SW1 134.8 mm to (72.4, 76.2)
- moved X1 125.3 mm to (195.6, 58.4), turned to 0 degrees
- moved C8 108.2 mm to (90.2, 85.1), turned to 270 degrees
- moved P1 97.1 mm to (175.3, 66.0), turned to 0 degrees
- moved U4 96.3 mm to (174.0, 57.1), turned to 0 degrees
- moved C10 81.8 mm to (161.9, 52.1), turned to 90 degrees
- moved C9 81.1 mm to (115.6, 72.8), turned to 270 degrees
- moved U5 68.9 mm to (134.9, 87.6), turned to 0 degrees
- moved P2 66.6 mm to (104.4, 125.3)
- moved C11 66.1 mm to (130.6, 109.3)
- moved C13 66.1 mm to (117.3, 109.3)
- moved U9 66.1 mm to (129.8, 75.4), turned to 0 degrees
- moved U12 65.9 mm to (114.8, 125.3)
- moved U11 65.9 mm to (128.0, 125.3)
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Connections:
- U11 pad 11: Net-(U10-Pad8) -> Net-(U11-Pad11)
- U12 pad 1: Net-(U10-Pad11) -> Net-(U12-Pad1)
- U12 pad 19: Net-(U10-Pad11) -> Net-(U12-Pad1)
- U4 pad 12: (no net) -> GND
- U4 pad 13: (no net) -> GND
- U5 pad 22: Net-(U10-Pad1) -> Net-(U5-Pad22)
- U9 pad 12: (no net) -> Net-(U11-Pad11)
- U9 pad 13: (no net) -> PHI2
- U9 pad 14: (no net) -> /RW
- U9 pad 15: (no net) -> Net-(U5-Pad22)
- U9 pad 9: (no net) -> Net-(U12-Pad1)
Routing:
- net GND: track 117.8 -> 421.1 mm
- net VCC: track 140.5 -> 386.7 mm, vias 0 -> 2
- net PHI2: track 54.6 -> 161.7 mm, vias 1 -> 4
- net /decoder/A7: track 189.3 -> 88.7 mm
- net /CS_IO1: track 0.00 -> 93.9 mm, vias 0 -> 1
- net /decoder/A6: track 186.6 -> 93.0 mm
- net /CS_IO0: track 0.00 -> 92.5 mm, vias 0 -> 1
- net /RESET: track 76.7 -> 168.1 mm, vias 1 -> 0
- net /NMI: track 2.21 -> 91.2 mm, vias 0 -> 2
- net /IRQ: track 6.38 -> 94.3 mm, vias 0 -> 1
- net /CS_IO2: track 0.00 -> 87.2 mm, vias 0 -> 1
- net Net-(U12-Pad1): track 0.00 -> 76.3 mm
- net /RW: track 229.9 -> 157.1 mm, vias 2 -> 1
- net /Connector/D1: track 147.9 -> 218.6 mm
- net Net-(U11-Pad11): track 0.00 -> 68.0 mm
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- added copper zone on F.Cu, net GND

Commit message: reset_trig, letzte ratsline fix
Connections:
- C2 pad 1: Net-(C2-Pad1) -> /Connector/RESET_TRIG
- P5 pad 36: (no net) -> /Connector/RESET_TRIG
- R5 pad 2: Net-(C2-Pad1) -> /Connector/RESET_TRIG
- SW1 pad 1: Net-(C2-Pad1) -> /Connector/RESET_TRIG
- U2 pad 2: Net-(C2-Pad1) -> /Connector/RESET_TRIG
Routing:
- net /Connector/RESET_TRIG: track 0.00 -> 238.8 mm
- net Net-(C2-Pad1): track 36.2 -> 0.00 mm
- net /Connector/A1: track 133.9 -> 132.9 mm
- net VCC: track 386.7 -> 387.4 mm
- net /Connector/A2: track 131.8 -> 131.3 mm

Commit message: beschriftung, masseflaeche
Other:
- board text added: "NON-WDC"
- board text added: "Steckschwein CPU/Memory Board 2015 Thomas Woinke / Marko Lauke http://www.steckschwein.de/"
- board text added: "WDC"

Commit message: qr code
Parts:
- added G***: LOGO, Steckschwein:QRCODE, F.Cu at (130.6, 58.5)

Commit message: verschoenert
Parts:
- U1: value W65C02SP -> 65C02
- U11: value 74LS273 -> 74HCT273
- U12: value 74LS244 -> 74HCT244
- U4: value 74LS393 -> 74HCT393
- U7, U8: value HM62256BLP-7 -> 62256
- U9: value 74LS139 -> 74HCT139
- moved G*** 66.2 mm to (74.2, 93.2)

Commit message: power anschluss
Parts:
- added P6: POWER, Pin_Headers:Pin_Header_Angled_1x04, F.Cu at (73.7, 127.0)
- U1: value 65C02 -> W65C02SP
- U11: value 74HCT273 -> 74LS273
- U12: value 74HCT244 -> 74LS244
- U4: value 74HCT393 -> 74LS393
- U7, U8: value 62256 -> HM62256BLP-7
- U9: value 74HCT139 -> 74LS139
- moved C16 138.0 mm to (80.0, 123.2), turned to 270 degrees
Routing:
- net GND: track 421.1 -> 437.9 mm
- net VCC: track 387.4 -> 402.0 mm
Other:
- board text added: "+5V"
