File: kicad/cpu_mem/decoder.sch (KiCad schematic (older format))
At the start: 7 parts, among them U10 74LS244, U11 74LS273, U5 GAL22V10, U9 74LS139

Commit message: rom banking pins
Parts:
- removed U10: 74LS244, Sockets_DIP:DIP-20__300_ELL, symbol 74LS244
- added P2: CONN_01X08, symbol CONN_01X08
Connections:
- net labels added: BANK1, BANK2
- wire segments 89 -> 84
- no-connect marks 8 -> 1
Changed lines of the file:
@@
 LIBS:74xgxx
 LIBS:ttl_ieee
-LIBS:steckschwein-cache
 EELAYER 24 0
 EELAYER END
@@
 $EndComp
 $Comp
-L GND #PWR028
+L GND #PWR34
 U 1 1 544D50D2
 P 4050 5250
-F 0 "#PWR028" H 4050 5250 30  0001 C CNN
+F 0 "#PWR34" H 4050 5250 30  0001 C CNN
 F 1 "GND" H 4050 5180 30  0001 C CNN
 F 2 "" H 4050 5250 60  0000 C CNN
@@
 $EndComp
 $Comp
-L VCC #PWR029
+L VCC #PWR33
 U 1 1 544D50D8
 P 4050 3550
-F 0 "#PWR029" H 4050 3650 30  0001 C CNN
+F 0 "#PWR33" H 4050 3650 30  0001 C CNN
 F 1 "VCC" H 4050 3650 30  0000 C CNN
 F 2 "" H 4050 3550 60  0000 C CNN
@@
 Text Label 3550 4850 0    60   ~ 0
 A4
-$Comp
-L 74LS244 U10
-U 1 1 544D53A2
-P 6850 3450
-F 0 "U10" H 6900 3250 60  0000 C CNN
-F 1 "74LS244" H 6950 3050 60  0000 C CNN
-F 2 "Sockets_DIP:DIP-20__300_ELL" H 6850 3450 60  0001 C CNN
-F 3 "" H 6850 3450 60  0000 C CNN
-	1    6850 3450
-	1    0    0    -1
-$EndComp
-Entry Wire Line
-	5900 2850 6000 2950
-Entry Wire Line
-	5900 2950 6000 3050
-Entry Wire Line
-	5900 3050 6000 3150
-Entry Wire Line
-	5900 3150 6000 3250
-Entry Wire Line
-	5900 3250 6000 3350
-Entry Wire Line
-	5900 3350 6000 3450
-Entry Wire Line
-	5900 3450 6000 3550
-Entry Wire Line
-	5900 3550 6000 3650
+Entry Wire Line
+	6450 2850 6550 2950
+Entry Wire Line
+	6450 2950 6550 3050
+Entry Wire Line
+	6450 3050 6550 3150
+Entry Wire Line
+	6450 3150 6550 3250
+Entry Wire Line
+	6450 3250 6550 3350
+Entry Wire Line
+	6450 3350 6550 3450
+Entry Wire Line
+	6450 3450 6550 3550
+Entry Wire Line
+	6450 3550 6550 3650
 Wire Wire Line
 	4050 5100 4050 5250
@@
 	5050 3950 5100 3950
 Wire Wire Line
-	5050 3850 6150 3850
-Wire Wire Line
-	6150 3850 6150 4050
+	5050 3850 6700 3850
 Wire Bus Line
-	5900 2800 5900 3550
-Wire Wire Line
-	6000 2950 6150 2950
-Wire Wire Line
-	6000 3050 6150 3050
-Wire Wire Line
-	6000 3150 6150 3150
-Wire Wire Line
-	6000 3250 6150 3250
-Wire Wire Line
-	6000 3350 6150 3350
-Wire Wire Line
-	6000 3450 6150 3450
-Wire Wire Line
-	6000 3550 6150 3550
-Wire Wire Line
-	6000 3650 6150 3650
-Text Label 5850 2800 0    60   ~ 0
+	6450 2800 6450 3550
+Wire Wire Line
+	6550 2950 6700 2950
+Wire Wire Line
+	6550 3050 6700 3050
+Wire Wire Line
+	6550 3150 6700 3150
+Wire Wire Line
+	6550 3250 6700 3250
+Wire Wire Line
+	6550 3350 6700 3350
+Wire Wire Line
+	6550 3450 6700 3450
+Wire Wire Line
+	6550 3550 6700 3550
+Wire Wire Line
+	6550 3650 6700 3650
+Text Label 6400 2800 0    60   ~ 0
 D
-Text Label 6000 2950 0    60   ~ 0
+Text Label 6550 2950 0    60   ~ 0
 D0
-Text Label 6000 3050 0    60   ~ 0
+Text Label 6550 3050 0    60   ~ 0
 D1
-Text Label 6000 3150 0    60   ~ 0
+Text Label 6550 3150 0    60   ~ 0
 D2
-Text Label 6000 3250 0    60   ~ 0
+Text Label 6550 3250 0    60   ~ 0
 D3
-Text Label 6000 3350 0    60   ~ 0
+Text Label 6550 3350 0    60   ~ 0
 D4
-Text Label 6000 3450 0    60   ~ 0
+Text Label 6550 3450 0    60   ~ 0
 D5
-Text Label 6000 3550 0    60   ~ 0
+Text Label 6550 3550 0    60   ~ 0
 D6
-Text Label 6000 3650 0    60   ~ 0
+Text Label 6550 3650 0    60   ~ 0
 D7
 $Comp
 L 74LS273 U11
 U 1 1 544D56DD
-P 8600 3450
-F 0 "U11" H 8600 3300 60  0000 C CNN
-F 1 "74LS273" H 8600 3100 60  0000 C CNN
-F 2 "Sockets_DIP:DIP-20__300_ELL" H 8600 3450 60  0001 C CNN
-F 3 "" H 8600 3450 60  0000 C CNN
-	1    8600 3450
-	1    0    0    -1
-$EndComp
-Wire Wire Line
-	7550 2950 7900 2950
-Wire Wire Line
-	7550 3050 7900 3050
-Wire Wire Line
-	7550 3150 7900 3150
-Wire Wire Line
-	7550 3250 7900 3250
-Wire Wire Line
-	7550 3350 7900 3350
-Wire Wire Line
-	7550 3450 7900 3450
-Wire Wire Line
-	7550 3550 7900 3550
-Wire Wire Line
-	7550 3650 7900 3650
-Wire Wire Line
-	7900 3950 7800 3950
-Wire Wire Line
-	7900 3850 7300 3850
-Wire Wire Line
-	7300 3850 7300 4050
-Wire Wire Line
-	7300 4050 6150 4050
-Connection ~ 6150 3950
+P 7400 3450
+F 0 "U11" H 7400 3300 60  0000 C CNN
+F 1 "74LS273" H 7400 3100 60  0000 C CNN
+F 2 "Sockets_DIP:DIP-20__300_ELL" H 7400 3450 60  0001 C CNN
+F 3 "" H 7400 3450 60  0000 C CNN
+	1    7400 3450
+	1    0    0    -1
+$EndComp
+Wire Wire Line
+	6700 3950 6600 3950
 Wire Wire Line
 	5800 4550 5800 2300
 Wire Wire Line
-	5800 2300 9400 2300
-Wire Wire Line
-	9400 2300 9400 2950
-Wire Wire Line
-	9400 2950 9300 2950
-NoConn ~ 9300 3050
-NoConn ~ 9300 3150
-NoConn ~ 9300 3250
-NoConn ~ 9300 3350
-NoConn ~ 9300 3450
-NoConn ~ 9300 3550
-NoConn ~ 9300 3650
+	5800 2300 8200 2300
+Wire Wire Line
+	8200 2300 8200 2950
+Wire Wire Line
+	8100 2950 8750 2950
 Text HLabel 850  2500 2    60   Input ~ 0
 A4
@@
 A15
 $Comp
-L VCC #PWR030
+L VCC #PWR30
 U 1 1 544D6887
 P 3450 3700
-F 0 "#PWR030" H 3450 3800 30  0001 C CNN
+F 0 "#PWR30" H 3450 3800 30  0001 C CNN
 F 1 "VCC" H 3450 3800 30  0000 C CNN
 F 2 "" H 3450 3700 60  0000 C CNN
@@
 	5050 3000 5200 3000
 $Comp
-L VCC #PWR031
+L VCC #PWR31
 U 1 1 544D68A5
 P 3750 2200
-F 0 "#PWR031" H 3750 2300 30  0001 C CNN
+F 0 "#PWR31" H 3750 2300 30  0001 C CNN
 F 1 "VCC" H 3750 2300 30  0000 C CNN
 F 2 "" H 3750 2200 60  0000 C CNN
@@
 $EndComp
 $Comp
-L GND #PWR032
+L GND #PWR32
 U 1 1 544D68AB
 P 3750 3200
-F 0 "#PWR032" H 3750 3200 30  0001 C CNN
+F 0 "#PWR32" H 3750 3200 30  0001 C CNN
 F 1 "GND" H 3750 3130 30  0001 C CNN
 F 2 "" H 3750 3200 60  0000 C CNN
@@
 Text HLabel 5200 3000 2    60   Output ~ 0
 /CS_IO3
-Text HLabel 7800 3950 0    60   Input ~ 0
+Text HLabel 6600 3950 0    60   Input ~ 0
 /RESET
 $Comp
-L VCC #PWR033
-U 1 1 544D6E00
-P 6550 2750
-F 0 "#PWR033" H 6550 2850 30  0001 C CNN
-F 1 "VCC" H 6550 2850 30  0000 C CNN
-F 2 "" H 6550 2750 60  0000 C CNN
-F 3 "" H 6550 2750 60  0000 C CNN
-	1    6550 2750
-	1    0    0    -1
-$EndComp
-Wire Wire Line
-	6550 2750 6550 2900
-$Comp
-L VCC #PWR034
+L VCC #PWR35
 U 1 1 544D6F18
-P 8300 2750
-F 0 "#PWR034" H 8300 2850 30  0001 C CNN
-F 1 "VCC" H 8300 2850 30  0000 C CNN
-F 2 "" H 8300 2750 60  0000 C CNN
-F 3 "" H 8300 2750 60  0000 C CNN
-	1    8300 2750
-	1    0    0    -1
-$EndComp
-Wire Wire Line
-	8300 2750 8300 2900
-$Comp
-L GND #PWR035
-U 1 1 544D6F9D
-P 6550 4200
-F 0 "#PWR035" H 6550 4200 30  0001 C CNN
-F 1 "GND" H 6550 4130 30  0001 C CNN
-F 2 "" H 6550 4200 60  0000 C CNN
-F 3 "" H 6550 4200 60  0000 C CNN
-	1    6550 4200
-	1    0    0    -1
-$EndComp
-Wire Wire Line
-	6550 4000 6550 4200
-$Comp
-L GND #PWR036
+P 7100 2750
+F 0 "#PWR35" H 7100 2850 30  0001 C CNN
+F 1 "VCC" H 7100 2850 30  0000 C CNN
+F 2 "" H 7100 2750 60  0000 C CNN
+F 3 "" H 7100 2750 60  0000 C CNN
+	1    7100 2750
+	1    0    0    -1
+$EndComp
+Wire Wire Line
+	7100 2750 7100 2900
+$Comp
+L GND #PWR36
 U 1 1 544D700F
-P 8300 4200
-F 0 "#PWR036" H 8300 4200 30  0001 C CNN
-F 1 "GND" H 8300 4130 30  0001 C CNN
-F 2 "" H 8300 4200 60  0000 C CNN
-F 3 "" H 8300 4200 60  0000 C CNN
-	1    8300 4200
-	1    0    0    -1
-$EndComp
-Wire Wire Line
-	8300 4000 8300 4200
-$Comp
-L VCC #PWR037
+P 7100 4200
+F 0 "#PWR36" H 7100 4200 30  0001 C CNN
+F 1 "GND" H 7100 4130 30  0001 C CNN
+F 2 "" H 7100 4200 60  0000 C CNN
+F 3 "" H 7100 4200 60  0000 C CNN
+	1    7100 4200
+	1    0    0    -1
+$EndComp
+Wire Wire Line
+	7100 4000 7100 4200
+$Comp
+L VCC #PWR28
 U 1 1 544E9402
 P 2600 5850
-F 0 "#PWR037" H 2600 5950 30  0001 C CNN
+F 0 "#PWR28" H 2600 5950 30  0001 C CNN
 F 1 "VCC" H 2600 5950 30  0000 C CNN
 F 2 "" H 2600 5850 60  0000 C CNN
@@
 $EndComp
 $Comp
-L GND #PWR038
+L GND #PWR29
 U 1 1 544E9408
 P 2600 6400
-F 0 "#PWR038" H 2600 6400 30  0001 C CNN
+F 0 "#PWR29" H 2600 6400 30  0001 C CNN
 F 1 "GND" H 2600 6330 30  0001 C CNN
 F 2 "" H 2600 6400 60  0000 C CNN
@@
 Connection ~ 3100 6300
 Connection ~ 2850 6300
+$Comp
+L CONN_01X08 P2
+U 1 1 544E9377
+P 8950 3300
+F 0 "P2" H 8950 3750 50  0000 C CNN
+F 1 "CONN_01X08" V 9050 3300 50  0000 C CNN
+F 2 "" H 8950 3300 60  0000 C CNN
+F 3 "" H 8950 3300 60  0000 C CNN
+	1    8950 3300
+	1    0    0    -1
+$EndComp
+Connection ~ 8200 2950
+Wire Wire Line
+	8100 3050 8750 3050
+Wire Wire Line
+	8100 3150 8750 3150
+Wire Wire Line
+	8100 3250 8750 3250
+Wire Wire Line
+	8750 3350 8100 3350
+Wire Wire Line
+	8100 3450 8750 3450
+Wire Wire Line
+	8100 3550 8750 3550
+Wire Wire Line
+	8100 3650 8750 3650
+Text HLabel 8350 2600 1    60   Output ~ 0
+BANK1
+Text HLabel 8500 2600 1    60   Output ~ 0
+BANK2
+Wire Wire Line
+	8350 2600 8350 3050
+Connection ~ 8350 3050
+Wire Wire Line
+	8500 2600 8500 3150
+Connection ~ 8500 3150
 $EndSCHEMATC

Commit message: memctl register auslesbar
Parts:
- added C14, C15: 100n, Discret:C1, symbol C
- added U10: 7400, Sockets_DIP:DIP-14__300_ELL, symbol 7400
- added U12: 74LS244, Sockets_DIP:DIP-20__300_ELL, symbol 74LS244
- P2: footprint (none) -> Pin_Headers:Pin_Header_Straight_1x08
Connections:
- net labels added: /ROMOFF
- wire segments 84 -> 109
Other:
- moved on the sheet: C11, C12, C13, U5, U9B

Commit message: update
Changed lines of the file:
@@
 LIBS:ttl_ieee
 LIBS:steckschwein-cache
-EELAYER 24 0
+EELAYER 25 0
 EELAYER END
 $Descr A4 11693 8268
@@
 $Comp
 L 74LS139 U9
-U 2 1 544D688D
+U 1 1 544D688D
 P 1700 4350
 F 0 "U9" H 1700 4450 60  0000 C CNN
@@
 F 2 "Sockets_DIP:DIP-16__300_ELL" H 1700 4350 60  0001 C CNN
 F 3 "" H 1700 4350 60  0000 C CNN
-	2    1700 4350
-	1    0    0    -1
-$EndComp
+	1    1700 4350
+	1    0    0    -1
+$EndComp

Commit message: 244 buffer
Parts:
- removed C15: 100n, Discret:C1, symbol C
- removed U10: 7400, Sockets_DIP:DIP-14__300_ELL, symbol 7400
- added unit 2 of U9
- U12: footprint Sockets_DIP:DIP-20__300_ELL -> (none)
Connections:
- wire segments 109 -> 113
Changed lines of the file:
@@
 	1050 6500 1150 6500
 Wire Wire Line
-	2550 6300 2600 6300
-Wire Wire Line
-	2550 6200 3300 6200
+	2550 6300 4100 6300
+Wire Wire Line
+	7850 6200 2550 6200
 Wire Wire Line
 	2550 6100 2600 6100
@@
 Text Label 6200 5400 0    60   ~ 0
 D7
-$Comp
-L 74LS273 U11
-U 1 1 544D56DD
-P 7050 5200
-F 0 "U11" H 7050 5050 60  0000 C CNN
-F 1 "74LS273" H 7050 4850 60  0000 C CNN
-F 2 "Sockets_DIP:DIP-20__300_ELL" H 7050 5200 60  0001 C CNN
-F 3 "" H 7050 5200 60  0000 C CNN
-	1    7050 5200
-	1    0    0    -1
-$EndComp
 Wire Wire Line
 	6350 5700 6250 5700
@@
 Text HLabel 2600 5900 2    60   Output ~ 0
 /CS_HIRAM
-Text HLabel 2600 6300 2    60   Input ~ 0
+Text HLabel 4100 6300 2    60   Input ~ 0
 RW
 Text HLabel 2600 5800 2    60   Output ~ 0
@@
 Text HLabel 2700 4650 2    60   Output ~ 0
 /CS_IO3
-Text HLabel 6250 5700 0    60   Input ~ 0
-/RESET
 $Comp
 L VCC #PWR032
@@
 	7750 5000 8750 5000
 Wire Wire Line
-	8750 5100 7750 5100
+	7750 5100 8750 5100
 Wire Wire Line
 	7750 5200 8750 5200
@@
 	8050 4400 8050 5550
 Connection ~ 8050 4900
-$Comp
-L 7400 U10
-U 1 1 546A6140
-P 4050 6000
-F 0 "U10" H 4050 6050 60  0000 C CNN
-F 1 "7400" H 4050 5900 60  0000 C CNN
-F 2 "Sockets_DIP:DIP-14__300_ELL" H 4050 6000 60  0001 C CNN
-F 3 "" H 4050 6000 60  0000 C CNN
-	1    4050 6000
-	1    0    0    -1
-$EndComp
-$Comp
-L 7400 U10
-U 3 1 546A616F
-P 5450 5600
-F 0 "U10" H 5450 5650 60  0000 C CNN
-F 1 "7400" H 5450 5500 60  0000 C CNN
-F 2 "Sockets_DIP:DIP-14__300_ELL" H 5450 5600 60  0001 C CNN
-F 3 "" H 5450 5600 60  0000 C CNN
-	3    5450 5600
-	1    0    0    -1
-$EndComp
-$Comp
-L 7400 U10
-U 4 1 546A61B5
-P 5450 6350
-F 0 "U10" H 5450 6400 60  0000 C CNN
-F 1 "7400" H 5450 6250 60  0000 C CNN
-F 2 "Sockets_DIP:DIP-14__300_ELL" H 5450 6350 60  0001 C CNN
-F 3 "" H 5450 6350 60  0000 C CNN
-	4    5450 6350
-	1    0    0    -1
-$EndComp
-$Comp
-L 7400 U10
-U 2 1 546A6200
-P 4050 6450
-F 0 "U10" H 4050 6500 60  0000 C CNN
-F 1 "7400" H 4050 6350 60  0000 C CNN
-F 2 "Sockets_DIP:DIP-14__300_ELL" H 4050 6450 60  0001 C CNN
-F 3 "" H 4050 6450 60  0000 C CNN
-	2    4050 6450
-	1    0    0    -1
-$EndComp
-$Comp
-L 74LS244 U12
-U 1 1 546A6264
-P 9450 5200
-F 0 "U12" H 9500 5000 60  0000 C CNN
-F 1 "74LS244" H 9550 4800 60  0000 C CNN
-F 2 "Sockets_DIP:DIP-20__300_ELL" H 9450 5200 60  0001 C CNN
-F 3 "" H 9450 5200 60  0000 C CNN
-	1    9450 5200
-	1    0    0    -1
-$EndComp
 Entry Wire Line
 	10350 4600 10250 4700
@@
 D7
 Wire Wire Line
-	6050 5600 6350 5600
-Wire Wire Line
-	8750 6350 6050 6350
-Wire Wire Line
-	8750 5600 8750 6350
-Connection ~ 8750 5700
-Wire Wire Line
-	4850 5700 4850 6250
-Wire Wire Line
-	4650 6000 4850 6000
-Connection ~ 4850 6000
-Wire Wire Line
-	3450 5500 3450 6100
+	5650 5600 6350 5600
+Wire Wire Line
+	3450 5500 3450 5850
 Wire Wire Line
 	2550 5500 3450 5500
-Connection ~ 3450 5900
-Wire Wire Line
-	2550 6300 2550 6450
-Wire Wire Line
-	2550 6450 3450 6450
-Wire Wire Line
-	3450 6350 3450 6700
-Connection ~ 3450 6450
-Wire Wire Line
-	4650 6450 4850 6450
-Wire Wire Line
-	4850 5500 4750 5500
-Wire Wire Line
-	4750 5500 4750 6700
-Wire Wire Line
-	4750 6700 3450 6700
-Connection ~ 3450 6550
 Text Label 7900 4700 0    60   ~ 0
 /ROMOFF
@@
 /ROMOFF
 Wire Wire Line
-	7850 4400 7850 4700
+	7850 4400 7850 6200
 Connection ~ 7850 4700
 Wire Wire Line
 	7950 4800 7900 4800
-Connection ~ 7900 4800
 Wire Wire Line
 	8150 4400 8150 5000
@@
 	1    0    0    -1
 $EndComp
-$Comp
-L C C15
-U 1 1 546A97B6
-P 6500 7200
-F 0 "C15" H 6500 7300 40  0000 L CNN
-F 1 "100n" H 6506 7115 40  0000 L CNN
-F 2 "Discret:C1" H 6538 7050 30  0001 C CNN
-F 3 "" H 6500 7200 60  0000 C CNN
-	1    6500 7200
-	1    0    0    -1
-$EndComp
 Connection ~ 6250 7000
 Connection ~ 6250 7400
+$Comp
+L 74LS139 U9
+U 2 1 548A0B1E
+P 4550 5600
+F 0 "U9" H 4550 5700 60  0000 C CNN
+F 1 "74LS139" H 4550 5500 60  0000 C CNN
+F 2 "Sockets_DIP:DIP-16__300_ELL" H 4550 5600 60  0001 C CNN
+F 3 "" H 4550 5600 60  0000 C CNN
+	2    4550 5600
+	1    0    0    -1
+$EndComp
+Wire Wire Line
+	3450 5850 3700 5850
+$Comp
+L GND #PWR036
+U 1 1 548A11B7
+P 3550 5450
+F 0 "#PWR036" H 3550 5450 30  0001 C CNN
+F 1 "GND" H 3550 5380 30  0001 C CNN
+F 2 "" H 3550 5450 60  0000 C CNN
+F 3 "" H 3550 5450 60  0000 C CNN
+	1    3550 5450
+	1    0    0    -1
+$EndComp
+Wire Wire Line
+	3700 5350 3550 5350
+Wire Wire Line
+	3550 5350 3550 5450
+Text GLabel 6250 5700 0    60   Input ~ 0
+/RESET
+Wire Wire Line
+	5650 5600 5650 5300
+Wire Wire Line
+	5650 5300 5400 5300
+$Comp
+L VCC #PWR037
+U 1 1 548A1DBF
+P 9450 4500
+F 0 "#PWR037" H 9450 4600 30  0001 C CNN
+F 1 "VCC" H 9450 4600 30  0000 C CNN
+F 2 "" H 9450 4500 60  0000 C CNN
+F 3 "" H 9450 4500 60  0000 C CNN
+	1    9450 4500
+	1    0    0    -1
+$EndComp
+Wire Wire Line
+	9450 4500 9450 4650
+$Comp
+L GND #PWR038
+U 1 1 548A1EB2
+P 9450 5950
+F 0 "#PWR038" H 9450 5950 30  0001 C CNN
+F 1 "GND" H 9450 5880 30  0001 C CNN
+F 2 "" H 9450 5950 60  0000 C CNN
+F 3 "" H 9450 5950 60  0000 C CNN
+	1    9450 5950
+	1    0    0    -1
+$EndComp
+Wire Wire Line
+	9450 5750 9450 5950
+$Comp
+L 74LS273 U11
+U 1 1 544D56DD
+P 7050 5200
+F 0 "U11" H 7050 5050 60  0000 C CNN
+F 1 "74LS273" H 7050 4850 60  0000 C CNN
+F 2 "Sockets_DIP:DIP-20__300_ELL" H 7050 5200 60  0001 C CNN
+F 3 "" H 7050 5200 60  0000 C CNN
+	1    7050 5200
+	1    0    0    -1
+$EndComp
+Wire Wire Line
+	3700 5500 3600 5500
+Wire Wire Line
+	3600 5500 3600 6300
+Connection ~ 3600 6300
+Wire Wire Line
+	5400 5500 5500 5500
+Wire Wire Line
+	5500 5500 5500 6100
+Wire Wire Line
+	5500 6100 8650 6100
+Wire Wire Line
+	8650 6100 8650 5600
+Wire Wire Line
+	8650 5700 8750 5700
+$Comp
+L 74LS244 U12
+U 1 1 54AD6087
+P 9450 5200
+F 0 "U12" H 9500 5000 60  0000 C CNN
+F 1 "74LS244" H 9550 4800 60  0000 C CNN
+F 2 "" H 9450 5200 60  0000 C CNN
+F 3 "" H 9450 5200 60  0000 C CNN
+	1    9450 5200
+	1    0    0    -1
+$EndComp
+Wire Wire Line
+	8650 5600 8750 5600
+Connection ~ 8650 5700
 $EndSCHEMATC

Commit message: anpassungen latch, decoder, 2. unit 393 inputs auf masse
Connections:
- net labels added: PHI2
- wire segments 113 -> 112
- no-connect marks 1 -> 3
Other:
- moved on the sheet: U9B
Changed lines of the file:
@@
 $EndComp
 $Comp
-L GND #PWR027
+L GND #PWR029
 U 1 1 544D50D2
 P 1550 6900
-F 0 "#PWR027" H 1550 6900 30  0001 C CNN
+F 0 "#PWR029" H 1550 6900 30  0001 C CNN
 F 1 "GND" H 1550 6830 30  0001 C CNN
 F 2 "" H 1550 6900 60  0000 C CNN
@@
 $EndComp
 $Comp
-L VCC #PWR028
+L VCC #PWR030
 U 1 1 544D50D8
 P 1550 5200
-F 0 "#PWR028" H 1550 5300 30  0001 C CNN
+F 0 "#PWR030" H 1550 5300 30  0001 C CNN
 F 1 "VCC" H 1550 5300 30  0000 C CNN
 F 2 "" H 1550 5200 60  0000 C CNN
@@
 Text Label 6200 5400 0    60   ~ 0
 D7
-Wire Wire Line
-	6350 5700 6250 5700
 Wire Wire Line
 	7750 4700 8750 4700
@@
 A15
 $Comp
-L VCC #PWR029
+L VCC #PWR031
 U 1 1 544D6887
 P 950 5350
-F 0 "#PWR029" H 950 5450 30  0001 C CNN
+F 0 "#PWR031" H 950 5450 30  0001 C CNN
 F 1 "VCC" H 950 5450 30  0000 C CNN
 F 2 "" H 950 5350 60  0000 C CNN
@@
 	2550 4650 2700 4650
 $Comp
-L VCC #PWR030
+L VCC #PWR032
 U 1 1 544D68A5
 P 1250 3850
-F 0 "#PWR030" H 1250 3950 30  0001 C CNN
+F 0 "#PWR032" H 1250 3950 30  0001 C CNN
 F 1 "VCC" H 1250 3950 30  0000 C CNN
 F 2 "" H 1250 3850 60  0000 C CNN
@@
 $EndComp
 $Comp
-L GND #PWR031
+L GND #PWR033
 U 1 1 544D68AB
 P 1250 4850
-F 0 "#PWR031" H 1250 4850 30  0001 C CNN
+F 0 "#PWR033" H 1250 4850 30  0001 C CNN
 F 1 "GND" H 1250 4780 30  0001 C CNN
 F 2 "" H 1250 4850 60  0000 C CNN
@@
 /CS_IO3
 $Comp
-L VCC #PWR032
+L VCC #PWR034
 U 1 1 544D6F18
 P 6750 4500
-F 0 "#PWR032" H 6750 4600 30  0001 C CNN
+F 0 "#PWR034" H 6750 4600 30  0001 C CNN
 F 1 "VCC" H 6750 4600 30  0000 C CNN
 F 2 "" H 6750 4500 60  0000 C CNN
@@
 	6750 4500 6750 4650
 $Comp
-L GND #PWR033
+L GND #PWR035
 U 1 1 544D700F
 P 6750 5950
-F 0 "#PWR033" H 6750 5950 30  0001 C CNN
+F 0 "#PWR035" H 6750 5950 30  0001 C CNN
 F 1 "GND" H 6750 5880 30  0001 C CNN
 F 2 "" H 6750 5950 60  0000 C CNN
@@
 	6750 5750 6750 5950
 $Comp
-L VCC #PWR034
+L VCC #PWR036
 U 1 1 544E9402
 P 5500 6950
-F 0 "#PWR034" H 5500 7050 30  0001 C CNN
+F 0 "#PWR036" H 5500 7050 30  0001 C CNN
 F 1 "VCC" H 5500 7050 30  0000 C CNN
 F 2 "" H 5500 6950 60  0000 C CNN
@@
 $EndComp
 $Comp
-L GND #PWR035
+L GND #PWR037
 U 1 1 544E9408
 P 5500 7500
-F 0 "#PWR035" H 5500 7500 30  0001 C CNN
+F 0 "#PWR037" H 5500 7500 30  0001 C CNN
 F 1 "GND" H 5500 7430 30  0001 C CNN
 F 2 "" H 5500 7500 60  0000 C CNN
@@
 D7
 Wire Wire Line
-	5650 5600 6350 5600
-Wire Wire Line
-	3450 5500 3450 5850
+	3450 5500 3450 5750
 Wire Wire Line
 	2550 5500 3450 5500
@@
 L 74LS139 U9
 U 2 1 548A0B1E
-P 4550 5600
-F 0 "U9" H 4550 5700 60  0000 C CNN
-F 1 "74LS139" H 4550 5500 60  0000 C CNN
-F 2 "Sockets_DIP:DIP-16__300_ELL" H 4550 5600 60  0001 C CNN
-F 3 "" H 4550 5600 60  0000 C CNN
-	2    4550 5600
-	1    0    0    -1
-$EndComp
-Wire Wire Line
-	3450 5850 3700 5850
-$Comp
-L GND #PWR036
-U 1 1 548A11B7
-P 3550 5450
-F 0 "#PWR036" H 3550 5450 30  0001 C CNN
-F 1 "GND" H 3550 5380 30  0001 C CNN
-F 2 "" H 3550 5450 60  0000 C CNN
-F 3 "" H 3550 5450 60  0000 C CNN
-	1    3550 5450
-	1    0    0    -1
-$EndComp
-Wire Wire Line
-	3700 5350 3550 5350
-Wire Wire Line
-	3550 5350 3550 5450
-Text GLabel 6250 5700 0    60   Input ~ 0
-/RESET
-Wire Wire Line
-	5650 5600 5650 5300
-Wire Wire Line
-	5650 5300 5400 5300
-$Comp
-L VCC #PWR037
+P 4550 5500
+F 0 "U9" H 4550 5600 60  0000 C CNN
+F 1 "74LS139" H 4550 5400 60  0000 C CNN
+F 2 "Sockets_DIP:DIP-16__300_ELL" H 4550 5500 60  0001 C CNN
+F 3 "" H 4550 5500 60  0000 C CNN
+	2    4550 5500
+	1    0    0    -1
+$EndComp
+Wire Wire Line
+	3450 5750 3700 5750
+Wire Wire Line
+	3700 5250 3500 5250
+$Comp
+L VCC #PWR038
 U 1 1 548A1DBF
 P 9450 4500
-F 0 "#PWR037" H 9450 4600 30  0001 C CNN
+F 0 "#PWR038" H 9450 4600 30  0001 C CNN
 F 1 "VCC" H 9450 4600 30  0000 C CNN
 F 2 "" H 9450 4500 60  0000 C CNN
@@
 	9450 4500 9450 4650
 $Comp
-L GND #PWR038
+L GND #PWR039
 U 1 1 548A1EB2
 P 9450 5950
-F 0 "#PWR038" H 9450 5950 30  0001 C CNN
+F 0 "#PWR039" H 9450 5950 30  0001 C CNN
 F 1 "GND" H 9450 5880 30  0001 C CNN
 F 2 "" H 9450 5950 60  0000 C CNN
@@
 $EndComp
 Wire Wire Line
-	3700 5500 3600 5500
-Wire Wire Line
-	3600 5500 3600 6300
+	3700 5400 3600 5400
+Wire Wire Line
+	3600 5400 3600 6300
 Connection ~ 3600 6300
 Wire Wire Line
-	5400 5500 5500 5500
-Wire Wire Line
-	5500 5500 5500 6100
-Wire Wire Line
-	5500 6100 8650 6100
-Wire Wire Line
-	8650 6100 8650 5600
-Wire Wire Line
-	8650 5700 8750 5700
+	5500 5800 5500 6050
+Wire Wire Line
+	8650 6050 5500 6050
 $Comp
 L 74LS244 U12
@@
 $EndComp
 Wire Wire Line
-	8650 5600 8750 5600
+	8750 5600 8650 5600
+Wire Wire Line
+	8650 5600 8650 6050
+Wire Wire Line
+	8750 5700 8650 5700
 Connection ~ 8650 5700
+Text GLabel 3500 5250 0    60   Input ~ 0
+PHI2
+Wire Wire Line
+	5500 5800 5400 5800
+NoConn ~ 5400 5400
+Wire Wire Line
+	6350 5600 5700 5600
+Wire Wire Line
+	5700 5600 5700 5200
+Wire Wire Line
+	5700 5200 5400 5200
+NoConn ~ 5400 5600
+Text HLabel 6200 5700 0    60   Input ~ 0
+/RESET
+Wire Wire Line
+	6200 5700 6350 5700
 $EndSCHEMATC
