File: kicad/cpu_mem/decoder.sch (KiCad schematic (older format))
At the start: 9 parts, among them P2 CONN_01X08, U11 74LS273, U12 74LS244, U5 GAL22V10, U9 74LS139

Commit message: reset_trig, letzte ratsline fix
Parts:
- removed C14: 100n, Discret:C1, symbol C
Changed lines of the file:
@@
 $EndComp
 $Comp
-L GND #PWR029
+L GND #PWR030
 U 1 1 544D50D2
 P 1550 6900
-F 0 "#PWR029" H 1550 6900 30  0001 C CNN
+F 0 "#PWR030" H 1550 6900 30  0001 C CNN
 F 1 "GND" H 1550 6830 30  0001 C CNN
 F 2 "" H 1550 6900 60  0000 C CNN
@@
 $EndComp
 $Comp
-L VCC #PWR030
+L VCC #PWR031
 U 1 1 544D50D8
 P 1550 5200
-F 0 "#PWR030" H 1550 5300 30  0001 C CNN
+F 0 "#PWR031" H 1550 5300 30  0001 C CNN
 F 1 "VCC" H 1550 5300 30  0000 C CNN
 F 2 "" H 1550 5200 60  0000 C CNN
@@
 A15
 $Comp
-L VCC #PWR031
+L VCC #PWR032
 U 1 1 544D6887
 P 950 5350
-F 0 "#PWR031" H 950 5450 30  0001 C CNN
+F 0 "#PWR032" H 950 5450 30  0001 C CNN
 F 1 "VCC" H 950 5450 30  0000 C CNN
 F 2 "" H 950 5350 60  0000 C CNN
@@
 	2550 4650 2700 4650
 $Comp
-L VCC #PWR032
+L VCC #PWR033
 U 1 1 544D68A5
 P 1250 3850
-F 0 "#PWR032" H 1250 3950 30  0001 C CNN
+F 0 "#PWR033" H 1250 3950 30  0001 C CNN
 F 1 "VCC" H 1250 3950 30  0000 C CNN
 F 2 "" H 1250 3850 60  0000 C CNN
@@
 $EndComp
 $Comp
-L GND #PWR033
+L GND #PWR034
 U 1 1 544D68AB
 P 1250 4850
-F 0 "#PWR033" H 1250 4850 30  0001 C CNN
+F 0 "#PWR034" H 1250 4850 30  0001 C CNN
 F 1 "GND" H 1250 4780 30  0001 C CNN
 F 2 "" H 1250 4850 60  0000 C CNN
@@
 /CS_IO3
 $Comp
-L VCC #PWR034
+L VCC #PWR035
 U 1 1 544D6F18
 P 6750 4500
-F 0 "#PWR034" H 6750 4600 30  0001 C CNN
+F 0 "#PWR035" H 6750 4600 30  0001 C CNN
 F 1 "VCC" H 6750 4600 30  0000 C CNN
 F 2 "" H 6750 4500 60  0000 C CNN
@@
 	1    0    0    -1
 $EndComp
-Wire Wire Line
-	6750 4500 6750 4650
-$Comp
-L GND #PWR035
+$Comp
+L GND #PWR036
 U 1 1 544D700F
 P 6750 5950
-F 0 "#PWR035" H 6750 5950 30  0001 C CNN
+F 0 "#PWR036" H 6750 5950 30  0001 C CNN
 F 1 "GND" H 6750 5880 30  0001 C CNN
 F 2 "" H 6750 5950 60  0000 C CNN
@@
 	6750 5750 6750 5950
 $Comp
-L VCC #PWR036
+L VCC #PWR037
 U 1 1 544E9402
 P 5500 6950
-F 0 "#PWR036" H 5500 7050 30  0001 C CNN
+F 0 "#PWR037" H 5500 7050 30  0001 C CNN
 F 1 "VCC" H 5500 7050 30  0000 C CNN
 F 2 "" H 5500 6950 60  0000 C CNN
@@
 $EndComp
 $Comp
-L GND #PWR037
+L GND #PWR038
 U 1 1 544E9408
 P 5500 7500
-F 0 "#PWR037" H 5500 7500 30  0001 C CNN
+F 0 "#PWR038" H 5500 7500 30  0001 C CNN
 F 1 "GND" H 5500 7430 30  0001 C CNN
 F 2 "" H 5500 7500 60  0000 C CNN
@@
 	1    0    0    -1
 $EndComp
-Wire Wire Line
-	5500 6950 5500 7000
 Wire Wire Line
 	5500 7400 5500 7500
@@
 Connection ~ 8550 5400
 $Comp
-L C C14
-U 1 1 546A978B
-P 6250 7200
-F 0 "C14" H 6250 7300 40  0000 L CNN
-F 1 "100n" H 6256 7115 40  0000 L CNN
-F 2 "Discret:C1" H 6288 7050 30  0001 C CNN
-F 3 "" H 6250 7200 60  0000 C CNN
-	1    6250 7200
-	1    0    0    -1
-$EndComp
-Connection ~ 6250 7000
-Connection ~ 6250 7400
-$Comp
 L 74LS139 U9
 U 2 1 548A0B1E
@@
 	3700 5250 3500 5250
 $Comp
-L VCC #PWR038
+L VCC #PWR039
 U 1 1 548A1DBF
 P 9450 4500
-F 0 "#PWR038" H 9450 4600 30  0001 C CNN
+F 0 "#PWR039" H 9450 4600 30  0001 C CNN
 F 1 "VCC" H 9450 4600 30  0000 C CNN
 F 2 "" H 9450 4500 60  0000 C CNN
@@
 	9450 4500 9450 4650
 $Comp
-L GND #PWR039
+L GND #PWR040
 U 1 1 548A1EB2
 P 9450 5950
-F 0 "#PWR039" H 9450 5950 30  0001 C CNN
+F 0 "#PWR040" H 9450 5950 30  0001 C CNN
 F 1 "GND" H 9450 5880 30  0001 C CNN
 F 2 "" H 9450 5950 60  0000 C CNN
@@
 	5500 5800 5500 6050
 Wire Wire Line
-	8650 6050 5500 6050
+	5500 6050 8650 6050
 $Comp
 L 74LS244 U12
@@
 Wire Wire Line
 	6200 5700 6350 5700
+Wire Wire Line
+	5500 7000 5500 6950
+Wire Wire Line
+	6750 4500 6750 4650
 $EndSCHEMATC

Commit message: power anschluss
Parts:
- U12: footprint (none) -> Sockets_DIP:DIP-20__300_ELL
Changed lines of the file:
@@
 $EndComp
 $Comp
-L GND #PWR030
+L GND #PWR032
 U 1 1 544D50D2
 P 1550 6900
-F 0 "#PWR030" H 1550 6900 30  0001 C CNN
+F 0 "#PWR032" H 1550 6900 30  0001 C CNN
 F 1 "GND" H 1550 6830 30  0001 C CNN
 F 2 "" H 1550 6900 60  0000 C CNN
@@
 $EndComp
 $Comp
-L VCC #PWR031
+L VCC #PWR033
 U 1 1 544D50D8
 P 1550 5200
-F 0 "#PWR031" H 1550 5300 30  0001 C CNN
+F 0 "#PWR033" H 1550 5300 30  0001 C CNN
 F 1 "VCC" H 1550 5300 30  0000 C CNN
 F 2 "" H 1550 5200 60  0000 C CNN
@@
 A15
 $Comp
-L VCC #PWR032
+L VCC #PWR034
 U 1 1 544D6887
 P 950 5350
-F 0 "#PWR032" H 950 5450 30  0001 C CNN
+F 0 "#PWR034" H 950 5450 30  0001 C CNN
 F 1 "VCC" H 950 5450 30  0000 C CNN
 F 2 "" H 950 5350 60  0000 C CNN
@@
 	2550 4650 2700 4650
 $Comp
-L VCC #PWR033
+L VCC #PWR035
 U 1 1 544D68A5
 P 1250 3850
-F 0 "#PWR033" H 1250 3950 30  0001 C CNN
+F 0 "#PWR035" H 1250 3950 30  0001 C CNN
 F 1 "VCC" H 1250 3950 30  0000 C CNN
 F 2 "" H 1250 3850 60  0000 C CNN
@@
 $EndComp
 $Comp
-L GND #PWR034
+L GND #PWR036
 U 1 1 544D68AB
 P 1250 4850
-F 0 "#PWR034" H 1250 4850 30  0001 C CNN
+F 0 "#PWR036" H 1250 4850 30  0001 C CNN
 F 1 "GND" H 1250 4780 30  0001 C CNN
 F 2 "" H 1250 4850 60  0000 C CNN
@@
 /CS_IO3
 $Comp
-L VCC #PWR035
+L VCC #PWR037
 U 1 1 544D6F18
 P 6750 4500
-F 0 "#PWR035" H 6750 4600 30  0001 C CNN
+F 0 "#PWR037" H 6750 4600 30  0001 C CNN
 F 1 "VCC" H 6750 4600 30  0000 C CNN
 F 2 "" H 6750 4500 60  0000 C CNN
@@
 $EndComp
 $Comp
-L GND #PWR036
+L GND #PWR038
 U 1 1 544D700F
 P 6750 5950
-F 0 "#PWR036" H 6750 5950 30  0001 C CNN
+F 0 "#PWR038" H 6750 5950 30  0001 C CNN
 F 1 "GND" H 6750 5880 30  0001 C CNN
 F 2 "" H 6750 5950 60  0000 C CNN
@@
 	6750 5750 6750 5950
 $Comp
-L VCC #PWR037
+L VCC #PWR039
 U 1 1 544E9402
 P 5500 6950
-F 0 "#PWR037" H 5500 7050 30  0001 C CNN
+F 0 "#PWR039" H 5500 7050 30  0001 C CNN
 F 1 "VCC" H 5500 7050 30  0000 C CNN
 F 2 "" H 5500 6950 60  0000 C CNN
@@
 $EndComp
 $Comp
-L GND #PWR038
+L GND #PWR040
 U 1 1 544E9408
 P 5500 7500
-F 0 "#PWR038" H 5500 7500 30  0001 C CNN
+F 0 "#PWR040" H 5500 7500 30  0001 C CNN
 F 1 "GND" H 5500 7430 30  0001 C CNN
 F 2 "" H 5500 7500 60  0000 C CNN
@@
 	3700 5250 3500 5250
 $Comp
-L VCC #PWR039
+L VCC #PWR041
 U 1 1 548A1DBF
 P 9450 4500
-F 0 "#PWR039" H 9450 4600 30  0001 C CNN
+F 0 "#PWR041" H 9450 4600 30  0001 C CNN
 F 1 "VCC" H 9450 4600 30  0000 C CNN
 F 2 "" H 9450 4500 60  0000 C CNN
@@
 	9450 4500 9450 4650
 $Comp
-L GND #PWR040
+L GND #PWR042
 U 1 1 548A1EB2
 P 9450 5950
-F 0 "#PWR040" H 9450 5950 30  0001 C CNN
+F 0 "#PWR042" H 9450 5950 30  0001 C CNN
 F 1 "GND" H 9450 5880 30  0001 C CNN
 F 2 "" H 9450 5950 60  0000 C CNN
@@
 F 0 "U12" H 9500 5000 60  0000 C CNN
 F 1 "74LS244" H 9550 4800 60  0000 C CNN
-F 2 "" H 9450 5200 60  0000 C CNN
+F 2 "Sockets_DIP:DIP-20__300_ELL" H 9450 5200 60  0001 C CNN
 F 3 "" H 9450 5200 60  0000 C CNN
 	1    9450 5200

Commit message: blinkenlights
Parts:
- added D10, D11, D4, D5, D6, D7, D8, D9: LED, LEDs:LED-3MM, symbol LED
- added R10, R11, R12, R13, R14, R15, R16, R17: 270, Discret:R3, symbol R
Connections:
- wire segments 112 -> 137
