File: kicad/tms9929/tms9929_sram_snd.sch (KiCad schematic (older format))
At the start: 59 parts, among them Q1 BC550, Q10 BC550, Q2 BC550, Q3 BC550, Q4 BC550, Q5 BC550, Q6 BC550, Q7 BC550, Q8 BC550, Q9 BC550, U1 TMS9929A, U10 7400, U2 74HCT04, U3 74HCT574, U4 74HCT574, U5 74HCT574, U6 HM62256BLFP-5SLT

Commit message: +review
Connections:
- wire segments 277 -> 241
Changed lines of the file:
@@
 LIBS:contrib
 LIBS:valves
+LIBS:tms9929_sram_snd-cache
 EELAYER 24 0
 EELAYER END
@@
 	1    0    0    -1
 $EndComp
-Entry Wire Line
-	5950 2250 6050 2350
-Entry Wire Line
-	5950 2350 6050 2450
-Entry Wire Line
-	5950 2450 6050 2550
-Entry Wire Line
-	5950 2550 6050 2650
-Entry Wire Line
-	5950 2650 6050 2750
-Entry Wire Line
-	5950 2750 6050 2850
-Entry Wire Line
-	5950 2850 6050 2950
 $Comp
 L CRYSTAL 10.738MHz1
@@
 	1    0    0    -1
 $EndComp
-Text Label 5900 2250 0    60   ~ 0
-AD1
-Text Label 5900 2150 0    60   ~ 0
-AD0
-Text Label 5900 2350 0    60   ~ 0
-AD2
-Text Label 5900 2450 0    60   ~ 0
-AD3
-Text Label 5900 2550 0    60   ~ 0
-AD4
-Text Label 5900 2650 0    60   ~ 0
-AD5
-Text Label 5900 2750 0    60   ~ 0
-AD6
-Text Label 5900 2850 0    60   ~ 0
-AD7
 Text Label 6000 3050 0    60   ~ 0
 RAS
@@
 	1    0    0    -1
 $EndComp
-Entry Wire Line
-	5950 2150 6050 2250
 $Comp
 L 7400 U10
@@
 	13000 4950 12750 4950
 Wire Wire Line
-	11850 6050 13950 6050
-Wire Wire Line
-	13950 6050 15100 6050
+	11850 6050 15100 6050
 Wire Wire Line
 	12600 8600 12600 7950
@@
 Connection ~ 12950 5350
 Wire Wire Line
-	12950 5350 12950 7100
-Wire Wire Line
-	12950 7100 12950 9000
+	12950 5350 12950 9000
 Wire Wire Line
 	13400 7100 12950 7100
@@
 Connection ~ 12600 5350
 Wire Wire Line
-	12600 5350 12950 5350
-Wire Wire Line
-	12950 5350 13000 5350
+	12600 5350 13000 5350
 Wire Wire Line
 	14600 5900 14600 5950
@@
 	12600 5900 12600 5950
 Wire Wire Line
-	11650 5000 12200 5000
-Wire Wire Line
-	12200 5000 12300 5000
-Wire Wire Line
-	12200 3950 12200 5000
-Wire Wire Line
-	12200 5000 12200 5400
-Wire Wire Line
-	12600 5200 12600 5350
-Wire Wire Line
-	12600 5350 12600 5400
+	11650 5000 12300 5000
+Wire Wire Line
+	12200 3950 12200 5400
+Wire Wire Line
+	12600 5200 12600 5400
 Wire Wire Line
 	12600 3650 12600 4800
@@
 Connection ~ 11850 6050
 Wire Wire Line
-	11850 3650 11850 6050
-Wire Wire Line
-	11850 6050 11850 7950
-Wire Wire Line
-	11850 7950 11850 9250
-Wire Wire Line
-	11850 7950 13950 7950
-Wire Wire Line
-	13950 7950 15100 7950
+	11850 3650 11850 9250
+Wire Wire Line
+	11850 7950 15100 7950
 Wire Wire Line
 	15100 8400 15100 8450
@@
 Connection ~ 12600 9150
 Wire Wire Line
-	12600 9000 12600 9150
-Wire Wire Line
-	12600 9150 12600 9200
-Wire Wire Line
-	12600 9150 12750 9150
-Wire Wire Line
-	12750 9150 13400 9150
+	12600 9000 12600 9200
+Wire Wire Line
+	12600 9150 13400 9150
 Connection ~ 13950 7950
 Connection ~ 13950 9000
@@
 	13950 9150 13900 9150
 Wire Wire Line
-	13950 8950 13950 9000
-Wire Wire Line
-	13950 9000 13950 9150
-Wire Wire Line
-	13950 9150 13950 9200
+	13950 8950 13950 9200
 Wire Wire Line
 	14000 8750 14600 8750
 Wire Wire Line
-	14600 8500 14600 8750
-Wire Wire Line
-	14600 8750 14600 9300
+	14600 8500 14600 9300
 Wire Wire Line
 	14100 8200 14800 8200
@@
 	15100 7950 15100 8000
 Wire Wire Line
-	13950 8450 13950 8500
-Wire Wire Line
-	13950 8500 13950 8550
+	13950 8450 13950 8550
 Wire Wire Line
 	14050 8500 13950 8500
@@
 	14600 7800 14600 7850
 Wire Wire Line
-	11650 6900 12200 6900
-Wire Wire Line
-	12200 6900 12300 6900
+	11650 6900 12300 6900
 Wire Wire Line
 	12200 7300 12200 6900
 Connection ~ 12600 7250
 Wire Wire Line
-	12600 7100 12600 7250
-Wire Wire Line
-	12600 7250 12600 7300
-Wire Wire Line
-	12600 7250 12850 7250
-Wire Wire Line
-	12850 7250 13400 7250
+	12600 7100 12600 7300
+Wire Wire Line
+	12600 7250 13400 7250
 Connection ~ 13950 6050
 Wire Wire Line
@@
 	13950 7250 13900 7250
 Wire Wire Line
-	13950 7050 13950 7100
-Wire Wire Line
-	13950 7100 13950 7250
-Wire Wire Line
-	13950 7250 13950 7300
+	13950 7050 13950 7300
 Wire Wire Line
 	14000 6850 14600 6850
 Wire Wire Line
-	14600 6600 14600 6850
-Wire Wire Line
-	14600 6850 14600 7400
+	14600 6600 14600 7400
 Wire Wire Line
 	14100 6300 14800 6300
@@
 	15100 6050 15100 6100
 Wire Wire Line
-	13950 6550 13950 6600
-Wire Wire Line
-	13950 6600 13950 6650
+	13950 6550 13950 6650
 Wire Wire Line
 	14050 6600 13950 6600
@@
 	15100 4600 15150 4600
 Wire Wire Line
-	11850 3650 14600 3650
-Wire Wire Line
-	14600 3650 15100 3650
-Wire Wire Line
-	15100 3650 15500 3650
+	11850 3650 15500 3650
 Wire Wire Line
 	15100 3650 15100 4200
@@
 Connection ~ 14600 5350
 Wire Wire Line
-	14600 5150 14600 5350
-Wire Wire Line
-	14600 5350 14600 5400
+	14600 5150 14600 5400
 Wire Wire Line
 	13500 5350 14600 5350
@@
 Connection ~ 13550 4950
 Wire Wire Line
-	13550 4950 13550 5150
-Wire Wire Line
-	13550 5150 13550 5400
-Wire Wire Line
-	13500 4950 13550 4950
-Wire Wire Line
-	13550 4950 13600 4950
+	13550 4950 13550 5400
+Wire Wire Line
+	13500 4950 13600 4950
 Connection ~ 14050 4950
 Wire Wire Line
@@
 	14550 4700 14600 4700
 Wire Wire Line
-	14000 4950 14050 4950
-Wire Wire Line
-	14050 4950 14300 4950
+	14000 4950 14300 4950
 Connection ~ 14600 4700
 Wire Wire Line
-	14600 4650 14600 4700
-Wire Wire Line
-	14600 4700 14600 4750
+	14600 4650 14600 4750
 Wire Wire Line
 	14800 4400 14750 4400
 Connection ~ 3650 1950
 Wire Wire Line
-	3650 950  3650 1350
-Wire Wire Line
-	3650 1350 3650 1950
-Wire Wire Line
-	3650 1950 3650 2150
-Wire Wire Line
-	4050 1350 4100 1350
-Wire Wire Line
-	4100 1350 4350 1350
-Wire Wire Line
-	4050 1950 4100 1950
-Wire Wire Line
-	4100 1950 4350 1950
-Wire Bus Line
-	6050 2100 6050 2250
-Wire Bus Line
-	6050 2250 6050 2350
-Wire Bus Line
-	6050 2350 6050 2450
-Wire Bus Line
-	6050 2450 6050 2550
-Wire Bus Line
-	6050 2550 6050 2650
-Wire Bus Line
-	6050 2650 6050 2750
-Wire Bus Line
-	6050 2750 6050 2850
-Wire Bus Line
-	6050 2850 6050 2950
-Wire Wire Line
-	11650 8800 12200 8800
-Wire Wire Line
-	12200 8800 12300 8800
-Wire Wire Line
-	2600 4450 2650 4450
-Wire Wire Line
-	2650 4450 2700 4450
+	3650 950  3650 2150
+Wire Wire Line
+	4050 1350 4350 1350
+Wire Wire Line
+	4050 1950 4350 1950
+Wire Wire Line
+	11650 8800 12300 8800
+Wire Wire Line
+	2600 4450 2700 4450
 Wire Wire Line
 	2650 4450 2650 5150
@@
 	2600 5350 2700 5350
 Wire Wire Line
-	1400 4900 1400 5250
-Wire Wire Line
-	1400 5250 1400 5450
+	1400 4900 1400 5450
 Wire Wire Line
 	1400 4900 2450 4900
@@
 	3900 4750 3900 5250
 Wire Bus Line
-	2550 1550 2550 1650
-Wire Bus Line
-	2550 1650 2550 1750
-Wire Bus Line
-	2550 1750 2550 1850
-Wire Bus Line
-	2550 1850 2550 1950
-Wire Bus Line
-	2550 1950 2550 2050
-Wire Bus Line
-	2550 2050 2550 2150
-Wire Bus Line
-	2550 2150 2550 2250
-Wire Bus Line
-	2550 2250 2550 2350
-Wire Bus Line
-	2550 2350 2550 2450
+	2550 1550 2550 2450
 Wire Wire Line
 	4350 3850 4250 3850
@@
 D7
 Wire Wire Line
-	1650 10050 1900 10050
-Wire Wire Line
-	1900 10050 2150 10050
-Wire Wire Line
-	2150 10050 2400 10050
-Wire Wire Line
-	2400 10050 2650 10050
-Wire Wire Line
-	2650 10050 2900 10050
-Wire Wire Line
-	1650 10450 1900 10450
-Wire Wire Line
-	1900 10450 2150 10450
-Wire Wire Line
-	2150 10450 2400 10450
-Wire Wire Line
-	2400 10450 2650 10450
-Wire Wire Line
-	2650 10450 2900 10450
+	1650 10050 2900 10050
+Wire Wire Line
+	1650 10450 2900 10450
 NoConn ~ 9600 3200
 NoConn ~ 9600 1950
+Wire Wire Line
+	6200 2150 5950 2150
+Wire Wire Line
+	6200 2250 5950 2250
+Wire Wire Line
+	6200 2350 5950 2350
+Wire Wire Line
+	6200 2450 5950 2450
+Wire Wire Line
+	6200 2550 5950 2550
+Wire Wire Line
+	6200 2650 5950 2650
+Wire Wire Line
+	6200 2750 5950 2750
+Wire Wire Line
+	6200 2850 5950 2850
+Text Label 6000 2150 0    60   ~ 0
+AD0
+Text Label 6000 2250 0    60   ~ 0
+AD1
+Text Label 6000 2350 0    60   ~ 0
+AD2
+Text Label 6000 2450 0    60   ~ 0
+AD3
+Text Label 6000 2550 0    60   ~ 0
+AD4
+Text Label 6000 2650 0    60   ~ 0
+AD5
+Text Label 6000 2750 0    60   ~ 0
+AD6
+Text Label 6000 2850 0    60   ~ 0
+AD7
 $EndSCHEMATC

Commit message: +review
Connections:
- wire segments 241 -> 249
Changed lines of the file:
@@
 	1    0    0    -1
 $EndComp
-Entry Wire Line
-	2450 1550 2550 1650
-Entry Wire Line
-	2450 1650 2550 1750
-Entry Wire Line
-	2450 1750 2550 1850
-Entry Wire Line
-	2450 1850 2550 1950
-Entry Wire Line
-	2450 1950 2550 2050
-Entry Wire Line
-	2450 2050 2550 2150
-Entry Wire Line
-	2450 2150 2550 2250
-Entry Wire Line
-	2450 2250 2550 2350
 Text GLabel 1000 4350 0    60   Input ~ 0
 /CS_VDP
 Text GLabel 4150 3650 0    60   Input ~ 0
 /IRQ
-$Sheet
-S 1750 1500 700  1500
-U 542278A8
-F0 "50Pin" 60
-F1 "50pin_connector.sch" 60
-F2 "A0" I R 2450 2900 60
-F3 "D0" I R 2450 1550 60
-F4 "D1" I R 2450 1650 60
-F5 "D2" I R 2450 1750 60
-F6 "D3" I R 2450 1850 60
-F7 "D4" I R 2450 1950 60
-F8 "D5" I R 2450 2050 60
-F9 "D6" I R 2450 2150 60
-F10 "D7" I R 2450 2250 60
-$EndSheet
 Text GLabel 4250 3850 0    60   Input ~ 0
 /RESET
@@
 Wire Wire Line
 	3900 4750 3900 5250
-Wire Bus Line
-	2550 1550 2550 2450
 Wire Wire Line
 	4350 3850 4250 3850
@@
 Text Label 6000 2850 0    60   ~ 0
 AD7
+$Sheet
+S 1750 1500 700  1500
+U 542278A8
+F0 "50Pin" 60
+F1 "50pin_connector.sch" 60
+F2 "A0" I R 2450 2900 60
+F3 "D0" I R 2450 1550 60
+F4 "D1" I R 2450 1650 60
+F5 "D2" I R 2450 1750 60
+F6 "D3" I R 2450 1850 60
+F7 "D4" I R 2450 1950 60
+F8 "D5" I R 2450 2050 60
+F9 "D6" I R 2450 2150 60
+F10 "D7" I R 2450 2250 60
+$EndSheet
+Wire Wire Line
+	2600 1550 2450 1550
+Wire Wire Line
+	2600 1650 2450 1650
+Wire Wire Line
+	2600 1750 2450 1750
+Wire Wire Line
+	2600 1850 2450 1850
+Wire Wire Line
+	2600 1950 2450 1950
+Wire Wire Line
+	2600 2050 2450 2050
+Wire Wire Line
+	2600 2150 2450 2150
+Wire Wire Line
+	2600 2250 2450 2250
+Text Label 2500 1550 0    60   ~ 0
+D0
+Text Label 2500 1650 0    60   ~ 0
+D1
+Text Label 2500 1750 0    60   ~ 0
+D2
+Text Label 2500 1850 0    60   ~ 0
+D3
+Text Label 2500 1950 0    60   ~ 0
+D4
+Text Label 2500 2050 0    60   ~ 0
+D5
+Text Label 2500 2150 0    60   ~ 0
+D6
+Text Label 2500 2250 0    60   ~ 0
+D7
 $EndSCHEMATC

Commit message: layout
Parts:
- removed GND1, GND2: GND, symbol GND
- added P1: CONN_01X05, symbol CONN_01X05
- 10.738MHz1: footprint (none) -> Crystals:Crystal_HC49-U_Horizontal_Typ1
Connections:
- wire segments 249 -> 260
Other:
- moved on the sheet: C13, C14, C15, C16, Q1, Q10, Q2, Q3, Q4, Q5, Q6, Q7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

Commit message: +review, update
Parts:
- removed P1: CONN_01X05, symbol CONN_01X05
- added C10: 100nF, symbol C
- added P?: CONN_01X05, symbol CONN_01X05
- 10.738MHz1: footprint Crystals:Crystal_HC49-U_Horizontal_Typ1 -> (none)
- C14: value CP2 -> 16µ/10V
Connections:
- net labels added: RGB-B, RGB-G, RGB-R, SYNC
- wire segments 260 -> 257
Other:
- moved on the sheet: C13, C14, C15, C16, Q1, Q10, Q2, Q3, Q4, Q5, Q6, Q7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

Commit message: +update
Parts:
- gave numbers to parts that had none: 1
Changed lines of the file:
@@
 $EndComp
 $Comp
-L CONN_01X05 P?
+L CONN_01X05 P1
 U 1 1 54B02B77
 P 15250 3750
-F 0 "P?" H 15250 4050 50  0000 C CNN
+F 0 "P1" H 15250 4050 50  0000 C CNN
 F 1 "CONN_01X05" V 15350 3750 50  0000 C CNN
 F 2 "" H 15250 3750 60  0000 C CNN
@@
 	14400 3550 15050 3550
 $Comp
-L GND #PWR?
+L GND #PWR019
 U 1 1 54B05606
 P 15000 4050
-F 0 "#PWR?" H 15000 4050 30  0001 C CNN
+F 0 "#PWR019" H 15000 4050 30  0001 C CNN
 F 1 "GND" H 15000 3980 30  0001 C CNN
 F 2 "" H 15000 4050 60  0000 C CNN

Commit message: +update, 6mm poti
Parts:
- RV1, RV2, RV3: value POT -> 5K
Connections:
- wire segments 257 -> 268
- no-connect marks 2 -> 4

Commit message: +update, add rca jacks
Parts:
- removed P1: CONN_01X05, symbol CONN_01X05
- added Blue1, Green1, Red1, Sync1: RCA, symbol CONN_01X02
Connections:
- net labels removed: RGB-R
- wire segments 268 -> 269
Other:
- moved on the sheet: R21
Changed lines of the file:
@@
 L R R21
 U 1 1 541A93AC
-P 13900 3650
-F 0 "R21" V 13980 3650 40  0000 C CNN
-F 1 "100" V 13907 3651 40  0000 C CNN
-F 2 "" V 13830 3650 30  0000 C CNN
-F 3 "" H 13900 3650 30  0000 C CNN
-	1    13900 3650
+P 13950 3800
+F 0 "R21" V 14030 3800 40  0000 C CNN
+F 1 "100" V 13957 3801 40  0000 C CNN
+F 2 "" V 13880 3800 30  0000 C CNN
+F 3 "" H 13950 3800 30  0000 C CNN
+	1    13950 3800
 	0    1    1    0
 $EndComp
@@
 	14150 5600 14400 5600
 Wire Wire Line
-	14150 3650 15050 3650
+	14200 3800 15100 3800
 Wire Wire Line
 	14000 3200 14000 3250
@@
 	12550 5650 12450 5650
 Connection ~ 12450 5650
-Wire Wire Line
-	13600 3650 13650 3650
 Wire Wire Line
 	10350 2700 14000 2700
@@
 Text Label 14200 3250 0    60   ~ 0
 SYNC
-Text Label 14200 3650 0    60   ~ 0
-RGB-R
 Text Label 14200 5600 0    60   ~ 0
 RGB-G
@@
 	1    0    0    -1
 $EndComp
-$Comp
-L CONN_01X05 P1
-U 1 1 54B02B77
-P 15250 3750
-F 0 "P1" H 15250 4050 50  0000 C CNN
-F 1 "CONN_01X05" V 15350 3750 50  0000 C CNN
-F 2 "" H 15250 3750 60  0000 C CNN
-F 3 "" H 15250 3750 60  0000 C CNN
-	1    15250 3750
-	1    0    0    -1
-$EndComp
-Wire Wire Line
-	14400 5600 14400 3750
-Wire Wire Line
-	14400 3750 15050 3750
-Wire Wire Line
-	14500 7500 14500 3850
-Wire Wire Line
-	14500 3850 15050 3850
-Wire Wire Line
-	14000 3250 14400 3250
-Wire Wire Line
-	14400 3250 14400 3550
-Wire Wire Line
-	14400 3550 15050 3550
+Wire Wire Line
+	14400 4100 15100 4100
+Wire Wire Line
+	14500 7500 14500 4400
+Wire Wire Line
+	14500 4400 15100 4400
+Wire Wire Line
+	14000 3250 15100 3250
 $Comp
 L GND #PWR019
 U 1 1 54B05606
-P 15000 4050
-F 0 "#PWR019" H 15000 4050 30  0001 C CNN
-F 1 "GND" H 15000 3980 30  0001 C CNN
-F 2 "" H 15000 4050 60  0000 C CNN
-F 3 "" H 15000 4050 60  0000 C CNN
-	1    15000 4050
-	1    0    0    -1
-$EndComp
-Wire Wire Line
-	15050 3950 15000 3950
-Wire Wire Line
-	15000 3950 15000 4050
+P 15000 4000
+F 0 "#PWR019" H 15000 4000 30  0001 C CNN
+F 1 "GND" H 15000 3930 30  0001 C CNN
+F 2 "" H 15000 4000 60  0000 C CNN
+F 3 "" H 15000 4000 60  0000 C CNN
+	1    15000 4000
+	0    1    1    0
+$EndComp
+Wire Wire Line
+	15100 4000 15000 4000
 Wire Wire Line
 	7800 2200 8000 2200
@@
 Wire Wire Line
 	8700 3500 8700 3550
+$Comp
+L CONN_01X02 Sync1
+U 1 1 54EA3E4A
+P 15300 3200
+F 0 "Sync1" H 15300 3350 50  0000 C CNN
+F 1 "RCA" V 15400 3200 50  0000 C CNN
+F 2 "" H 15300 3200 60  0000 C CNN
+F 3 "" H 15300 3200 60  0000 C CNN
+	1    15300 3200
+	1    0    0    -1
+$EndComp
+$Comp
+L CONN_01X02 Red1
+U 1 1 54EA3E9B
+P 15300 3750
+F 0 "Red1" H 15300 3900 50  0000 C CNN
+F 1 "RCA" V 15400 3750 50  0000 C CNN
+F 2 "" H 15300 3750 60  0000 C CNN
+F 3 "" H 15300 3750 60  0000 C CNN
+	1    15300 3750
+	1    0    0    -1
+$EndComp
+$Comp
+L CONN_01X02 Green1
+U 1 1 54EA3ECE
+P 15300 4050
+F 0 "Green1" H 15300 4200 50  0000 C CNN
+F 1 "RCA" V 15400 4050 50  0000 C CNN
+F 2 "" H 15300 4050 60  0000 C CNN
+F 3 "" H 15300 4050 60  0000 C CNN
+	1    15300 4050
+	1    0    0    -1
+$EndComp
+$Comp
+L CONN_01X02 Blue1
+U 1 1 54EA3EFF
+P 15300 4350
+F 0 "Blue1" H 15300 4500 50  0000 C CNN
+F 1 "RCA" V 15400 4350 50  0000 C CNN
+F 2 "" H 15300 4350 60  0000 C CNN
+F 3 "" H 15300 4350 60  0000 C CNN
+	1    15300 4350
+	1    0    0    -1
+$EndComp
+Wire Wire Line
+	13600 3650 13600 3800
+Wire Wire Line
+	13600 3800 13700 3800
+$Comp
+L GND #PWR031
+U 1 1 54EA4F07
+P 15000 3700
+F 0 "#PWR031" H 15000 3700 30  0001 C CNN
+F 1 "GND" H 15000 3630 30  0001 C CNN
+F 2 "" H 15000 3700 60  0000 C CNN
+F 3 "" H 15000 3700 60  0000 C CNN
+	1    15000 3700
+	0    1    1    0
+$EndComp
+Wire Wire Line
+	15100 3700 15000 3700
+$Comp
+L GND #PWR032
+U 1 1 54EA4FCE
+P 15000 3150
+F 0 "#PWR032" H 15000 3150 30  0001 C CNN
+F 1 "GND" H 15000 3080 30  0001 C CNN
+F 2 "" H 15000 3150 60  0000 C CNN
+F 3 "" H 15000 3150 60  0000 C CNN
+	1    15000 3150
+	0    1    1    0
+$EndComp
+Wire Wire Line
+	15100 3150 15000 3150
+$Comp
+L GND #PWR033
+U 1 1 54EA5095
+P 15000 4300
+F 0 "#PWR033" H 15000 4300 30  0001 C CNN
+F 1 "GND" H 15000 4230 30  0001 C CNN
+F 2 "" H 15000 4300 60  0000 C CNN
+F 3 "" H 15000 4300 60  0000 C CNN
+	1    15000 4300
+	0    1    1    0
+$EndComp
+Wire Wire Line
+	15100 4300 15000 4300
+Wire Wire Line
+	14400 5600 14400 4100
 $EndSCHEMATC

Commit message: +update
Parts:
- added L1: 47µH, symbol INDUCTOR_SMALL
- added P1, P2, P3: CONN_01X04, symbol CONN_01X04
Connections:
- net labels added: RGB-R
- wire segments 269 -> 279
Other:
- moved on the sheet: C10, C13, C14, C15, C16, C4, C5, C6, C7, C8, C9, Q1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
