File: kicad/tms9929/tms9929_sram.sch (KiCad schematic (older format))
At the start: 64 parts, among them P1 CONN_01X03, P4 Power, Q1 BC550, Q10 BC550, Q2 BC550, Q3 BC550, Q4 BC550, Q5 BC550, Q6 BC550, Q7 BC550, Q8 BC550, Q9 BC550, U1 TMS9929A, U10 7400, U2 74HCT04, U3 74HCT574, U4 74HCT574, U5 74HCT574, U6 HM62256BLFP-5SLT

Commit message: +update rev.1.1
Parts:
- added C10: 5-50pf, symbol CTRIM
Connections:
- wire segments 280 -> 282
Changed lines of the file:
@@
 LIBS:valves
 LIBS:tms99xx
-LIBS:tms9929_sram_snd-cache
 EELAYER 24 0
 EELAYER END
@@
 	1850 7450 2050 7450
 Wire Wire Line
-	3650 1350 3650 2150
+	3650 1050 3650 2150
 Wire Wire Line
 	13700 3550 13700 3650
@@
 Connection ~ 3400 6900
 Connection ~ 3650 6900
+$Comp
+L CTRIM C10
+U 1 1 5526BE0E
+P 3850 1050
+F 0 "C10" H 3980 970 50  0000 C CNN
+F 1 "5-50pf" H 4000 890 50  0000 C CNN
+F 2 "" H 3850 1050 60  0000 C CNN
+F 3 "" H 3850 1050 60  0000 C CNN
+	1    3850 1050
+	0    -1   -1   0
+$EndComp
+Wire Wire Line
+	4050 1050 4100 1050
+Wire Wire Line
+	4100 1050 4100 1350
 $EndSCHEMATC

Commit message: +Sync amplifier
Parts:
- added C?: 16µ/10V, symbol CP2
- added Q?: BC550, TO92, symbol BC550
- added R?: 470, symbol R
Connections:
- wire segments 282 -> 289
Changed lines of the file:
@@
 LIBS:valves
 LIBS:tms99xx
+LIBS:tms9929_sram-cache
 EELAYER 24 0
 EELAYER END
@@
 Wire Wire Line
 	4100 1050 4100 1350
+$Comp
+L BC550 Q?
+U 1 1 565D960A
+P 7950 8700
+F 0 "Q?" H 7950 8551 40  0000 R CNN
+F 1 "BC550" H 7950 8850 40  0000 R CNN
+F 2 "TO92" H 7850 8802 29  0000 C CNN
+F 3 "" H 7950 8700 60  0000 C CNN
+	1    7950 8700
+	1    0    0    -1
+$EndComp
+$Comp
+L R R?
+U 1 1 565D96FE
+P 7200 9050
+F 0 "R?" V 7280 9050 40  0000 C CNN
+F 1 "470" V 7207 9051 40  0000 C CNN
+F 2 "" V 7130 9050 30  0000 C CNN
+F 3 "" H 7200 9050 30  0000 C CNN
+	1    7200 9050
+	1    0    0    -1
+$EndComp
+$Comp
+L CP2 C?
+U 1 1 565D97C6
+P 7450 8700
+F 0 "C?" H 7450 8800 40  0000 L CNN
+F 1 "16µ/10V" H 7456 8615 40  0000 L CNN
+F 2 "" H 7488 8550 30  0000 C CNN
+F 3 "" H 7450 8700 60  0000 C CNN
+	1    7450 8700
+	0    -1   -1   0
+$EndComp
+Wire Wire Line
+	7200 8800 7200 8700
+Wire Wire Line
+	6750 8700 7250 8700
+Wire Wire Line
+	7650 8700 7750 8700
+$Comp
+L GND #PWR?
+U 1 1 565DC9B5
+P 7200 9400
+F 0 "#PWR?" H 7200 9400 30  0001 C CNN
+F 1 "GND" H 7200 9330 30  0001 C CNN
+F 2 "" H 7200 9400 60  0000 C CNN
+F 3 "" H 7200 9400 60  0000 C CNN
+	1    7200 9400
+	1    0    0    -1
+$EndComp
+Wire Wire Line
+	7200 9400 7200 9300
+$Comp
+L +12V #PWR?
+U 1 1 565DD636
+P 8050 8350
+F 0 "#PWR?" H 8050 8300 20  0001 C CNN
+F 1 "+12V" H 8050 8450 30  0000 C CNN
+F 2 "" H 8050 8350 60  0000 C CNN
+F 3 "" H 8050 8350 60  0000 C CNN
+	1    8050 8350
+	1    0    0    -1
+$EndComp
+Wire Wire Line
+	8050 8350 8050 8500
+Wire Wire Line
+	8050 8900 8050 9150
+Wire Wire Line
+	8050 9150 8350 9150
+Connection ~ 7200 8700
+Text Label 6800 8700 0    60   ~ 0
+Y
+Text Label 8250 9150 0    60   ~ 0
+SYNC
 $EndSCHEMATC

Commit message: +revision - before tag rev1.1
Parts:
- removed C?: 16µ/10V, symbol CP2
- removed Q?: BC550, TO92, symbol BC550
- removed R?: 470, symbol R
Connections:
- wire segments 289 -> 282
Changed lines of the file:
@@
 Wire Wire Line
 	4100 1050 4100 1350
-$Comp
-L BC550 Q?
-U 1 1 565D960A
-P 7950 8700
-F 0 "Q?" H 7950 8551 40  0000 R CNN
-F 1 "BC550" H 7950 8850 40  0000 R CNN
-F 2 "TO92" H 7850 8802 29  0000 C CNN
-F 3 "" H 7950 8700 60  0000 C CNN
-	1    7950 8700
-	1    0    0    -1
-$EndComp
-$Comp
-L R R?
-U 1 1 565D96FE
-P 7200 9050
-F 0 "R?" V 7280 9050 40  0000 C CNN
-F 1 "470" V 7207 9051 40  0000 C CNN
-F 2 "" V 7130 9050 30  0000 C CNN
-F 3 "" H 7200 9050 30  0000 C CNN
-	1    7200 9050
-	1    0    0    -1
-$EndComp
-$Comp
-L CP2 C?
-U 1 1 565D97C6
-P 7450 8700
-F 0 "C?" H 7450 8800 40  0000 L CNN
-F 1 "16µ/10V" H 7456 8615 40  0000 L CNN
-F 2 "" H 7488 8550 30  0000 C CNN
-F 3 "" H 7450 8700 60  0000 C CNN
-	1    7450 8700
-	0    -1   -1   0
-$EndComp
-Wire Wire Line
-	7200 8800 7200 8700
-Wire Wire Line
-	6750 8700 7250 8700
-Wire Wire Line
-	7650 8700 7750 8700
-$Comp
-L GND #PWR?
-U 1 1 565DC9B5
-P 7200 9400
-F 0 "#PWR?" H 7200 9400 30  0001 C CNN
-F 1 "GND" H 7200 9330 30  0001 C CNN
-F 2 "" H 7200 9400 60  0000 C CNN
-F 3 "" H 7200 9400 60  0000 C CNN
-	1    7200 9400
-	1    0    0    -1
-$EndComp
-Wire Wire Line
-	7200 9400 7200 9300
-$Comp
-L +12V #PWR?
-U 1 1 565DD636
-P 8050 8350
-F 0 "#PWR?" H 8050 8300 20  0001 C CNN
-F 1 "+12V" H 8050 8450 30  0000 C CNN
-F 2 "" H 8050 8350 60  0000 C CNN
-F 3 "" H 8050 8350 60  0000 C CNN
-	1    8050 8350
-	1    0    0    -1
-$EndComp
-Wire Wire Line
-	8050 8350 8050 8500
-Wire Wire Line
-	8050 8900 8050 9150
-Wire Wire Line
-	8050 9150 8350 9150
-Connection ~ 7200 8700
-Text Label 6800 8700 0    60   ~ 0
-Y
-Text Label 8250 9150 0    60   ~ 0
-SYNC
 $EndSCHEMATC

Commit message: +revision
Parts:
- C1, C2, C3, C4, C5, C6, C7, C8, C9: symbol C -> C-RESCUE-tms9929_sram
- C10: symbol CTRIM -> CTRIM-RESCUE-tms9929_sram
- R1, R10, R11, R12, R13, R14, R15, R16, R17, R18, R19, R2, R20, R21, R22, R23, R3, R4, R5, R6, R7, R8, R9: symbol R -> R-RESCUE-tms9929_sram
- RV1, RV2, RV3: symbol POT -> POT-RESCUE-tms9929_sram
- U6: symbol HM62256BLFP-5SLT -> HM62256BLFP-5SLT-RESCUE-tms9929_sram
Changed lines of the file:
@@
 EESchema Schematic File Version 2
+LIBS:tms9929_sram-rescue
 LIBS:power
 LIBS:device
@@
 LIBS:memory
 LIBS:xilinx
-LIBS:special
 LIBS:microcontrollers
 LIBS:dsp
@@
 LIBS:tms99xx
 LIBS:tms9929_sram-cache
-EELAYER 24 0
+EELAYER 25 0
 EELAYER END
 $Descr A3 16535 11693
@@
 $EndComp
 $Comp
-L GND #GND4
+L GND-RESCUE-tms9929_sram #GND4
 U 1 1 5419EC6F
 P 4900 5750
@@
 $EndComp
 $Comp
-L C C1
+L C-RESCUE-tms9929_sram C1
 U 1 1 5419ED2E
 P 3850 1350
@@
 $EndComp
 $Comp
-L C C2
+L C-RESCUE-tms9929_sram C2
 U 1 1 5419EDDB
 P 3850 1950
@@
 $EndComp
 $Comp
-L GND #GND3
+L GND-RESCUE-tms9929_sram #GND3
 U 1 1 5419F293
 P 3650 2150
@@
 $EndComp
 $Comp
-L R R5
+L R-RESCUE-tms9929_sram R5
 U 1 1 5419DE0B
 P 10800 7450
@@
 $EndComp
 $Comp
-L R R10
+L R-RESCUE-tms9929_sram R10
 U 1 1 5419DE3D
 P 11750 5550
@@
 $EndComp
 $Comp
-L R R7
+L R-RESCUE-tms9929_sram R7
 U 1 1 5419DEE9
 P 11450 4850
@@
 $EndComp
 $Comp
-L R R8
+L R-RESCUE-tms9929_sram R8
 U 1 1 5419DF21
 P 11450 5050
@@
 $EndComp
 $Comp
-L R R9
+L R-RESCUE-tms9929_sram R9
 U 1 1 5419DFBC
 P 11450 5250
@@
 $EndComp
 $Comp
-L R R12
+L R-RESCUE-tms9929_sram R12
 U 1 1 5419E03C
 P 11850 7150
@@
 $EndComp
 $Comp
-L R R11
+L R-RESCUE-tms9929_sram R11
 U 1 1 5419E069
 P 11850 7000
@@
 $EndComp
 $Comp
-L R R15
+L R-RESCUE-tms9929_sram R15
 U 1 1 5419E09B
 P 12150 7450
@@
 $EndComp
 $Comp
-L R R20
+L R-RESCUE-tms9929_sram R20
 U 1 1 5419E0D2
 P 12800 5550
@@
 $EndComp
 $Comp
-L R R2
+L R-RESCUE-tms9929_sram R2
 U 1 1 5419E2BF
 P 10400 7450
@@
 $EndComp
 $Comp
-L POT RV3
+L POT-RESCUE-tms9929_sram RV3
 U 1 1 541A1879
 P 12800 4300
@@
 $EndComp
 $Comp
-L R R17
+L R-RESCUE-tms9929_sram R17
 U 1 1 541A3EED
 P 12500 4600
@@
 $EndComp
 $Comp
-L R R21
+L R-RESCUE-tms9929_sram R21
 U 1 1 541A93AC
 P 13650 4600
@@
 $EndComp
 $Comp
-L R R22
+L R-RESCUE-tms9929_sram R22
 U 1 1 541A94BA
 P 13600 6450
@@
 $EndComp
 $Comp
-L POT RV1
+L POT-RESCUE-tms9929_sram RV1
 U 1 1 541A206E
 P 12150 6200
@@
 $EndComp
 $Comp
-L R R18
+L R-RESCUE-tms9929_sram R18
 U 1 1 541A4123
 P 12500 6500
@@
 $EndComp
 $Comp
-L GND #PWR24
+L GND-RESCUE-tms9929_sram #PWR24
 U 1 1 541B699C
 P 12150 7750
@@
 $EndComp
 $Comp
-L GND #PWR21
+L GND-RESCUE-tms9929_sram #PWR21
 U 1 1 541B69F6
 P 10800 7750
@@
 $EndComp
 $Comp
-L GND #PWR16
+L GND-RESCUE-tms9929_sram #PWR16
 U 1 1 541B6A4E
 P 10400 7750
@@
 $EndComp
 $Comp
-L GND #PWR27
+L GND-RESCUE-tms9929_sram #PWR27
 U 1 1 541B6AC2
 P 12800 7750
@@
 $EndComp
 $Comp
-L R R6
+L R-RESCUE-tms9929_sram R6
 U 1 1 541BDEA5
 P 10800 9350
@@
 $EndComp
 $Comp
-L R R14
+L R-RESCUE-tms9929_sram R14
 U 1 1 541BDEAB
 P 11850 9050
@@
 $EndComp
 $Comp
-L R R13
+L R-RESCUE-tms9929_sram R13
 U 1 1 541BDEB1
 P 11850 8900
@@
 $EndComp
 $Comp
-L R R16
+L R-RESCUE-tms9929_sram R16
 U 1 1 541BDEB7
 P 12150 9350
@@
 $EndComp
 $Comp
-L R R3
+L R-RESCUE-tms9929_sram R3
 U 1 1 541BDEBD
 P 10400 9350
@@
 $EndComp
 $Comp
-L R R23
+L R-RESCUE-tms9929_sram R23
 U 1 1 541BDEC3
 P 13600 8350
@@
 $EndComp
 $Comp
-L POT RV2
+L POT-RESCUE-tms9929_sram RV2
 U 1 1 541BDECF
 P 12150 8100
@@
 $EndComp
 $Comp
-L R R19
+L R-RESCUE-tms9929_sram R19
 U 1 1 541BDEE3
 P 12500 8400
@@
 $EndComp
 $Comp
-L GND #PWR25
+L GND-RESCUE-tms9929_sram #PWR25
 U 1 1 541BDEFB
 P 12150 9650
@@
 $EndComp
 $Comp
-L GND #PWR22
+L GND-RESCUE-tms9929_sram #PWR22
 U 1 1 541BDF01
 P 10800 9650
@@
 $EndComp
 $Comp
-L GND #PWR17
+L GND-RESCUE-tms9929_sram #PWR17
 U 1 1 541BDF07
 P 10400 9650
@@
 $EndComp
 $Comp
-L GND #PWR28
+L GND-RESCUE-tms9929_sram #PWR28
 U 1 1 541BDF0D
 P 12800 9650
@@
 $EndComp
 $Comp
-L GND #PWR14
+L GND-RESCUE-tms9929_sram #PWR14
 U 1 1 541BEEF6
 P 10050 9650
@@
 $EndComp
 $Comp
-L R R4
+L R-RESCUE-tms9929_sram R4
 U 1 1 541BF5C0
 P 10800 5550
@@
 $EndComp
 $Comp
-L R R1
+L R-RESCUE-tms9929_sram R1
 U 1 1 541BF5C6
 P 10400 5550
@@
 $EndComp
 $Comp
-L GND #PWR20
+L GND-RESCUE-tms9929_sram #PWR20
 U 1 1 541BF5D2
 P 10800 5850
@@
 $EndComp
 $Comp
-L GND #PWR15
+L GND-RESCUE-tms9929_sram #PWR15
 U 1 1 541BF5D8
 P 10400 5850
@@
 $EndComp
 $Comp
-L GND #PWR23
+L GND-RESCUE-tms9929_sram #PWR23
 U 1 1 541BF8B0
 P 11750 5850
@@
 $EndComp
 $Comp
-L GND #PWR26
+L GND-RESCUE-tms9929_sram #PWR26
 U 1 1 541BF8EA
 P 12800 5850
@@
 V_RW
 $Comp
-L C C4
+L C-RESCUE-tms9929_sram C4
 U 1 1 542329DF
 P 2400 6700
@@
 $EndComp
 $Comp
-L C C5
+L C-RESCUE-tms9929_sram C5
 U 1 1 54232CDC
 P 2650 6700
@@
 $EndComp
 $Comp
-L C C6
+L C-RESCUE-tms9929_sram C6
 U 1 1 54232D35
 P 2900 6700
@@
 $EndComp
 $Comp
-L C C7
+L C-RESCUE-tms9929_sram C7
 U 1 1 54232D87
 P 3150 6700
@@
 $EndComp
 $Comp
-L GND #PWR2
+L GND-RESCUE-tms9929_sram #PWR2
 U 1 1 5423480D
 P 1750 6900
@@
 $EndComp
 $Comp
-L HM62256BLFP-5SLT U6
+L HM62256BLFP-5SLT-RESCUE-tms9929_sram U6
 U 1 1 544A67F3
 P 10750 1550
@@
 RGB-B
 $Comp
-L GND #PWR31
+L GND-RESCUE-tms9929_sram #PWR31
 U 1 1 54B05606
 P 14900 4700
@@
 $EndComp
 $Comp
-L GND #GND2
+L GND-RESCUE-tms9929_sram #GND2
 U 1 1 54BF1560
 P 3100 4850
@@
 $EndComp
 $Comp
-L GND #PWR12
+L GND-RESCUE-tms9929_sram #PWR12
 U 1 1 54BF5ED0
 P 8700 4700
@@
 $EndComp
 $Comp
-L GND #PWR10
+L GND-RESCUE-tms9929_sram #PWR10
 U 1 1 54BF70EA
 P 8700 3300
@@
 $EndComp
 $Comp
-L GND #PWR8
+L GND-RESCUE-tms9929_sram #PWR8
 U 1 1 54BF8680
 P 8700 1900
@@
 $EndComp
 $Comp
-L GND #PWR19
+L GND-RESCUE-tms9929_sram #PWR19
 U 1 1 54BF8AD3
 P 10750 2350
@@
 $EndComp
 $Comp
-L GND #PWR30
+L GND-RESCUE-tms9929_sram #PWR30
 U 1 1 54EA4F07
 P 14900 4400
@@
 $EndComp
 $Comp
-L GND #PWR29
+L GND-RESCUE-tms9929_sram #PWR29
 U 1 1 54EA4FCE
 P 14900 4100
@@
 $EndComp
 $Comp
-L GND #PWR32
+L GND-RESCUE-tms9929_sram #PWR32
 U 1 1 54EA5095
 P 14900 5000
@@
 $EndComp
 $Comp
-L GND #GND1
+L GND-RESCUE-tms9929_sram #GND1
 U 1 1 54FF5A12
 P 1800 7650
@@
 NoConn ~ 4350 4050
 $Comp
-L C C3
+L C-RESCUE-tms9929_sram C3
 U 1 1 55224E4F
 P 3400 6700
@@
 $EndComp
 $Comp
-L C C8
+L C-RESCUE-tms9929_sram C8
 U 1 1 55224EB6
 P 3650 6700
@@
 $EndComp
 $Comp
-L C C9
+L C-RESCUE-tms9929_sram C9
 U 1 1 55224F16
 P 3900 6700
@@
 Connection ~ 3650 6900
 $Comp
-L CTRIM C10
+L CTRIM-RESCUE-tms9929_sram C10
 U 1 1 5526BE0E
 P 3850 1050
