File: kicad/cpu_mem_uart/50pin_connector.sch (KiCad schematic (older format))
At the start: 0 parts

Commit message: crap
Parts:
- added P5: CONN_02X25, Pin_Headers:Pin_Header_Angled_2x25, symbol CONN_02X25
Connections:
- new net /CS_IO0: P5.21 (P21)
- new net /CS_IO1: P5.20 (P20)
- new net /CS_IO2: P5.19 (P19)
- new net /CS_UART: P5.23 (P23)
- new net /CS_VDP: P5.24 (P24)
- new net /CS_VIA: P5.22 (P22)
- new net /IRQ: P5.4 (P4)
- new net /NMI: P5.3 (P3)
- new net /OE: P5.33 (P33)
- new net /RESET: P5.2 (P2)
- new net /RW: P5.15 (P15)
- new net /WE: P5.34 (P34)
- new net A0: P5.30 (P30)
- new net A1: P5.29 (P29)
- new net A2: P5.28 (P28)
- new net A3: P5.27 (P27)
- new net A4: P5.26 (P26)
- new net A5: P5.25 (P25)
- new net D0: P5.13 (P13)
- new net D1: P5.12 (P12)
- new net D2: P5.11 (P11)
- new net D3: P5.10 (P10)
- new net D4: P5.9 (P9)
- new net D5: P5.8 (P8)
- new net D6: P5.7 (P7)
- new net D7: P5.6 (P6)
- new net GND: P5.31 (P31), P5.32 (P32), P5.35 (P35), P5.37 (P37), P5.47 (P47), P5.48 (P48), P5.49 (P49), P5.50 (P50)
- new net PHI2: P5.36 (P36)
- new net RDY: P5.17 (P17)
- new net RESET_TRIG: P5.38 (P38)
- new net VCC: P5.1 (P1), P5.43 (P43), P5.44 (P44), P5.45 (P45), P5.46 (P46)
- no-connect marks 0 -> 8
