File: kicad/cpu_mem_uart/cpu_mem_uart.kicad_pcb (KiCad board)
At the start: 2 copper layers, 160 x 100.3 mm, 66 parts, among them P1 CONN_02X04, P2 CONN_01X08, P3 CONN_01X03, P4 CONN_02X02, P5 CONN_02X25, P6 POWER, SW1 SW_PUSH, U1 W65C02SP, U11 74LS273, U12 74LS244, U2 LM555N, U3 74HCT00, U4 74LS393, U5 GAL22V10, U6 28C256, U7 HM62256BLP-7, U8 HM62256BLP-7, U9 74LS139, X1 OSC

Commit message: crap
Parts:
- added C18: 1µF, Capacitors_ThroughHole:C_Radial_D5_L6_P2.5, F.Cu at (142.2, 156.1)
- added C19, C20, C21: CP2, Capacitors_ThroughHole:C_Radial_D5_L6_P2.5, F.Cu at (142.2, 156.1)
- added C22: CP2, Capacitors_ThroughHole:C_Radial_D5_L11_P2.5, F.Cu at (142.2, 156.1)
- added J1: DB9, w_conn_d-sub:DB_9M, F.Cu at (73.7, 91.4)
- added R18: 4k7, Discret:R3, F.Cu at (142.2, 156.1)
- added R19: 3k3, Discret:R3, F.Cu at (142.2, 156.1)
- added U10: 74LS06, Housings_DIP:DIP-14_W7.62mm_LongPads, F.Cu at (121.9, 162.6)
- added U13: 16550, Housings_DIP:DIP-40_W15.24mm_LongPads, F.Cu at (154.9, 67.3)
- added U14: GAL16V8, Housings_DIP:DIP-20_W7.62mm_LongPads, F.Cu at (125.7, 78.7)
- added U15: MAX232, Housings_DIP:DIP-16_W7.62mm_LongPads, F.Cu at (126.0, 187.6)
- added X2: OSC, Oscillators:KXO-200_LargePads, F.Cu at (104.1, 185.4)
- SW1: footprint Discret:PUSH_BUTT_SHAPE1 -> Buttons_Switches_ThroughHole:SW_PUSH_SMALL
- U2: footprint Sockets_DIP:DIP-8__300_ELL -> Housings_DIP:DIP-8_W7.62mm_LongPads
- U3, U4: footprint Sockets_DIP:DIP-14__300_ELL -> Housings_DIP:DIP-14_W7.62mm_LongPads
- U5: footprint Sockets_DIP:DIP-24__300_ELL -> Housings_DIP:DIP-24_W7.62mm_LongPads
- U9: footprint Sockets_DIP:DIP-16__300_ELL -> Housings_DIP:DIP-16_W7.62mm_LongPads
- moved D4 72.9 mm to (109.2, 157.5)
- moved D6 67.3 mm to (106.7, 162.6)
- moved D5 58.8 mm to (99.1, 152.4)
- moved D7 55.3 mm to (96.5, 160.0)
- moved P2 53.0 mm to (53.3, 139.7)
- moved R17 52.1 mm to (45.7, 149.9)
- moved R15 51.9 mm to (45.7, 144.8)
- moved R16 51.9 mm to (45.7, 147.3)
- moved R14 51.8 mm to (45.7, 142.2)
- moved R13 51.8 mm to (45.7, 139.7)
- moved R12 51.7 mm to (45.7, 137.2)
- moved R10 51.6 mm to (45.7, 132.1)
- moved R11 51.6 mm to (45.7, 134.6)
- moved D8 47.1 mm to (88.9, 160.0)
- moved P1 41.8 mm to (164.8, 25.5)
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Connections:
- P5 pad 14: (no net) -> Net-(P5-Pad14)
- P5 pad 16: (no net) -> Net-(P5-Pad16)
- P5 pad 18: (no net) -> Net-(P5-Pad18)
- P5 pad 39: (no net) -> Net-(P5-Pad39)
- P5 pad 40: (no net) -> Net-(P5-Pad40)
- P5 pad 41: (no net) -> Net-(P5-Pad41)
- P5 pad 42: (no net) -> Net-(P5-Pad42)
- P5 pad 5: (no net) -> Net-(P5-Pad5)
- P6 pad 4: (no net) -> Net-(P6-Pad4)
- U1 pad 3: (no net) -> Net-(U1-Pad3)
- U1 pad 35: (no net) -> Net-(U1-Pad35)
- U1 pad 38: (no net) -> Net-(U1-Pad38)
- U1 pad 5: (no net) -> Net-(U1-Pad5)
- U1 pad 7: (no net) -> Net-(U1-Pad7)
- U4 pad 10: (no net) -> Net-(U4-Pad10)
- U4 pad 11: (no net) -> Net-(U4-Pad11)
- U4 pad 8: (no net) -> Net-(U4-Pad8)
- U4 pad 9: (no net) -> Net-(U4-Pad9)
- U9 pad 10: (no net) -> Net-(U11-Pad11)
- U9 pad 11: (no net) -> Net-(U9-Pad11)
- U9 pad 12: Net-(U11-Pad11) -> Net-(U9-Pad12)
- U9 pad 7: (no net) -> /decoder//CS_IO3
- X1 pad 1: (no net) -> Net-(X1-Pad1)
Routing:
- net /Connector/RESET_TRIG: track 239.7 -> 52.4 mm
- net /RESET: track 168.3 -> 2.46 mm
- net VCC: track 425.6 -> 297.0 mm, vias 5 -> 3
- net GND: track 566.4 -> 452.7 mm
- net /WE: track 139.2 -> 235.4 mm, vias 0 -> 2
- net /CS_IO0: track 93.2 -> 0.00 mm, vias 1 -> 0
- net /CS_IO2: track 87.4 -> 0.00 mm, vias 1 -> 0
- net /RW: track 157.3 -> 87.4 mm, vias 1 -> 0
- net /decoder/A13: track 136.1 -> 68.5 mm, vias 1 -> 0
- net Net-(U12-Pad1): track 76.3 -> 9.03 mm
- net Net-(U11-Pad11): track 67.4 -> 0.36 mm
- net /decoder//ROMOFF: track 80.1 -> 15.3 mm, vias 1 -> 0
- net /decoder/BANK2: track 78.1 -> 14.9 mm, vias 1 -> 0
- net /decoder/BANK1: track 75.6 -> 14.6 mm, vias 2 -> 0
- net PHI2: track 164.8 -> 104.2 mm
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- removed copper zone on F.Cu, net GND
