File: kicad/cpu_mem_uart/cpu_mem_uart.sch (KiCad schematic (older format))
At the start: 36 parts, among them P1 CONN_02X04, P3 CONN_01X03, P4 CONN_02X02, P6 POWER, SW1 SW_PUSH, U1 W65C02SP, U2 LM555N, U3 74HCT00, U4 74LS393, U6 28C256, U7 HM62256BLP-7, U8 HM62256BLP-7, X1 OSC

Commit message: crap
Parts:
- C16: footprint Capacitors_Elko_ThroughHole:Elko_vert_11.2x7.5mm_RM2.5 -> Capacitors_ThroughHole:C_Radial_D5_L11_P2.5
- C4: footprint Capacitors_Elko_ThroughHole:Elko_vert_DM5_RM2-5 -> Capacitors_ThroughHole:C_Radial_D5_L6_P2.5
- SW1: footprint Discret:PUSH_BUTT_SHAPE1 -> Buttons_Switches_ThroughHole:SW_PUSH_SMALL
- U1: footprint Sockets_DIP:DIP-40__600_ELL -> Housings_DIP:DIP-40_W15.24mm_LongPads
- U2: footprint Sockets_DIP:DIP-8__300_ELL -> Housings_DIP:DIP-8_W7.62mm_LongPads
- U3, U4: footprint Sockets_DIP:DIP-14__300_ELL -> Housings_DIP:DIP-14_W7.62mm_LongPads
- U6, U7, U8: footprint Sockets_DIP:DIP-28__600_ELL -> Housings_DIP:DIP-28_W15.24mm_LongPads
- X1: footprint Oscillator-Modules:OSCILLATOR_KXO-200_LargePads -> Oscillators:KXO-200_LargePads
Changed lines of the file:
@@
 $Descr A4 11693 8268
 encoding utf-8
-Sheet 1 3
+Sheet 1 4
 Title ""
 Date ""
@@
 F 0 "U1" H 2000 2550 50  0000 L BNN
 F 1 "W65C02SP" H 1600 950 50  0000 L BNN
-F 2 "Sockets_DIP:DIP-40__600_ELL" H 2000 2700 50  0001 C CNN
+F 2 "Housings_DIP:DIP-40_W15.24mm_LongPads" H 2000 2700 50  0001 C CNN
 F 3 "" H 2000 2550 60  0000 C CNN
 	1    2000 2550
@@
 F 0 "U2" H 2250 6800 70  0000 C CNN
 F 1 "LM555N" H 2250 6600 70  0000 C CNN
-F 2 "Sockets_DIP:DIP-8__300_ELL" H 2250 6700 60  0001 C CNN
+F 2 "Housings_DIP:DIP-8_W7.62mm_LongPads" H 2250 6700 60  0001 C CNN
 F 3 "" H 2250 6700 60  0000 C CNN
 	1    2250 6700
@@
 F 0 "C4" H 3000 7250 40  0000 L CNN
 F 1 "1µ" H 3006 7065 40  0000 L CNN
-F 2 "Capacitors_Elko_ThroughHole:Elko_vert_DM5_RM2-5" H 3038 7000 30  0001 C CNN
+F 2 "Capacitors_ThroughHole:C_Radial_D5_L6_P2.5" H 3038 7000 30  0001 C CNN
 F 3 "" H 3000 7150 60  0000 C CNN
 	1    3000 7150
@@
 F 0 "U3" H 3850 6450 60  0000 C CNN
 F 1 "74HCT00" H 3850 6300 60  0000 C CNN
-F 2 "Sockets_DIP:DIP-14__300_ELL" H 3850 6400 60  0001 C CNN
+F 2 "Housings_DIP:DIP-14_W7.62mm_LongPads" H 3850 6400 60  0001 C CNN
 F 3 "" H 3850 6400 60  0000 C CNN
 	4    3850 6400
@@
 F 0 "U4" H 3450 5150 60  0000 C CNN
 F 1 "74LS393" H 3500 4650 60  0000 C CNN
-F 2 "Sockets_DIP:DIP-14__300_ELL" H 3300 4900 60  0001 C CNN
+F 2 "Housings_DIP:DIP-14_W7.62mm_LongPads" H 3300 4900 60  0001 C CNN
 F 3 "" H 3300 4900 60  0000 C CNN
 	1    3300 4900
@@
 F 0 "U3" H 8600 6250 60  0000 C CNN
 F 1 "74HCT00" H 8600 6100 60  0000 C CNN
-F 2 "Sockets_DIP:DIP-14__300_ELL" H 8600 6200 60  0001 C CNN
+F 2 "Housings_DIP:DIP-14_W7.62mm_LongPads" H 8600 6200 60  0001 C CNN
 F 3 "" H 8600 6200 60  0000 C CNN
 	1    8600 6200
@@
 F 0 "U3" H 9900 5600 60  0000 C CNN
 F 1 "74HCT00" H 9900 5450 60  0000 C CNN
-F 2 "Sockets_DIP:DIP-14__300_ELL" H 9900 5550 60  0001 C CNN
+F 2 "Housings_DIP:DIP-14_W7.62mm_LongPads" H 9900 5550 60  0001 C CNN
 F 3 "" H 9900 5550 60  0000 C CNN
 	2    9900 5550
@@
 F 0 "U3" H 9900 6150 60  0000 C CNN
 F 1 "74HCT00" H 9900 6000 60  0000 C CNN
-F 2 "Sockets_DIP:DIP-14__300_ELL" H 9900 6100 60  0001 C CNN
+F 2 "Housings_DIP:DIP-14_W7.62mm_LongPads" H 9900 6100 60  0001 C CNN
 F 3 "" H 9900 6100 60  0000 C CNN
 	3    9900 6100
@@
 F 0 "U7" H 6350 5150 50  0000 C CNN
 F 1 "HM62256BLP-7" H 7050 3450 50  0000 C CNN
-F 2 "Sockets_DIP:DIP-28__600_ELL" H 6650 4250 30  0000 C CIN
+F 2 "Housings_DIP:DIP-28_W15.24mm_LongPads" H 6650 4250 30  0000 C CIN
 F 3 "" H 6650 4250 60  0000 C CNN
 	1    6650 4250
@@
 F 0 "SW1" H 3350 7260 50  0000 C CNN
 F 1 "SW_PUSH" H 3200 7070 50  0000 C CNN
-F 2 "Discret:PUSH_BUTT_SHAPE1" H 3200 7150 60  0001 C CNN
+F 2 "Buttons_Switches_ThroughHole:SW_PUSH_SMALL" H 3200 7150 60  0001 C CNN
 F 3 "" H 3200 7150 60  0000 C CNN
 	1    3200 7150
@@
 F 0 "U8" H 8450 5150 50  0000 C CNN
 F 1 "HM62256BLP-7" H 9150 3450 50  0000 C CNN
-F 2 "Sockets_DIP:DIP-28__600_ELL" H 8750 4250 30  0000 C CIN
+F 2 "Housings_DIP:DIP-28_W15.24mm_LongPads" H 8750 4250 30  0000 C CIN
 F 3 "" H 8750 4250 60  0000 C CNN
 	1    8750 4250
@@
 F 0 "X1" H 1550 5200 70  0000 C CNN
 F 1 "OSC" H 1550 4900 70  0000 C CNN
-F 2 "Oscillator-Modules:OSCILLATOR_KXO-200_LargePads" H 1550 4900 60  0001 C CNN
+F 2 "Oscillators:KXO-200_LargePads" H 1550 4900 60  0001 C CNN
 F 3 "" H 1550 4900 60  0000 C CNN
 	1    1550 4900
@@
 F 0 "U6" H 8300 2950 70  0000 C CNN
 F 1 "28C256" H 8400 950 70  0000 C CNN
-F 2 "Sockets_DIP:DIP-28__600_ELL" H 8100 1950 60  0001 C CNN
+F 2 "Housings_DIP:DIP-28_W15.24mm_LongPads" H 8100 1950 60  0001 C CNN
 F 3 "" H 8100 1950 60  0000 C CNN
 	1    8100 1950
@@
 	1    0    0    -1
 $EndComp
-$Sheet
-S 10050 600  650  2950
-U 54206EE0
-F0 "Connector" 60
-F1 "50pin_connector.sch" 60
-F2 "A0" I L 10050 1800 60
-F3 "A1" I L 10050 1900 60
-F4 "A2" I L 10050 2000 60
-F5 "A3" I L 10050 2100 60
-F6 "A4" I L 10050 2200 60
-F7 "D0" I L 10050 2800 60
-F8 "D1" I L 10050 2900 60
-F9 "D2" I L 10050 3000 60
-F10 "D3" I L 10050 3100 60
-F11 "D4" I L 10050 3200 60
-F12 "D5" I L 10050 3300 60
-F13 "D6" I L 10050 3400 60
-F14 "D7" I L 10050 3500 60
-F15 "A5" I L 10050 2300 60
-F16 "RESET_TRIG" I L 10050 1250 60
-$EndSheet
 $Sheet
 S 3550 700  1300 2550
@@
 F 0 "C16" H 6650 7300 40  0000 L CNN
 F 1 "CP2" H 6656 7115 40  0000 L CNN
-F 2 "Capacitors_Elko_ThroughHole:Elko_vert_11.2x7.5mm_RM2.5" H 6688 7050 30  0001 C CNN
+F 2 "Capacitors_ThroughHole:C_Radial_D5_L11_P2.5" H 6688 7050 30  0001 C CNN
 F 3 "" H 6650 7200 60  0000 C CNN
 	1    6650 7200
@@
 F 0 "U4" H 5700 5950 60  0000 C CNN
 F 1 "74LS393" H 5750 5450 60  0000 C CNN
-F 2 "Sockets_DIP:DIP-14__300_ELL" H 5550 5700 60  0001 C CNN
+F 2 "Housings_DIP:DIP-14_W7.62mm_LongPads" H 5550 5700 60  0001 C CNN
 F 3 "" H 5550 5700 60  0000 C CNN
 	2    5550 5700
@@
 NoConn ~ 6250 5850
 Wire Wire Line
-	10050 1250 9550 1250
-Text Label 9550 1250 0    60   ~ 0
+	10050 1250 9500 700
+Text Label 9500 700  0    60   ~ 0
 RESET_TRIG
 Text Label 500  6500 0    60   ~ 0
@@
 Wire Wire Line
 	3350 3100 3550 3100
+$Sheet
+S 10550 3850 600  1350
+U 56AC06C6
+F0 "UART" 60
+F1 "uart.sch" 60
+F2 "D0" B L 10550 3950 60
+F3 "D1" B L 10550 4050 60
+F4 "D2" B L 10550 4150 60
+F5 "D3" B L 10550 4250 60
+F6 "D4" B L 10550 4350 60
+F7 "D5" B L 10550 4450 60
+F8 "D6" B L 10550 4550 60
+F9 "D7" B L 10550 4650 60
+F10 "A0" I L 10550 4950 60
+F11 "A1" I L 10550 5050 60
+F12 "A2" I L 10550 5150 60
+$EndSheet
+$Sheet
+S 10050 600  650  2950
+U 54206EE0
+F0 "Connector" 60
+F1 "50pin_connector.sch" 60
+F2 "A0" I L 10050 1800 60
+F3 "A1" I L 10050 1900 60
+F4 "A2" I L 10050 2000 60
+F5 "A3" I L 10050 2100 60
+F6 "A4" I L 10050 2200 60
+F7 "D0" I L 10050 2800 60
+F8 "D1" I L 10050 2900 60
+F9 "D2" I L 10050 3000 60
+F10 "D3" I L 10050 3100 60
+F11 "D4" I L 10050 3200 60
+F12 "D5" I L 10050 3300 60
+F13 "D6" I L 10050 3400 60
+F14 "D7" I L 10050 3500 60
+F15 "A5" I L 10050 2300 60
+F16 "RESET_TRIG" I L 10050 1250 60
+$EndSheet
+Entry Wire Line
+	10400 3950 10300 3850
+Entry Wire Line
+	10400 4050 10300 3950
+Entry Wire Line
+	10400 4150 10300 4050
+Entry Wire Line
+	10400 4250 10300 4150
+Entry Wire Line
+	10400 4350 10300 4250
+Entry Wire Line
+	10400 4450 10300 4350
+Entry Wire Line
+	10400 4550 10300 4450
+Entry Wire Line
+	10400 4650 10300 4550
+Text Label 10300 3800 2    60   ~ 0
+D
+Text Label 10400 3950 0    60   ~ 0
+D0
+Text Label 10400 4050 0    60   ~ 0
+D1
+Text Label 10400 4150 0    60   ~ 0
+D2
+Text Label 10400 4250 0    60   ~ 0
+D3
+Text Label 10400 4350 0    60   ~ 0
+D4
+Text Label 10400 4450 0    60   ~ 0
+D5
+Text Label 10400 4550 0    60   ~ 0
+D6
+Text Label 10400 4650 0    60   ~ 0
+D7
+Wire Bus Line
+	10300 3750 10300 4550
+Wire Wire Line
+	10400 3950 10550 3950
+Wire Wire Line
+	10550 4050 10400 4050
+Wire Wire Line
+	10400 4150 10550 4150
+Wire Wire Line
+	10550 4250 10400 4250
+Wire Wire Line
+	10400 4350 10550 4350
+Wire Wire Line
+	10550 4450 10400 4450
+Wire Wire Line
+	10400 4550 10550 4550
+Wire Wire Line
+	10550 4650 10400 4650
+Entry Wire Line
+	10350 4850 10450 4950
+Text Label 10200 4800 0    60   ~ 0
+A[0..15]
+Text Label 10450 4950 0    60   ~ 0
+A0
+Entry Wire Line
+	10350 4950 10450 5050
+Entry Wire Line
+	10350 5050 10450 5150
+Text Label 10450 5050 0    60   ~ 0
+A1
+Text Label 10450 5150 0    60   ~ 0
+A2
+Wire Bus Line
+	10350 4850 10350 5050
+Wire Wire Line
+	10450 4950 10550 4950
+Wire Wire Line
+	10450 5050 10550 5050
+Wire Wire Line
+	10450 5150 10550 5150
 $EndSCHEMATC
