File: kicad/cpu_mem_uart/decoder.sch (KiCad schematic (older format))
At the start: 26 parts, among them P2 CONN_01X08, U11 74LS273, U12 74LS244, U14 GAL16V8, U5 GAL22V10, U9 74LS139

Commit message: crap
Parts:
- U11, U12: footprint Sockets_DIP:DIP-20__300_ELL -> Housings_DIP:DIP-20_W7.62mm_LongPads
- U14: footprint (none) -> Housings_DIP:DIP-20_W7.62mm_LongPads
- U5: footprint Sockets_DIP:DIP-24__300_ELL -> Housings_DIP:DIP-24_W7.62mm_LongPads
- U9: footprint Sockets_DIP:DIP-16__300_ELL -> Housings_DIP:DIP-16_W7.62mm_LongPads
Connections:
- net /CS_ROM: now also U14.5 (I5); no longer U14.2 (I2)
- net /CS_VDP: now also U14.2 (I2); no longer U14.5 (I5)
Changed lines of the file:
@@
 $Descr A4 11693 8268
 encoding utf-8
-Sheet 3 3
+Sheet 2 4
 Title ""
 Date ""
@@
 F 0 "U5" H 1900 6800 60  0000 C CNN
 F 1 "GAL22V10" H 1900 5300 60  0000 C CNN
-F 2 "Sockets_DIP:DIP-24__300_ELL" H 1850 6050 60  0001 C CNN
+F 2 "Housings_DIP:DIP-24_W7.62mm_LongPads" H 1850 6050 60  0001 C CNN
 F 3 "" H 1850 6050 60  0000 C CNN
 	1    1850 6050
@@
 F 0 "U9" H 1700 4450 60  0000 C CNN
 F 1 "74LS139" H 1700 4250 60  0000 C CNN
-F 2 "Sockets_DIP:DIP-16__300_ELL" H 1700 4350 60  0001 C CNN
+F 2 "Housings_DIP:DIP-16_W7.62mm_LongPads" H 1700 4350 60  0001 C CNN
 F 3 "" H 1700 4350 60  0000 C CNN
 	1    1700 4350
@@
 F 0 "U9" H 4550 5600 60  0000 C CNN
 F 1 "74LS139" H 4550 5400 60  0000 C CNN
-F 2 "Sockets_DIP:DIP-16__300_ELL" H 4550 5500 60  0001 C CNN
+F 2 "Housings_DIP:DIP-16_W7.62mm_LongPads" H 4550 5500 60  0001 C CNN
 F 3 "" H 4550 5500 60  0000 C CNN
 	2    4550 5500
@@
 F 0 "U11" H 7050 5050 60  0000 C CNN
 F 1 "74LS273" H 7050 4850 60  0000 C CNN
-F 2 "Sockets_DIP:DIP-20__300_ELL" H 7050 5200 60  0001 C CNN
+F 2 "Housings_DIP:DIP-20_W7.62mm_LongPads" H 7050 5200 60  0001 C CNN
 F 3 "" H 7050 5200 60  0000 C CNN
 	1    7050 5200
@@
 F 0 "U12" H 9500 5000 60  0000 C CNN
 F 1 "74LS244" H 9550 4800 60  0000 C CNN
-F 2 "Sockets_DIP:DIP-20__300_ELL" H 9450 5200 60  0001 C CNN
+F 2 "Housings_DIP:DIP-20_W7.62mm_LongPads" H 9450 5200 60  0001 C CNN
 F 3 "" H 9450 5200 60  0000 C CNN
 	1    9450 5200
@@
 F 0 "U14" H 4050 7750 50  0000 L CNN
 F 1 "GAL16V8" H 4450 7750 50  0000 L CNN
-F 2 "" H 4400 7100 50  0001 C CNN
+F 2 "Housings_DIP:DIP-20_W7.62mm_LongPads" H 4400 7100 50  0001 C CNN
 F 3 "" H 4400 7100 50  0000 C CNN
 	1    4400 7100
@@
 	3600 6600 3900 6600
 Wire Wire Line
-	2800 6700 3900 6700
-Wire Wire Line
-	2750 6800 3900 6800
-Wire Wire Line
-	2700 6900 3900 6900
-Wire Wire Line
-	2800 6700 2800 6100
-Connection ~ 2800 6100
-Wire Wire Line
-	2750 6800 2750 5700
-Connection ~ 2750 5700
-Wire Wire Line
-	2700 6900 2700 5800
-Connection ~ 2700 5800
-Wire Wire Line
-	3900 7000 2650 7000
-Wire Wire Line
-	2650 7000 2650 5600
-Connection ~ 2650 5600
-Wire Wire Line
-	3900 7100 3100 7100
+	2700 6800 2700 5700
+Connection ~ 2700 5700
+Wire Wire Line
+	2650 6900 2650 5800
+Connection ~ 2650 5800
+Wire Wire Line
+	2750 6700 2750 5600
+Connection ~ 2750 5600
 Wire Wire Line
 	2550 4050 3250 4050
@@
 $EndComp
 Wire Wire Line
-	3700 7650 3700 7400
+	3700 7400 3700 7650
 Wire Wire Line
 	3700 7400 3900 7400
@@
 	1    0    0    -1
 $EndComp
+Wire Wire Line
+	2750 6700 3900 6700
+Wire Wire Line
+	2700 6800 3900 6800
+Wire Wire Line
+	2650 6900 3900 6900
+Wire Wire Line
+	3900 7000 2600 7000
+Wire Wire Line
+	2600 7000 2600 6100
+Connection ~ 2600 6100
+Wire Wire Line
+	3100 7100 3900 7100
 $EndSCHEMATC
