File: kicad/V9958_OPL2/v9958.sch (KiCad schematic (older format))
At the start: 51 parts, among them P1 RED, P2 GREEN, P3 BLUE, P4 SYNC/C, U1 74LS139, U2 V9958, U3 DRAM_64KX4, U4 DRAM_64KX4, U5 DRAM_64KX4, U6 DRAM_64KX4, U7 cxa2075M, U8 YM3812, U9 Y3014B, X1 OSC, X2 S-VIDEO, Y1 21,443Mhz

Commit message: analog audio section
Parts:
- removed U9: Y3014B, Housings_DIP:DIP-8_W7.62mm_LongPads, symbol Y3014B
Other:
- moved on the sheet: X1, X2
Changed lines of the file:
@@
 $Descr A4 11693 8268
 encoding utf-8
-Sheet 1 2
+Sheet 1 3
 Title ""
 Date ""
@@
 L OSC X1
 U 1 1 5A874348
-P 6200 5050
-F 0 "X1" H 6200 5350 70  0000 C CNN
-F 1 "OSC" H 6200 5050 70  0000 C CNN
-F 2 "Oscillators:KXO-200_LargePads" H 6200 5050 60  0001 C CNN
-F 3 "" H 6200 5050 60  0000 C CNN
-	1    6200 5050
+P 6400 5050
+F 0 "X1" H 6400 5350 70  0000 C CNN
+F 1 "OSC" H 6400 5050 70  0000 C CNN
+F 2 "Oscillators:KXO-200_LargePads" H 6400 5050 60  0001 C CNN
+F 3 "" H 6400 5050 60  0000 C CNN
+	1    6400 5050
 	1    0    0    -1
 $EndComp
@@
 L VCC #PWR022
 U 1 1 5A878B2E
-P 5350 4700
-F 0 "#PWR022" H 5350 4800 30  0001 C CNN
-F 1 "VCC" H 5350 4800 30  0000 C CNN
-F 2 "" H 5350 4700 60  0000 C CNN
-F 3 "" H 5350 4700 60  0000 C CNN
-	1    5350 4700
+P 5650 4850
+F 0 "#PWR022" H 5650 4950 30  0001 C CNN
+F 1 "VCC" H 5650 4950 30  0000 C CNN
+F 2 "" H 5650 4850 60  0000 C CNN
+F 3 "" H 5650 4850 60  0000 C CNN
+	1    5650 4850
 	1    0    0    -1
 $EndComp
@@
 L GND-RESCUE-v9958 #PWR023
 U 1 1 5A879985
-P 5350 5550
-F 0 "#PWR023" H 5350 5550 30  0001 C CNN
-F 1 "GND" H 5350 5480 30  0001 C CNN
-F 2 "" H 5350 5550 60  0000 C CNN
-F 3 "" H 5350 5550 60  0000 C CNN
-	1    5350 5550
-	1    0    0    -1
-$EndComp
-NoConn ~ 6900 5200
+P 5650 5300
+F 0 "#PWR023" H 5650 5300 30  0001 C CNN
+F 1 "GND" H 5650 5230 30  0001 C CNN
+F 2 "" H 5650 5300 60  0000 C CNN
+F 3 "" H 5650 5300 60  0000 C CNN
+	1    5650 5300
+	1    0    0    -1
+$EndComp
+NoConn ~ 7100 5200
 $Comp
 L R-RESCUE-v9958 R5
@@
 L MINI_DIN_4 X2
 U 1 1 5A87FE97
-P 6100 7050
-F 0 "X2" H 5700 7575 50  0000 L BNN
-F 1 "S-VIDEO" H 6100 7575 50  0000 L BNN
-F 2 "mini_din:mini_din-M_DIN4" H 6100 7200 50  0001 C CNN
-F 3 "" H 6100 7050 60  0000 C CNN
-	1    6100 7050
+P 6600 6050
+F 0 "X2" H 6200 6575 50  0000 L BNN
+F 1 "S-VIDEO" H 6600 6575 50  0000 L BNN
+F 2 "mini_din:mini_din-M_DIN4" H 6600 6200 50  0001 C CNN
+F 3 "" H 6600 6050 60  0000 C CNN
+	1    6600 6050
 	1    0    0    -1
 $EndComp
@@
 L GND-RESCUE-v9958 #PWR028
 U 1 1 5A8769F1
-P 5450 7050
-F 0 "#PWR028" H 5450 7050 30  0001 C CNN
-F 1 "GND" H 5450 6980 30  0001 C CNN
-F 2 "" H 5450 7050 60  0000 C CNN
-F 3 "" H 5450 7050 60  0000 C CNN
-	1    5450 7050
+P 5950 6050
+F 0 "#PWR028" H 5950 6050 30  0001 C CNN
+F 1 "GND" H 5950 5980 30  0001 C CNN
+F 2 "" H 5950 6050 60  0000 C CNN
+F 3 "" H 5950 6050 60  0000 C CNN
+	1    5950 6050
 	1    0    0    -1
 $EndComp
@@
 L GND-RESCUE-v9958 #PWR029
 U 1 1 5A876BB4
-P 6750 7050
-F 0 "#PWR029" H 6750 7050 30  0001 C CNN
-F 1 "GND" H 6750 6980 30  0001 C CNN
-F 2 "" H 6750 7050 60  0000 C CNN
-F 3 "" H 6750 7050 60  0000 C CNN
-	1    6750 7050
+P 7250 6050
+F 0 "#PWR029" H 7250 6050 30  0001 C CNN
+F 1 "GND" H 7250 5980 30  0001 C CNN
+F 2 "" H 7250 6050 60  0000 C CNN
+F 3 "" H 7250 6050 60  0000 C CNN
+	1    7250 6050
 	1    0    0    -1
 $EndComp
@@
 Connection ~ 7750 5000
 Wire Wire Line
-	6900 4900 7250 4900
+	7100 4900 7250 4900
 Wire Wire Line
 	7750 4900 7850 4900
@@
 	10650 5300 10650 5400
 Wire Wire Line
-	5350 4700 5350 4900
-Wire Wire Line
-	5350 4900 5500 4900
-Wire Wire Line
-	5500 5200 5350 5200
-Wire Wire Line
-	5350 5200 5350 5550
+	5650 4850 5650 4900
+Wire Wire Line
+	5650 4900 5700 4900
+Wire Wire Line
+	5700 5200 5650 5200
+Wire Wire Line
+	5650 5200 5650 5300
 Wire Wire Line
 	7750 5300 7850 5300
@@
 	10750 3950 10750 4050
 Wire Wire Line
-	5450 7050 5450 6950
-Wire Wire Line
-	5450 6950 5500 6950
-Wire Wire Line
-	6700 6950 6750 6950
-Wire Wire Line
-	6750 6950 6750 7050
-Wire Wire Line
-	5600 6850 5300 6850
-Wire Wire Line
-	6600 6850 6900 6850
-Text Label 6850 6850 2    60   ~ 0
+	5950 6050 5950 5950
+Wire Wire Line
+	5950 5950 6000 5950
+Wire Wire Line
+	7200 5950 7250 5950
+Wire Wire Line
+	7250 5950 7250 6050
+Wire Wire Line
+	6100 5850 5800 5850
+Wire Wire Line
+	7100 5850 7400 5850
+Text Label 7350 5850 2    60   ~ 0
 Y_OUT
-Text Label 5550 6850 2    60   ~ 0
+Text Label 6050 5850 2    60   ~ 0
 C_OUT
 Wire Wire Line
-	5600 7250 5600 7450
-Wire Wire Line
-	5600 7450 6600 7450
-Wire Wire Line
-	6600 7450 6600 7250
-Connection ~ 6100 7450
+	6100 6250 6100 6450
+Wire Wire Line
+	6100 6450 7100 6450
+Wire Wire Line
+	7100 6450 7100 6250
+Connection ~ 6600 6450
 $Comp
 L GND-RESCUE-v9958 #PWR030
 U 1 1 5A879426
-P 6100 7550
-F 0 "#PWR030" H 6100 7550 30  0001 C CNN
-F 1 "GND" H 6100 7480 30  0001 C CNN
-F 2 "" H 6100 7550 60  0000 C CNN
-F 3 "" H 6100 7550 60  0000 C CNN
-	1    6100 7550
-	1    0    0    -1
-$EndComp
-Wire Wire Line
-	6100 7450 6100 7550
+P 6600 6550
+F 0 "#PWR030" H 6600 6550 30  0001 C CNN
+F 1 "GND" H 6600 6480 30  0001 C CNN
+F 2 "" H 6600 6550 60  0000 C CNN
+F 3 "" H 6600 6550 60  0000 C CNN
+	1    6600 6550
+	1    0    0    -1
+$EndComp
+Wire Wire Line
+	6600 6450 6600 6550
 Entry Wire Line
 	6650 1050 6750 1150
@@
 D7
 Wire Bus Line
-	1050 5950 1050 5250
+	1050 5250 1050 5950
 Wire Wire Line
 	1150 5850 1300 5850
@@
 	1    0    0    -1
 $EndComp
-$Comp
-L Y3014B U9
-U 1 1 5BDF4865
-P 3900 5450
-F 0 "U9" H 3900 5500 60  0000 C CNN
-F 1 "Y3014B" H 3900 5400 60  0000 C CNN
-F 2 "Housings_DIP:DIP-8_W7.62mm_LongPads" H 3900 5450 60  0001 C CNN
-F 3 "" H 3900 5450 60  0000 C CNN
-	1    3900 5450
-	1    0    0    -1
-$EndComp
-Wire Wire Line
-	2900 5250 3100 5250
-Wire Wire Line
-	2900 5350 3100 5350
-Wire Wire Line
-	2900 5450 3100 5450
 Wire Wire Line
 	4650 1500 4350 1500
@@
 Text Label 700  6750 0    60   ~ 0
 OPL_CLK
+$Sheet
+S 3250 5100 1050 1300
+U 5BE22706
+F0 "Audio" 60
+F1 "audio.sch" 60
+F2 "fl" I L 3250 5250 60
+F3 "LOAD" I L 3250 5350 60
+F4 "SD" I L 3250 5450 60
+$EndSheet
+Wire Wire Line
+	2900 5250 3250 5250
+Wire Wire Line
+	2900 5350 3250 5350
+Wire Wire Line
+	2900 5450 3250 5450
 $EndSCHEMATC

Commit message: ext mem
Parts:
- removed C10, C12, C13, C19, C9: 100n, Capacitors_ThroughHole:C_Disc_D3_P2.5, symbol C
- removed C11, C17: 47µF, Capacitors_ThroughHole:C_Radial_D5_L11_P2.5, symbol CP
- removed C14, C15, C16, C18, C20, C21: 220µF, Capacitors_ThroughHole:C_Radial_D6.3_L11.2_P2.5, symbol CP
- removed P1: RED, w_conn_av:rca_black, symbol CONN_01X02
- removed P2: GREEN, w_conn_av:rca_black, symbol CONN_01X02
- removed P3: BLUE, w_conn_av:rca_black, symbol CONN_01X02
- removed P4: SYNC/C, w_conn_av:rca_black, symbol CONN_01X02
- removed R1, R2, R3: 470, Discret:R3, symbol R-RESCUE-v9958
- removed R10: 2.61k/10%, Discret:R3, symbol R-RESCUE-v9958
- removed R11, R12, R6, R7, R8: 75, Discret:R3, symbol R-RESCUE-v9958
- removed R13: 240, Discret:R3, symbol R-RESCUE-v9958
- removed R4, R5: 2.2k, Discret:R3, symbol R-RESCUE-v9958
- removed R9: 43, Discret:R3, symbol R-RESCUE-v9958
- removed U7: cxa2075M, Housings_SOIC:SOIC-24_7.5x15.4mm_Pitch1.27mm, symbol cxa2075M
- removed X1: OSC, Oscillators:KXO-200_LargePads, symbol OSC
- removed X2: S-VIDEO, mini_din:mini_din-M_DIN4, symbol MINI_DIN_4
- added U? (x2): DRAM_64KX4, Housings_DIP:DIP-18_W7.62mm_LongPads, symbol DRAM_64KX4
Connections:
- net labels added: /CAS_X
- net labels removed: B_OUT, CV_OUT, C_OUT, G_OUT, R_OUT, Y_OUT
- wire segments 247 -> 202
- no-connect marks 13 -> 10
Other:
- moved on the sheet: U3, U4, U5, U6

Commit message: stuff
Parts:
- added C10, C9: 100n, Capacitors_ThroughHole:C_Disc_D3.0mm_W1.6mm_P2.50mm, symbol C
- C1, C2, C3, C4, C5, C6, C7, C8: footprint Capacitors_ThroughHole:C_Disc_D3_P2.5 -> Capacitors_ThroughHole:C_Disc_D3.0mm_W1.6mm_P2.50mm
- gave numbers to parts that had none: 2
Connections:
- wire segments 202 -> 207
Changed lines of the file:
@@
 LIBS:steckschwein
 LIBS:yamaha_opl
+LIBS:w_connectors
 LIBS:v9958-cache
 EELAYER 25 0
@@
 F 0 "C1" H 5125 850 50  0000 L CNN
 F 1 "22p" H 5125 650 50  0000 L CNN
-F 2 "Capacitors_ThroughHole:C_Disc_D3_P2.5" H 5138 600 50  0001 C CNN
+F 2 "Capacitors_ThroughHole:C_Disc_D3.0mm_W1.6mm_P2.50mm" H 5138 600 50  0001 C CNN
 F 3 "" H 5100 750 50  0001 C CNN
 	1    5100 750
@@
 F 0 "C2" H 5725 850 50  0000 L CNN
 F 1 "22p" H 5725 650 50  0000 L CNN
-F 2 "Capacitors_ThroughHole:C_Disc_D3_P2.5" H 5738 600 50  0001 C CNN
+F 2 "Capacitors_ThroughHole:C_Disc_D3.0mm_W1.6mm_P2.50mm" H 5738 600 50  0001 C CNN
 F 3 "" H 5700 750 50  0001 C CNN
 	1    5700 750
@@
 F 0 "C3" H 2425 1050 50  0000 L CNN
 F 1 "100n" H 2425 850 50  0000 L CNN
-F 2 "Capacitors_ThroughHole:C_Disc_D3_P2.5" H 2438 800 50  0001 C CNN
+F 2 "Capacitors_ThroughHole:C_Disc_D3.0mm_W1.6mm_P2.50mm" H 2438 800 50  0001 C CNN
 F 3 "" H 2400 950 50  0001 C CNN
 	1    2400 950
@@
 F 0 "C4" H 2725 1050 50  0000 L CNN
 F 1 "100n" H 2725 850 50  0000 L CNN
-F 2 "Capacitors_ThroughHole:C_Disc_D3_P2.5" H 2738 800 50  0001 C CNN
+F 2 "Capacitors_ThroughHole:C_Disc_D3.0mm_W1.6mm_P2.50mm" H 2738 800 50  0001 C CNN
 F 3 "" H 2700 950 50  0001 C CNN
 	1    2700 950
@@
 F 0 "C5" H 3025 1050 50  0000 L CNN
 F 1 "100n" H 3025 850 50  0000 L CNN
-F 2 "Capacitors_ThroughHole:C_Disc_D3_P2.5" H 3038 800 50  0001 C CNN
+F 2 "Capacitors_ThroughHole:C_Disc_D3.0mm_W1.6mm_P2.50mm" H 3038 800 50  0001 C CNN
 F 3 "" H 3000 950 50  0001 C CNN
 	1    3000 950
@@
 F 0 "C6" H 3325 1050 50  0000 L CNN
 F 1 "100n" H 3325 850 50  0000 L CNN
-F 2 "Capacitors_ThroughHole:C_Disc_D3_P2.5" H 3338 800 50  0001 C CNN
+F 2 "Capacitors_ThroughHole:C_Disc_D3.0mm_W1.6mm_P2.50mm" H 3338 800 50  0001 C CNN
 F 3 "" H 3300 950 50  0001 C CNN
 	1    3300 950
@@
 F 0 "C7" H 3625 1050 50  0000 L CNN
 F 1 "100n" H 3625 850 50  0000 L CNN
-F 2 "Capacitors_ThroughHole:C_Disc_D3_P2.5" H 3638 800 50  0001 C CNN
+F 2 "Capacitors_ThroughHole:C_Disc_D3.0mm_W1.6mm_P2.50mm" H 3638 800 50  0001 C CNN
 F 3 "" H 3600 950 50  0001 C CNN
 	1    3600 950
@@
 F 0 "C8" H 3925 1050 50  0000 L CNN
 F 1 "100n" H 3925 850 50  0000 L CNN
-F 2 "Capacitors_ThroughHole:C_Disc_D3_P2.5" H 3938 800 50  0001 C CNN
+F 2 "Capacitors_ThroughHole:C_Disc_D3.0mm_W1.6mm_P2.50mm" H 3938 800 50  0001 C CNN
 F 3 "" H 3900 950 50  0001 C CNN
 	1    3900 950
@@
 $EndComp
 $Comp
-L GND-RESCUE-v9958 #PWR031
+L GND-RESCUE-v9958 #PWR014
 U 1 1 5A93119E
 P 1650 2650
-F 0 "#PWR031" H 1650 2650 30  0001 C CNN
+F 0 "#PWR014" H 1650 2650 30  0001 C CNN
 F 1 "GND" H 1650 2580 30  0001 C CNN
 F 2 "" H 1650 2650 60  0000 C CNN
@@
 /CS_IO0
 $Comp
-L GND-RESCUE-v9958 #PWR032
+L GND-RESCUE-v9958 #PWR015
 U 1 1 5BBC1C06
 P 1650 3650
-F 0 "#PWR032" H 1650 3650 30  0001 C CNN
+F 0 "#PWR015" H 1650 3650 30  0001 C CNN
 F 1 "GND" H 1650 3580 30  0001 C CNN
 F 2 "" H 1650 3650 60  0000 C CNN
@@
 F3 "LOAD" I L 3250 5350 60
 F4 "SD" I L 3250 5450 60
+F5 "AUDIO_OUT" O L 3250 5650 60
 $EndSheet
 Wire Wire Line
@@
 	2200 1300 2200 1100
 Wire Wire Line
-	2200 1100 3900 1100
+	2200 1100 4500 1100
 Connection ~ 2400 1100
 Wire Wire Line
 	2200 700  2200 800
 Wire Wire Line
-	2200 800  3900 800
+	2200 800  4500 800
 Connection ~ 2400 800
 Connection ~ 2700 800
@@
 F4 "RGB_G" I L 7250 3950 60
 F5 "CSYNC" I L 7250 4050 60
+F6 "AUDIO_OUT" I L 7250 4250 60
 $EndSheet
 Text Label 6950 3750 0    60   ~ 0
@@
 	6950 4050 7250 4050
 $Comp
-L DRAM_64KX4 U?
+L DRAM_64KX4 U7
 U 1 1 5BE3012F
 P 10100 3750
-F 0 "U?" H 10100 3750 50  0000 C CNN
+F 0 "U7" H 10100 3750 50  0000 C CNN
 F 1 "DRAM_64KX4" H 10100 3250 50  0000 C CNN
 F 2 "Housings_DIP:DIP-18_W7.62mm_LongPads" H 10100 3750 50  0001 C CNN
@@
 $EndComp
 $Comp
-L DRAM_64KX4 U?
+L DRAM_64KX4 U9
 U 1 1 5BE30135
 P 10100 4900
-F 0 "U?" H 10100 4900 50  0000 C CNN
+F 0 "U9" H 10100 4900 50  0000 C CNN
 F 1 "DRAM_64KX4" H 10100 4400 50  0000 C CNN
 F 2 "Housings_DIP:DIP-18_W7.62mm_LongPads" H 10100 4900 50  0001 C CNN
@@
 $EndComp
 $Comp
-L GND-RESCUE-v9958 #PWR?
+L GND-RESCUE-v9958 #PWR016
 U 1 1 5BE3013B
 P 10850 4250
-F 0 "#PWR?" H 10850 4250 30  0001 C CNN
+F 0 "#PWR016" H 10850 4250 30  0001 C CNN
 F 1 "GND" H 10850 4180 30  0001 C CNN
 F 2 "" H 10850 4250 60  0000 C CNN
@@
 $EndComp
 $Comp
-L GND-RESCUE-v9958 #PWR?
+L GND-RESCUE-v9958 #PWR017
 U 1 1 5BE30141
 P 10850 5400
-F 0 "#PWR?" H 10850 5400 30  0001 C CNN
+F 0 "#PWR017" H 10850 5400 30  0001 C CNN
 F 1 "GND" H 10850 5330 30  0001 C CNN
 F 2 "" H 10850 5400 60  0000 C CNN
@@
 Text Label 6300 1750 0    60   ~ 0
 /CAS_X
+$Comp
+L C C9
+U 1 1 5BE31936
+P 4200 950
+F 0 "C9" H 4225 1050 50  0000 L CNN
+F 1 "100n" H 4225 850 50  0000 L CNN
+F 2 "Capacitors_ThroughHole:C_Disc_D3.0mm_W1.6mm_P2.50mm" H 4238 800 50  0001 C CNN
+F 3 "" H 4200 950 50  0001 C CNN
+	1    4200 950
+	1    0    0    -1
+$EndComp
+$Comp
+L C C10
+U 1 1 5BE31A15
+P 4500 950
+F 0 "C10" H 4525 1050 50  0000 L CNN
+F 1 "100n" H 4525 850 50  0000 L CNN
+F 2 "Capacitors_ThroughHole:C_Disc_D3.0mm_W1.6mm_P2.50mm" H 4538 800 50  0001 C CNN
+F 3 "" H 4500 950 50  0001 C CNN
+	1    4500 950
+	1    0    0    -1
+$EndComp
+Connection ~ 3900 800
+Connection ~ 4200 800
+Connection ~ 3900 1100
+Connection ~ 4200 1100
+Wire Wire Line
+	3250 5650 2950 5650
+Wire Wire Line
+	2950 5650 2950 6650
+Wire Wire Line
+	2950 6650 6800 6650
+Wire Wire Line
+	6800 6650 6800 4250
+Wire Wire Line
+	6800 4250 7250 4250
 $EndSCHEMATC

Commit message: layout almost done
Changed lines of the file:
@@
 $Comp
 L 74LS139 U1
-U 1 1 5A930A3D
+U 2 1 5A930A3D
 P 2800 2900
 F 0 "U1" H 2800 3000 50  0000 C CNN
@@
 F 2 "Housings_DIP:DIP-16_W7.62mm_LongPads" H 2800 2900 50  0001 C CNN
 F 3 "" H 2800 2900 50  0000 C CNN
-	1    2800 2900
+	2    2800 2900
 	1    0    0    -1
 $EndComp
@@
 $Comp
 L 74LS139 U1
-U 2 1 5BBC17E7
+U 1 1 5BBC17E7
 P 2800 3900
 F 0 "U1" H 2800 4000 50  0000 C CNN
@@
 F 2 "Housings_DIP:DIP-16_W7.62mm_LongPads" H 2800 3900 50  0001 C CNN
 F 3 "" H 2800 3900 50  0000 C CNN
-	2    2800 3900
+	1    2800 3900
 	1    0    0    -1
 $EndComp
