File: kicad/V9958_OPL2/video.sch (KiCad schematic (older format))
At the start: 33 parts

Commit message: stuff
Parts:
- removed P?: RED, w_conn_av:rca_black, symbol CONN_01X02
- removed P?: GREEN, w_conn_av:rca_black, symbol CONN_01X02
- removed P?: BLUE, w_conn_av:rca_black, symbol CONN_01X02
- removed P?: SYNC/C, w_conn_av:rca_black, symbol CONN_01X02
- added J2: RGB, w_conn_av:din-8, symbol DIN-8
- added J3: Composite, w_conn_av:rca_yellow, symbol Conn_Coaxial
- C15, C16, C18, C19: renamed from C?; footprint Capacitors_ThroughHole:C_Disc_D3_P2.5 -> Capacitors_ThroughHole:C_Disc_D3.0mm_W1.6mm_P2.50mm
- C17, C23: renamed from C?; footprint Capacitors_ThroughHole:C_Radial_D5_L11_P2.5 -> Capacitors_ThroughHole:CP_Radial_D6.3mm_P2.50mm
- C20, C21, C22, C24, C26, C27: renamed from C?; footprint Capacitors_ThroughHole:C_Radial_D6.3_L11.2_P2.5 -> Capacitors_ThroughHole:CP_Radial_D6.3mm_P2.50mm
- C25: renamed from C?; footprint Capacitors_ThroughHole:C_Disc_D3_P2.5 -> Capacitors_ThroughHole:C_Disc_D3.0mm_W2.0mm_P2.50mm
- U12: renamed from U?; footprint Housings_SOIC:SOIC-24_7.5x15.4mm_Pitch1.27mm -> Housings_SOIC:SOIC-24W_7.5x15.4mm_Pitch1.27mm
- X1: renamed from X?; footprint Oscillators:KXO-200_LargePads -> Oscillators:Oscillator_DIP-14_LargePads
- gave numbers to parts that had none: 14
Connections:
- net labels added: AUDIO_OUT
- wire segments 92 -> 97

Commit message: din 8 jack footprint
Parts:
- J2: footprint w_conn_av:din-8 -> w_conn_av:DIN-8
Changed lines of the file:
@@
 F 0 "J2" H 7575 1475 50  0000 C CNN
 F 1 "RGB" H 7000 1050 50  0000 L CNN
-F 2 "w_conn_av:din-8" H 7450 1250 50  0001 C CNN
+F 2 "w_conn_av:DIN-8" H 7450 1250 50  0001 C CNN
 F 3 "" H 7450 1250 50  0001 C CNN
 	1    7450 1250

Commit message: DRC fixes
Connections:
- net labels removed: B_OUT, CV_OUT, R_OUT
- wire segments 97 -> 100
Changed lines of the file:
@@
 	0    -1   -1   0
 $EndComp
-Text Label 7000 2550 1    60   ~ 0
-R_OUT
-Text Label 7250 2550 1    60   ~ 0
-G_OUT
-Text Label 7500 2550 1    60   ~ 0
-B_OUT
-Text Label 7750 2600 1    60   ~ 0
-CV_OUT
 Text Label 6850 4250 1    60   ~ 0
 C_OUT
@@
 	4350 3650 4250 3650
 Wire Wire Line
-	7000 2500 7000 2300
-Wire Wire Line
-	7250 2500 7250 2300
-Wire Wire Line
-	7500 2500 7500 2300
+	7000 1350 7000 2500
+Wire Wire Line
+	7250 2000 7250 2500
+Wire Wire Line
+	7500 1550 7500 2500
 Wire Wire Line
 	7750 2500 7750 2300
@@
 	7150 1150 6800 1150
 Wire Wire Line
-	7150 1350 6800 1350
-Wire Wire Line
 	7450 950  7450 850
 Wire Wire Line
@@
 	7750 1150 8100 1150
 Wire Wire Line
-	7750 1250 8100 1250
-Wire Wire Line
-	7750 1350 8100 1350
-Text Label 7800 1250 0    60   ~ 0
-CV_OUT
-Text Label 7800 1350 0    60   ~ 0
-CV_OUT
-Text Label 6800 1350 0    60   ~ 0
-R_OUT
+	7750 1250 8900 1250
+Wire Wire Line
+	7750 1350 8400 1350
 Text Label 7850 1150 0    60   ~ 0
 G_OUT
-Wire Wire Line
-	7450 1550 8100 1550
-Text Label 7850 1550 0    60   ~ 0
-B_OUT
 $Comp
 L VCC #PWR052
@@
 	9050 1450 9050 1600
 Wire Wire Line
-	8900 1250 8550 1250
-Text Label 8550 1250 0    60   ~ 0
-CV_OUT
+	7750 2300 8400 2300
+Wire Wire Line
+	8400 2300 8400 1250
+Connection ~ 8400 1350
+Wire Wire Line
+	7450 1550 7500 1550
+Wire Wire Line
+	7250 2000 8100 2000
+Wire Wire Line
+	8100 2000 8100 1150
+Wire Wire Line
+	7000 1350 7150 1350
+Connection ~ 8400 1250
 $EndSCHEMATC

Commit message: correct rca footprint, layers setup
Parts:
- J3: footprint w_conn_av:rca_yellow -> misc:rca
Changed lines of the file:
@@
 F 0 "J3" H 9060 1370 50  0000 C CNN
 F 1 "Composite" V 9165 1250 50  0000 C CNN
-F 2 "w_conn_av:rca_yellow" H 9050 1250 50  0001 C CNN
+F 2 "misc:rca" H 9050 1250 50  0001 C CNN
 F 3 "" H 9050 1250 50  0001 C CNN
 	1    9050 1250
