File: kicad/sbc/cpu_mem_cpld.sch (KiCad schematic (older format))
At the start: 82 parts, among them CON1 BARREL_JACK, IC1 ATMEGA8-P, J1 USB, J2 DB9, P3 ISP, P4 PS/2 Keyboard, SW1 SW_PUSH, U1 65C02, U10 G65SC22P, U2 7400, U2 LM555N, U3 74HCT00, U3 74LS244, U4 74125, U4 XC95108PC84, U5 74LS06, U5 LP2950, U6 28C256, U7 AS6C4008-55PCN, U7 DS1306, U8 16550, U9 MAX232, X1 CRYSTAL_SMD, X1 OSC, X2 OSC

Commit message: io
Parts:
- gave numbers to parts that had none: 1
- renumbered C8 to C10, C9 to C11, C10 to C12, C11 to C13, C18 to C14, C12 to C15, C13 to C16, C14 to C17, C19 to C18, C20 to C19, C21 to C20, C6 to C21, C15 to C22, C7 to C23, C16 to C24, C17 to C25, C8 to C26, C9 to C5, C10 to C6, C5 to C7, C6 to C8, C7 to C9, P3 to P2, P4 to P3, R12 to R10, R13 to R11, R14 to R12, R15 to R13, R16 to R14, R17 to R15, R4 to R16, R1 to R17, R2 to R18, R3 to R19, R4 to R20, R5 to R21, R20 to R22, R21 to R23, R6 to R4, R7 to R5, R8 to R6, R9 to R7, R10 to R8, R11 to R9, U8 to U10, U10 to U11, U9 to U12, U4 to U13, U5 to U14, U6 to U15, U3 to U16, U7 to U6, U6 to U7, U2 to U8, U7 to U9, X1 to X2, X2 to X3
