File: kicad/sbc/sbc.kicad_pcb (KiCad board)
At the start: 4 copper layers, 72 parts, among them CON1 BARREL_JACK, J1 USB, J2 DB9, P1 USERPORT, SW1 SW_PUSH, U1 W65C02, U10 LM555N, U11 W65C22NxPL, U12 74HCT245, U13 74HCT245, U14 7407, U15 SD_Card, U2 CHUCK, U3 AS6C4008, U4 28C256, U5 74LS06, U6 16550, U7 74125, U8 MAX232, U9 LP2950, X1 OSC, X2 OSC

Commit message: audio video stuff, new placement
Parts:
- removed C1: 10n, Capacitor_THT:C_Disc_D3.0mm_W2.0mm_P2.50mm
- removed C10, C11, C12, C13, C14, C5, C6, C7, C8, C9: 100n, Capacitor_SMD:C_1206_3216Metric_Pad1.33x1.80mm_HandSolder
- removed C15, C16, C23, C24: 100nF, Capacitor_SMD:C_1206_3216Metric_Pad1.33x1.80mm_HandSolder
- removed C17: 1µF, Capacitor_THT:CP_Radial_D4.0mm_P2.00mm
- removed C18, C3: 470µF, Capacitor_THT:CP_Radial_D10.0mm_P5.00mm
- removed C2: 1n, Capacitor_THT:C_Disc_D3.0mm_W2.0mm_P2.50mm
- removed C20: 10µF, Capacitor_THT:CP_Radial_D5.0mm_P2.50mm
- removed C4: 1µ, Capacitor_THT:CP_Radial_D4.0mm_P2.00mm
- removed CON1: BARREL_JACK, Connector_BarrelJack:BarrelJack_Horizontal
- removed J1: USB, Connector_USB:USB_B_OST_USB-B1HSxx_Horizontal
- removed JP1: Jumper_3_Bridged12, Connector_PinHeader_2.54mm:PinHeader_1x03_P2.54mm_Vertical
- removed JTAG1: Conn_01x06_Male, Connector_PinHeader_2.54mm:PinHeader_1x06_P2.54mm_Vertical
- removed P1: USERPORT, Connector_PinHeader_2.54mm:PinHeader_2x08_P2.54mm_Horizontal
- removed R1, R2: 1M, Resistor_THT:R_Axial_DIN0204_L3.6mm_D1.6mm_P5.08mm_Horizontal
- removed R10, R11, R12, R13, R14, R15, R17, R4, R5, R6, R7, R8, R9: 1k, Resistor_THT:R_Axial_DIN0204_L3.6mm_D1.6mm_P5.08mm_Horizontal
- removed R16, R3: 4k7, Resistor_THT:R_Axial_DIN0204_L3.6mm_D1.6mm_P5.08mm_Horizontal
- removed R19, R20: 10k, Resistor_THT:R_Axial_DIN0204_L3.6mm_D1.6mm_P5.08mm_Horizontal
- removed R21, R22: 47k, Resistor_THT:R_Axial_DIN0204_L3.6mm_D1.6mm_P5.08mm_Horizontal
- removed RN1: 3k3, Resistor_THT:R_Array_SIP5
- removed SW1: SW_PUSH, Button_Switch_THT:Push_E-Switch_KS01Q01
- removed U10: LM555N, Package_DIP:DIP-8_W7.62mm_LongPads
- removed U14: 7407, Package_DIP:DIP-14_W7.62mm_Socket_LongPads
- removed U15: SD_Card, Connector_Card:SD_TE_2041021
- removed U5: 74LS06, Package_DIP:DIP-14_W7.62mm_LongPads
- removed U7: 74125, Package_DIP:DIP-14_W7.62mm_Socket_LongPads
- removed U9: LP2950, Package_TO_SOT_THT:TO-92_Inline
- removed X1: OSC, Oscillator:Oscillator_DIP-14_LargePads
- added U16: YM3812, Package_DIP:DIP-24_W15.24mm_LongPads, F.Cu at (215.3, 113.0)
- added U17: 74LS139, Package_DIP:DIP-16_W7.62mm_Socket_LongPads, F.Cu at (260.4, 163.8)
- added U18: V9958, SDIP:SDIP64, F.Cu at (214.4, 142.9)
- added U19: DRAM_64KX4, Package_DIP:DIP-18_W7.62mm_Socket_LongPads, F.Cu at (295.9, 120.0)
- added U20: DRAM_64KX4, Package_DIP:DIP-18_W7.62mm_Socket_LongPads, F.Cu at (295.9, 131.8)
- added U21: DRAM_64KX4, Package_DIP:DIP-18_W7.62mm_Socket_LongPads, F.Cu at (295.9, 143.5)
- added U22: DRAM_64KX4, Package_DIP:DIP-18_W7.62mm_Socket_LongPads, F.Cu at (269.8, 120.2)
- added U23: DRAM_64KX4, Package_DIP:DIP-18_W7.62mm_Socket_LongPads, F.Cu at (269.8, 132.0)
- added U24: DRAM_64KX4, Package_DIP:DIP-18_W7.62mm_Socket_LongPads, F.Cu at (269.8, 143.8)
- moved U13 227.0 mm to (193.0, 163.8), turned to -90 degrees
- moved C19 224.5 mm to (158.8, 108.0), turned to 180 degrees
- moved U6 219.1 mm to (169.5, 132.1), turned to 0 degrees
- moved U8 215.1 mm to (153.7, 113.0), turned to -90 degrees
- moved C21 212.6 mm to (148.1, 108.0), turned to 180 degrees
- moved U12 209.9 mm to (161.9, 163.8), turned to -90 degrees
- moved C25 209.3 mm to (153.1, 108.0)
- moved C22 206.1 mm to (143.0, 108.0), turned to 180 degrees
- moved R18 190.4 mm to (160.0, 81.3), turned to 180 degrees
- moved J2 183.8 mm to (151.6, 76.6)
- moved U2 180.9 mm to (281.9, 198.1)
- moved X2 170.8 mm to (141.0, 132.1), turned to -90 degrees
- moved U11 125.5 mm to (151.8, 182.2)
- moved U3 114.2 mm to (239.4, 184.2), turned to -90 degrees
- moved U1 111.2 mm to (182.9, 182.2)
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Connections:
- U2 pad 1: /CPU_D0 -> /CPU_A6
- U2 pad 13: /CPU_A14 -> unconnected-(U2-P13-Pad13)
- U2 pad 14: /CPU_RDY -> unconnected-(U2-P14-Pad14)
- U2 pad 15: /CPU_A1 -> unconnected-(U2-P15-Pad15)
- U2 pad 17: /CPU_A8 -> unconnected-(U2-P17-Pad17)
- U2 pad 18: /EXT_A15 -> unconnected-(U2-P18-Pad18)
- U2 pad 2: /CPU_D1 -> /CPU_A8
- U2 pad 23: /CPU_D6 -> unconnected-(U2-P23-Pad23)
- U2 pad 25: /~{CS_RAM} -> unconnected-(U2-P25-Pad25)
- U2 pad 26: /~{CS_UART} -> unconnected-(U2-P26-Pad26)
- U2 pad 3: /CPU_A15 -> /CPU_A4
- U2 pad 31: /~{CS_ROM} -> unconnected-(U2-P31-Pad31)
- U2 pad 33: /~{CS_VDP} -> unconnected-(U2-P33-Pad33)
- U2 pad 35: /~{CS_OPL} -> unconnected-(U2-P35-Pad35)
- U2 pad 37: /~{OE} -> unconnected-(U2-P37-Pad37)
- U2 pad 39: /~{WE} -> unconnected-(U2-P39-Pad39)
- U2 pad 4: unconnected-(U2-Pad4) -> /CPU_A5
- U2 pad 43: /~{CS_VIA} -> unconnected-(U2-P43-Pad43)
- U2 pad 44: /CPU_A9 -> unconnected-(U2-P44-Pad44)
- U2 pad 46: /CPU_D2 -> /~{CS_VDP}
- U2 pad 47: /EXT_A16 -> /~{CS_OPL}
- U2 pad 48: /CPU_A4 -> /~{CS_UART}
- U2 pad 5: /EXT_A14 -> /CPU_A1
- U2 pad 52: /EXT_A17 -> /CPU_D2
- U2 pad 53: /CPU_A6 -> /CPU_D3
- U2 pad 54: unconnected-(U2-Pad54) -> /CPU_D4
- U2 pad 55: unconnected-(U2-Pad55) -> /CPU_D1
- U2 pad 56: /CPU_A12 -> /CPU_D5
- U2 pad 57: unconnected-(U2-Pad57) -> /CPU_D0
- U2 pad 58: unconnected-(U2-Pad58) -> /CPU_D6
- U2 pad 6: unconnected-(U2-Pad6) -> /CPU_A0
- U2 pad 61: /EXT_A18 -> /CPU_D7
- U2 pad 65: /CPU_A10 -> unconnected-(U2-P65-Pad65)
- U2 pad 66: /CPU_A11 -> unconnected-(U2-P66-Pad66)
- U2 pad 67: unconnected-(U2-Pad67) -> /~{OE}
- U2 pad 68: /CPU_D4 -> /~{WE}
- U2 pad 69: unconnected-(U2-Pad69) -> /EXT_A14
- U2 pad 70: /CPU_A5 -> /EXT_A17
- U2 pad 71: /CPU_R~{W} -> /EXT_A16
- U2 pad 72: /CPU_D3 -> /EXT_A15
- U2 pad 75: /~{CS_BUFFER} -> /CPU_A15
- U2 pad 76: unconnected-(U2-Pad76) -> /EXT_A18
- U2 pad 77: unconnected-(U2-Pad77) -> /CPU_A13
- U2 pad 79: /CPU_D7 -> /CPU_A12
- U2 pad 80: unconnected-(U2-Pad80) -> /CPU_A14
- U2 pad 81: /CPU_A0 -> /CPU_A9
- U2 pad 82: /CPU_D5 -> /CPU_A11
- U2 pad 84: /CPU_A13 -> /CPU_A10
Routing:
- net /~{RESET}: track 0.00 -> 220.1 mm
- net /PHI2: track 0.00 -> 183.8 mm
- net /Video_Audio/RD0: track 0.00 -> 137.2 mm
- net /~{WE}: track 13.5 -> 150.4 mm, vias 0 -> 1
- net /~{CS_UART}: track 0.00 -> 133.6 mm
- net /CPU_D7: track 52.4 -> 185.5 mm
- net /Video_Audio/RD1: track 0.00 -> 127.5 mm
- net /Video_Audio/A0..A7: track 0.00 -> 126.6 mm
- net /Video_Audio/RD4: track 0.00 -> 126.4 mm
- net /Video_Audio/RD3: track 0.00 -> 124.3 mm
- net /Video_Audio/RD5: track 0.00 -> 124.0 mm
- net /Video_Audio/AD1: track 0.00 -> 123.3 mm
- net /Video_Audio/RD2: track 0.00 -> 121.2 mm
- net /~{OE}: track 21.3 -> 141.8 mm
- net /CPU_D2: track 53.7 -> 173.6 mm
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- added copper zone on In2.Cu, net GND
- added copper zone on In1.Cu, net VCC
Other:
- board outline added: 299.7 x 159.4 mm

Commit message: cpld pinout
Parts:
- added C1: 10n, Capacitor_THT:C_Disc_D3.0mm_W2.0mm_P2.50mm, F.Cu at (165.1, 106.7)
- added C10: 100n, Capacitor_SMD:C_1206_3216Metric_Pad1.33x1.80mm_HandSolder, F.Cu at (243.2, 197.8)
- added C11: 100n, Capacitor_SMD:C_1206_3216Metric_Pad1.33x1.80mm_HandSolder, B.Cu at (282.6, 184.4)
- added C12: 100n, Capacitor_SMD:C_1206_3216Metric_Pad1.33x1.80mm_HandSolder, F.Cu at (273.7, 145.1)
- added C13: 100n, Capacitor_SMD:C_1206_3216Metric_Pad1.33x1.80mm_HandSolder, B.Cu at (247.0, 184.4)
- added C14: 100n, Capacitor_SMD:C_1206_3216Metric_Pad1.33x1.80mm_HandSolder, B.Cu at (272.4, 174.3)
- added C15: 100nF, Capacitor_SMD:C_1206_3216Metric_Pad1.33x1.80mm_HandSolder, B.Cu at (256.2, 193.0)
- added C16: 100nF, Capacitor_SMD:C_1206_3216Metric_Pad1.33x1.80mm_HandSolder, B.Cu at (254.6, 188.9)
- added C17: 1µF, Capacitor_THT:CP_Radial_D4.0mm_P2.00mm, F.Cu at (137.2, 108.0)
- added C18: 470µF, Capacitor_THT:CP_Radial_D10.0mm_P5.00mm, F.Cu at (318.9, 160.0)
- added C2: 1n, Capacitor_THT:C_Disc_D3.0mm_W2.0mm_P2.50mm, F.Cu at (181.6, 95.2)
- added C20: 10µF, Capacitor_THT:CP_Radial_D5.0mm_P2.50mm, F.Cu at (77.5, 161.9)
- added C23: 100nF, Capacitor_SMD:C_1206_3216Metric_Pad1.33x1.80mm_HandSolder, F.Cu at (73.7, 156.8)
- added C24: 100nF, Capacitor_SMD:C_1206_3216Metric_Pad1.33x1.80mm_HandSolder, F.Cu at (94.6, 179.1)
- added C26: 100n, Capacitor_SMD:C_1206_3216Metric_Pad1.33x1.80mm_HandSolder, F.Cu at (273.7, 133.1)
- added C27: 100n, Capacitor_SMD:C_1206_3216Metric_Pad1.33x1.80mm_HandSolder, F.Cu at (273.7, 121.6)
- added C28: 100n, Capacitor_SMD:C_1206_3216Metric_Pad1.33x1.80mm_HandSolder, F.Cu at (246.4, 121.6)
- added C29: 100n, Capacitor_SMD:C_1206_3216Metric_Pad1.33x1.80mm_HandSolder, F.Cu at (246.4, 133.7)
- added C3: 470µF, Capacitor_THT:CP_Radial_D10.0mm_P5.00mm, F.Cu at (86.4, 106.6)
- added C30: 100n, Capacitor_SMD:C_1206_3216Metric_Pad1.33x1.80mm_HandSolder, F.Cu at (246.4, 145.1)
- added C31: 100n, Capacitor_SMD:C_1206_3216Metric_Pad1.33x1.80mm_HandSolder, F.Cu at (243.8, 126.7)
- added C32: 22p, Capacitor_SMD:C_1206_3216Metric_Pad1.33x1.80mm_HandSolder, F.Cu at (233.0, 157.8)
- added C33: 100n, Capacitor_SMD:C_1206_3216Metric_Pad1.33x1.80mm_HandSolder, F.Cu at (218.4, 114.6)
- added C34: 100n, Capacitor_SMD:C_1206_3216Metric_Pad1.33x1.80mm_HandSolder, B.Cu at (207.4, 136.5)
- added C35: 22p, Capacitor_SMD:C_1206_3216Metric_Pad1.33x1.80mm_HandSolder, F.Cu at (249.6, 157.5)
- added C36: 100n, Capacitor_SMD:C_1206_3216Metric_Pad1.33x1.80mm_HandSolder, F.Cu at (160.7, 114.6)
- added C37: 100n, Capacitor_SMD:C_1206_3216Metric_Pad1.33x1.80mm_HandSolder, B.Cu at (155.3, 142.2)
- added C38: 100µF, Capacitor_THT:CP_Radial_D4.0mm_P2.00mm, F.Cu at (182.9, 142.8)
- added C4: 1µ, Capacitor_THT:CP_Radial_D4.0mm_P2.00mm, F.Cu at (176.5, 95.2)
- added C5: 100n, Capacitor_SMD:C_1206_3216Metric_Pad1.33x1.80mm_HandSolder, B.Cu at (152.7, 200.0)
- added C6: 100n, Capacitor_SMD:C_1206_3216Metric_Pad1.33x1.80mm_HandSolder, B.Cu at (193.0, 186.3)
- added C7: 100n, Capacitor_SMD:C_1206_3216Metric_Pad1.33x1.80mm_HandSolder, F.Cu at (165.1, 169.8)
- added C8: 100n, Capacitor_SMD:C_1206_3216Metric_Pad1.33x1.80mm_HandSolder, F.Cu at (196.2, 169.8)
- added C9: 100n, Capacitor_SMD:C_1206_3216Metric_Pad1.33x1.80mm_HandSolder, F.Cu at (237.5, 175.9)
- added CON1: BARREL_JACK, Connector_BarrelJack:BarrelJack_Horizontal, F.Cu at (77.1, 96.5)
- added J1: USB, Connector_USB:USB_B_OST_USB-B1HSxx_Horizontal, F.Cu at (77.7, 115.5)
- added JP1: Jumper_3_Bridged12, Connector_PinHeader_2.54mm:PinHeader_1x03_P2.54mm_Vertical, F.Cu at (238.1, 180.3)
- added JP2: JUMPER, Connector_PinHeader_2.54mm:PinHeader_1x02_P2.54mm_Vertical, F.Cu at (200.7, 159.4)
- added JTAG1: Conn_01x06_Male, Connector_PinHeader_2.54mm:PinHeader_1x06_P2.54mm_Vertical, F.Cu at (287.7, 165.1)
- added P1: USERPORT, Connector_PinHeader_2.54mm:PinHeader_2x08_P2.54mm_Horizontal, F.Cu at (128.3, 76.8)
- added R1: 1M, Resistor_THT:R_Axial_DIN0204_L3.6mm_D1.6mm_P5.08mm_Horizontal, F.Cu at (165.1, 99.1)
- added R10: 1k, Resistor_THT:R_Axial_DIN0204_L3.6mm_D1.6mm_P5.08mm_Horizontal, F.Cu at (142.2, 81.3)
- added R11: 1k, Resistor_THT:R_Axial_DIN0204_L3.6mm_D1.6mm_P5.08mm_Horizontal, F.Cu at (144.7, 81.3)
- added R12: 1k, Resistor_THT:R_Axial_DIN0204_L3.6mm_D1.6mm_P5.08mm_Horizontal, F.Cu at (147.3, 81.3)
- added R13: 1k, Resistor_THT:R_Axial_DIN0204_L3.6mm_D1.6mm_P5.08mm_Horizontal, F.Cu at (149.9, 81.3)
- added R14: 1k, Resistor_THT:R_Axial_DIN0204_L3.6mm_D1.6mm_P5.08mm_Horizontal, F.Cu at (92.7, 163.2)
- added R15: 1k, Resistor_THT:R_Axial_DIN0204_L3.6mm_D1.6mm_P5.08mm_Horizontal, F.Cu at (92.7, 165.7)
- added R16: 4k7, Resistor_THT:R_Axial_DIN0204_L3.6mm_D1.6mm_P5.08mm_Horizontal, F.Cu at (182.2, 112.4)
- added R17: 1k, Resistor_THT:R_Axial_DIN0204_L3.6mm_D1.6mm_P5.08mm_Horizontal, F.Cu at (97.8, 176.5)
- added R19: 10k, Resistor_THT:R_Axial_DIN0204_L3.6mm_D1.6mm_P5.08mm_Horizontal, F.Cu at (92.7, 182.9)
- added R2: 1M, Resistor_THT:R_Axial_DIN0204_L3.6mm_D1.6mm_P5.08mm_Horizontal, F.Cu at (167.6, 104.1)
- added R20: 10k, Resistor_THT:R_Axial_DIN0204_L3.6mm_D1.6mm_P5.08mm_Horizontal, F.Cu at (97.8, 185.4)
- added R21: 47k, Resistor_THT:R_Axial_DIN0204_L3.6mm_D1.6mm_P5.08mm_Horizontal, F.Cu at (97.8, 168.3)
- added R22: 47k, Resistor_THT:R_Axial_DIN0204_L3.6mm_D1.6mm_P5.08mm_Horizontal, F.Cu at (97.8, 188.0)
- added R3: 4k7, Resistor_THT:R_Axial_DIN0204_L3.6mm_D1.6mm_P5.08mm_Horizontal, F.Cu at (162.6, 99.1)
- added R4: 1k, Resistor_THT:R_Axial_DIN0204_L3.6mm_D1.6mm_P5.08mm_Horizontal, F.Cu at (127.0, 81.3)
- added R5: 1k, Resistor_THT:R_Axial_DIN0204_L3.6mm_D1.6mm_P5.08mm_Horizontal, F.Cu at (129.5, 81.3)
- added R6: 1k, Resistor_THT:R_Axial_DIN0204_L3.6mm_D1.6mm_P5.08mm_Horizontal, F.Cu at (132.1, 81.3)
- added R7: 1k, Resistor_THT:R_Axial_DIN0204_L3.6mm_D1.6mm_P5.08mm_Horizontal, F.Cu at (134.6, 81.3)
- added R8: 1k, Resistor_THT:R_Axial_DIN0204_L3.6mm_D1.6mm_P5.08mm_Horizontal, F.Cu at (137.2, 81.3)
- added R9: 1k, Resistor_THT:R_Axial_DIN0204_L3.6mm_D1.6mm_P5.08mm_Horizontal, F.Cu at (139.7, 81.3)
- added RN1: 3k3, Resistor_THT:R_Array_SIP5, F.Cu at (167.0, 199.4)
- added SLOT0: Conn_02x12_Odd_Even, Connector_PinHeader_2.54mm:PinHeader_2x12_P2.54mm_Vertical, F.Cu at (118.1, 115.6)
- added SW1: SW_PUSH, Button_Switch_THT:Push_E-Switch_KS01Q01, F.Cu at (69.9, 73.7)
- added U10: LM555N, Package_DIP:DIP-8_W7.62mm_LongPads, F.Cu at (171.4, 106.7)
- added U14: 7407, Package_DIP:DIP-14_W7.62mm_Socket_LongPads, F.Cu at (129.5, 176.5)
- added U15: SD_Card, Connector_Card:SD_TE_2041021, F.Cu at (76.8, 178.4)
- added U5: 74LS06, Package_DIP:DIP-14_W7.62mm_LongPads, F.Cu at (163.8, 120.7)
- added U7: 74125, Package_DIP:DIP-14_W7.62mm_Socket_LongPads, F.Cu at (129.5, 163.8)
- added U9: LP2950, Package_TO_SOT_THT:TO-92_Inline, F.Cu at (67.9, 159.4)
- added X1: OSC, Oscillator:Oscillator_DIP-14_LargePads, F.Cu at (288.3, 183.5)
- added Y1: 21,443Mhz, Crystal:Crystal_HC49-U_Vertical, F.Cu at (238.8, 157.5)
- moved U17 48.3 mm to (240.0, 120.0)
- moved X2 37.8 mm to (113.0, 157.5), turned to 0 degrees
- moved J2 24.3 mm to (175.9, 76.6)
- moved U2 17.1 mm to (264.8, 198.1)
- moved R18 7.81 mm to (167.8, 81.3), turned to 0 degrees
- moved U19 1.27 mm to (297.2, 120.0)
- moved U20 1.27 mm to (297.2, 131.8)
- moved U21 1.27 mm to (297.2, 143.5)
Connections:
- U2 pad 1: /CPU_A6 -> /EXT_A17
- U2 pad 19: /PHI2 -> unconnected-(U2-P19-Pad19)
- U2 pad 2: /CPU_A8 -> /EXT_A18
- U2 pad 3: /CPU_A4 -> /PHI2
- U2 pad 35: unconnected-(U2-P35-Pad35) -> /PHI2
- U2 pad 39: unconnected-(U2-P39-Pad39) -> /~{CS_SLOT0}
- U2 pad 4: /CPU_A5 -> /~{CS_ROM}
- U2 pad 40: unconnected-(U2-P40-Pad40) -> /CPU_RDY
- U2 pad 46: /~{CS_VDP} -> unconnected-(U2-P46-Pad46)
- U2 pad 47: /~{CS_OPL} -> /~{CS_VDP}
- U2 pad 5: /CPU_A1 -> /~{CS_RAM}
- U2 pad 50: unconnected-(U2-P50-Pad50) -> /~{CS_SLOT1}
- U2 pad 51: unconnected-(U2-P51-Pad51) -> /~{CS_VIA}
- U2 pad 52: /CPU_D2 -> /~{CS_BUFFER}
- U2 pad 53: /CPU_D3 -> /~{CS_OPL}
- U2 pad 54: /CPU_D4 -> /CPU_D0
- U2 pad 56: /CPU_D5 -> /CPU_D2
- U2 pad 57: /CPU_D0 -> /CPU_D3
- U2 pad 58: /CPU_D6 -> /CPU_D4
- U2 pad 6: /CPU_A0 -> /~{OE}
- U2 pad 61: /CPU_D7 -> /CPU_D5
- U2 pad 62: unconnected-(U2-P62-Pad62) -> /CPU_D6
- U2 pad 63: unconnected-(U2-P63-Pad63) -> /CPU_D7
- U2 pad 65: unconnected-(U2-P65-Pad65) -> /CPU_A0
- U2 pad 66: unconnected-(U2-P66-Pad66) -> /CPU_A1
- U2 pad 67: /~{OE} -> /CPU_A4
- U2 pad 68: /~{WE} -> /CPU_A5
- U2 pad 69: /EXT_A14 -> /CPU_A6
- U2 pad 7: unconnected-(U2-P7-Pad7) -> /~{WE}
- U2 pad 70: /EXT_A17 -> /CPU_A7
- U2 pad 71: /EXT_A16 -> /CPU_A8
- U2 pad 72: /EXT_A15 -> /CPU_A9
- U2 pad 75: /CPU_A15 -> /CPU_A10
- U2 pad 76: /EXT_A18 -> /CPU_A11
- U2 pad 77: /CPU_A13 -> /CPU_A12
- U2 pad 79: /CPU_A12 -> /CPU_A13
- U2 pad 81: /CPU_A9 -> /CPU_A15
- U2 pad 82: /CPU_A11 -> /EXT_A14
- U2 pad 83: /CPU_A7 -> /EXT_A15
- U2 pad 84: /CPU_A10 -> /EXT_A16
Routing:
- net /~{RESET}: track 220.1 -> 0.00 mm
- net /CPU_D2: track 173.6 -> 0.00 mm
- net /CPU_D5: track 170.1 -> 0.00 mm
- net /CPU_D7: track 185.5 -> 21.2 mm
- net /CPU_D4: track 160.3 -> 0.00 mm, vias 1 -> 0
- net /PHI2: track 183.8 -> 30.0 mm
- net /CPU_D3: track 170.7 -> 25.7 mm
- net /CPU_A1: track 183.5 -> 39.1 mm
- net /CPU_A0: track 176.6 -> 33.0 mm
- net /CPU_D1: track 161.7 -> 21.1 mm
- net /CPU_D0: track 161.3 -> 21.1 mm
- net /Video_Audio/RD0: track 137.2 -> 0.00 mm
- net /CPU_A8: track 137.0 -> 0.00 mm
- net /CPU_D6: track 157.7 -> 21.1 mm
- net /~{CS_UART}: track 133.6 -> 0.00 mm
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
Commit message: more vias to gnd
Routing:
- net /~{RESET}: track 0.00 -> 312.7 mm, vias 0 -> 1
- net /~{IRQ}: track 0.00 -> 230.4 mm, vias 0 -> 2
- net /CPU_D5: track 0.00 -> 180.5 mm
- net /BUF_A0: track 0.00 -> 175.7 mm, vias 0 -> 1
- net /CPU_D2: track 0.00 -> 166.3 mm, vias 0 -> 2
- net /CPU_D4: track 0.00 -> 165.0 mm
- net /PHI2: track 30.0 -> 192.6 mm, vias 0 -> 1
- net /BUF_D1: track 0.00 -> 146.6 mm
- net /BUF_D0: track 0.00 -> 143.7 mm, vias 0 -> 1
- net /BUF_D5: track 0.00 -> 142.0 mm
- net /Video_Audio/RD0: track 0.00 -> 136.1 mm
- net /CPU_D7: track 21.2 -> 157.2 mm
- net /CPU_RDY: track 0.00 -> 131.3 mm
- net /Video_Audio/RD1: track 0.00 -> 128.7 mm
- net /BUF_D6: track 0.00 -> 127.6 mm, vias 0 -> 1
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
Commit message: complete schematics
Parts:
- added C39: 47µF, Capacitor_THT:CP_Radial_D4.0mm_P2.00mm, F.Cu at (193.4, 87.0)
- added C40: 10µF, Capacitor_THT:CP_Radial_D5.0mm_P2.50mm, F.Cu at (198.2, 87.0)
- added C41: 470p, Capacitor_THT:C_Disc_D3.0mm_W2.0mm_P2.50mm, F.Cu at (193.0, 102.2)
- added C42: 470p, Capacitor_THT:C_Disc_D3.0mm_W2.0mm_P2.50mm, F.Cu at (195.6, 102.2)
- added C43: 10µF, Capacitor_THT:CP_Radial_D5.0mm_P2.50mm, F.Cu at (210.2, 90.2)
- added C44: 100n, Capacitor_SMD:C_1206_3216Metric_Pad1.33x1.80mm_HandSolder, F.Cu at (215.5, 105.9)
- added C45: 100n, Capacitor_SMD:C_1206_3216Metric_Pad1.33x1.80mm_HandSolder, F.Cu at (215.5, 112.3)
- added C46: 47µF, Capacitor_THT:CP_Radial_D5.0mm_P2.50mm, F.Cu at (241.3, 111.8)
- added C47: 100n, Capacitor_SMD:C_1206_3216Metric_Pad1.33x1.80mm_HandSolder, F.Cu at (215.5, 109.1)
- added C48: 100n, Capacitor_SMD:C_1206_3216Metric_Pad1.33x1.80mm_HandSolder, F.Cu at (236.9, 110.8)
- added C49: 220µF, Capacitor_THT:CP_Radial_D4.0mm_P2.00mm, F.Cu at (266.1, 88.1)
- added C50: 220µF, Capacitor_THT:CP_Radial_D4.0mm_P2.00mm, F.Cu at (234.9, 88.1)
- added C51: 220µF, Capacitor_THT:CP_Radial_D4.0mm_P2.00mm, F.Cu at (261.0, 88.1)
- added C52: 47µF, Capacitor_THT:CP_Radial_D5.0mm_P2.50mm, F.Cu at (241.3, 105.4)
- added C53: 220µF, Capacitor_THT:CP_Radial_D4.0mm_P2.00mm, F.Cu at (247.7, 88.4)
- added C54: 100n, Capacitor_SMD:C_1206_3216Metric_Pad1.33x1.80mm_HandSolder, F.Cu at (236.9, 104.1)
- added C55: 220µF, Capacitor_THT:CP_Radial_D4.0mm_P2.00mm, F.Cu at (241.1, 88.1)
- added C56: 220µF, Capacitor_THT:CP_Radial_D4.0mm_P2.00mm, F.Cu at (254.0, 88.1)
- added IC1: ATMEGA8-P, Package_DIP:DIP-28_W7.62mm_LongPads, F.Cu at (113.7, 118.7)
- added J3: Audio, Connector_Audio:Jack_3.5mm_Lumberg_1503_07_Horizontal, F.Cu at (208.7, 69.5)
- added J4: S-VIDEO, DIN:mini_din-M_DIN4, F.Cu at (263.3, 68.5)
- added J5: RGB, DIN:DIN-8, F.Cu at (243.7, 76.2)
- added P2: CONN_01X03, Connector_PinHeader_2.54mm:PinHeader_1x03_P2.54mm_Vertical, F.Cu at (113.7, 130.8)
- added P3: ISP, Connector_PinHeader_2.54mm:PinHeader_2x03_P2.54mm_Horizontal, F.Cu at (76.2, 125.1)
- added P4: PS/2 Keyboard, DIN:mini_din-M_DIN6, F.Cu at (68.6, 104.1)
- added Port1: DB9, Connector_Dsub:DSUB-9_Male_Horizontal_P2.77x2.84mm_EdgePinOffset4.94mm_Housed_MountingHolesOffset7.48mm, F.Cu at (99.1, 77.8)
- added Port2: DB9, Connector_Dsub:DSUB-9_Male_Horizontal_P2.77x2.84mm_EdgePinOffset4.94mm_Housed_MountingHolesOffset7.48mm, F.Cu at (134.0, 77.8)
- added R23: 4K7, Resistor_THT:R_Axial_DIN0204_L3.6mm_D1.6mm_P5.08mm_Horizontal, F.Cu at (207.0, 92.1)
- added R24: 33K, Resistor_THT:R_Axial_DIN0204_L3.6mm_D1.6mm_P5.08mm_Horizontal, F.Cu at (209.6, 99.7)
- added R25: 15K, Resistor_THT:R_Axial_DIN0204_L3.6mm_D1.6mm_P5.08mm_Horizontal, F.Cu at (204.5, 87.0)
- added R26: 27K, Resistor_THT:R_Axial_DIN0204_L3.6mm_D1.6mm_P5.08mm_Horizontal, F.Cu at (204.5, 94.6)
- added R27: 4K7, Resistor_THT:R_Axial_DIN0204_L3.6mm_D1.6mm_P5.08mm_Horizontal, F.Cu at (207.0, 99.7)
- added R28: 470, Resistor_THT:R_Axial_DIN0204_L3.6mm_D1.6mm_P5.08mm_Horizontal, F.Cu at (204.5, 111.8)
- added R29: 470, Resistor_THT:R_Axial_DIN0204_L3.6mm_D1.6mm_P5.08mm_Horizontal, F.Cu at (204.5, 109.2)
- added R30: 470, Resistor_THT:R_Axial_DIN0204_L3.6mm_D1.6mm_P5.08mm_Horizontal, F.Cu at (204.5, 106.7)
- added R31: 2.2k, Resistor_THT:R_Axial_DIN0204_L3.6mm_D1.6mm_P5.08mm_Horizontal, F.Cu at (225.4, 99.1)
- added R32: 2.2k, Resistor_THT:R_Axial_DIN0204_L3.6mm_D1.6mm_P5.08mm_Horizontal, F.Cu at (226.7, 115.6)
- added R33: 75, Resistor_THT:R_Axial_DIN0204_L3.6mm_D1.6mm_P5.08mm_Horizontal, F.Cu at (234.9, 95.6)
- added R34: 75, Resistor_THT:R_Axial_DIN0204_L3.6mm_D1.6mm_P5.08mm_Horizontal, F.Cu at (247.7, 95.9)
- added R35: 75, Resistor_THT:R_Axial_DIN0204_L3.6mm_D1.6mm_P5.08mm_Horizontal, F.Cu at (241.1, 95.6)
- added R36: 43, Resistor_THT:R_Axial_DIN0204_L3.6mm_D1.6mm_P5.08mm_Horizontal, F.Cu at (254.0, 95.6)
- added R37: 2.61k/10%, Resistor_THT:R_Axial_DIN0204_L3.6mm_D1.6mm_P5.08mm_Horizontal, F.Cu at (229.2, 99.1)
- added R38: 75, Resistor_THT:R_Axial_DIN0204_L3.6mm_D1.6mm_P5.08mm_Horizontal, F.Cu at (261.0, 95.7)
- added R39: 75, Resistor_THT:R_Axial_DIN0204_L3.6mm_D1.6mm_P5.08mm_Horizontal, F.Cu at (266.1, 95.7)
- added R40: 240, Resistor_THT:R_Axial_DIN0204_L3.6mm_D1.6mm_P5.08mm_Horizontal, F.Cu at (256.5, 90.5)
- added R41: 1k, Resistor_THT:R_Axial_DIN0204_L3.6mm_D1.6mm_P5.08mm_Horizontal, F.Cu at (108.0, 84.5)
- added R42: 1k, Resistor_THT:R_Axial_DIN0204_L3.6mm_D1.6mm_P5.08mm_Horizontal, F.Cu at (108.0, 87.6)
- added RR1: 1k, Resistor_THT:R_Array_SIP8, F.Cu at (102.9, 87.6)
- added SLOT1: Conn_02x12_Odd_Even, Connector_PinSocket_2.54mm:PinSocket_2x12_P2.54mm_Vertical, F.Cu at (123.2, 91.4)
- added U25: Y3014B, Package_DIP:DIP-8_W7.62mm_LongPads, F.Cu at (179.7, 91.4)
- added U26: LM324, Package_DIP:DIP-14_W7.62mm_LongPads, F.Cu at (200.7, 91.4)
- added U27: cxa2075M, Package_SO:SOIC-24W_7.5x15.4mm_P1.27mm, F.Cu at (227.3, 107.7)
- added U28: 7400, Package_DIP:DIP-14_W7.62mm_LongPads, F.Cu at (98.4, 101.0)
- added U29: 74LS244, Package_DIP:DIP-20_W7.62mm_LongPads, F.Cu at (90.8, 113.0)
- added X3: OSC, Oscillator:Oscillator_DIP-14_LargePads, F.Cu at (221.6, 78.1)
- R14: value 1k -> 33K
- SLOT0: footprint Connector_PinHeader_2.54mm:PinHeader_2x12_P2.54mm_Vertical -> Connector_PinSocket_2.54mm:PinSocket_2x12_P2.54mm_Vertical
- U14, U7: footprint Package_DIP:DIP-14_W7.62mm_Socket_LongPads -> Package_DIP:DIP-14_W7.62mm_LongPads
- U15: value SD_Card -> Micro_SD_Card_Det1; footprint Connector_Card:SD_TE_2041021 -> Connector_Card:microSD_HC_Hirose_DM3BT-DSF-PEJS
- U17: footprint Package_DIP:DIP-16_W7.62mm_Socket_LongPads -> Package_DIP:DIP-16_W7.62mm_LongPads
- U3: footprint Package_DIP:DIP-32_W15.24mm_LongPads -> Package_DIP:DIP-32_W15.24mm_Socket_LongPads
- moved J1 320.7 mm to (385.0, 24.1)
- moved CON1 265.1 mm to (332.7, 26.3), turned to -90 degrees
- moved C3 250.0 mm to (333.6, 69.3), turned to 0 degrees
- moved C18 151.0 mm to (173.4, 119.4)
- moved R14 137.7 mm to (212.1, 94.6), turned to -90 degrees
- moved R1 116.3 mm to (104.1, 198.1), turned to 0 degrees
- moved P1 115.7 mm to (76.8, 180.3), turned to 180 degrees
- moved SW1 114.4 mm to (68.7, 188.0)
- moved R5 113.7 mm to (83.8, 185.4), turned to 0 degrees
- moved C2 112.6 mm to (127.0, 193.7), turned to 0 degrees
- moved R7 111.3 mm to (83.8, 180.3), turned to 0 degrees
- moved R3 110.7 mm to (104.1, 193.0), turned to 0 degrees
- moved R16 110.5 mm to (104.1, 190.5), turned to 0 degrees
- moved R4 110.4 mm to (83.8, 182.9), turned to 0 degrees
- moved R2 108.5 mm to (109.2, 195.6), turned to 180 degrees
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Connections:
- net Net-(U15-CLK) renamed /SD Card/CLK
- net Net-(U15-DAT0) renamed /SD Card/DAT0
- net Net-(U15-DAT1) renamed /SD Card/DAT1
- C20 pad 1: Net-(U15-VDD) -> Net-(U15-VSS)
- C24 pad 1: Net-(U15-VDD) -> Net-(U15-VSS)
- R14 pad 1: /~{SD_WRITE_PROTECT} -> Net-(U26A--)
- R14 pad 2: Net-(U11-PB5) -> Net-(C42-Pad2)
- R17 pad 1: Net-(U15-VDD) -> Net-(U15-VSS)
- R19 pad 1: Net-(U15-VDD) -> Net-(U15-VSS)
- R19 pad 2: Net-(U15-CMD) -> /SD Card/CMD
- R20 pad 1: Net-(U15-VDD) -> Net-(U15-VSS)
- R20 pad 2: Net-(U15-CD/DAT3) -> /SD Card/DAT3
- R21 pad 1: Net-(U15-VDD) -> Net-(U15-VSS)
- R22 pad 1: Net-(U15-VDD) -> Net-(U15-VSS)
- R22 pad 2: Net-(U15-DAT2) -> /SD Card/DAT2
- SLOT0 pad 10: unconnected-(SLOT0-Pin_10-Pad10) -> /BUF_R~{W}
- SLOT0 pad 12: unconnected-(SLOT0-Pin_12-Pad12) -> /BUF_PHI2
- SLOT0 pad 16: unconnected-(SLOT0-Pin_16-Pad16) -> /~{CS_SLOT0}
- SLOT0 pad 23: unconnected-(SLOT0-Pin_23-Pad23) -> VCC
- SLOT0 pad 24: unconnected-(SLOT0-Pin_24-Pad24) -> GND
- U11 pad 16: Net-(U11-PB5) -> unconnected-(U11-PB5-Pad16)
- U14 pad 10: Net-(U15-CMD) -> /SD Card/CMD
- U14 pad 12: Net-(U15-CD/DAT3) -> /SD Card/DAT3
- U15 pad 1: Net-(U15-CD/DAT3) -> /SD Card/DAT2
- U15 pad 10: /~{SD_CARD_DETECT} -> GND
- U15 pad 11: /~{SD_WRITE_PROTECT} -> (no net)
- U15 pad 2: Net-(U15-CMD) -> /SD Card/DAT3
- U15 pad 3: GND -> /SD Card/CMD
- U15 pad 4: Net-(U15-VDD) -> GND
- U15 pad 6: GND -> Net-(U15-VSS)
- U15 pad 9: Net-(U15-DAT2) -> /~{SD_CARD_DETECT}
- U16 pad 20: unconnected-(U16-SH-Pad20) -> /Video_Audio/Audio_analog/LOAD
- U16 pad 21: unconnected-(U16-MO-Pad21) -> /Video_Audio/Audio_analog/SD
- U16 pad 23: unconnected-(U16-fSY-Pad23) -> /Video_Audio/Audio_analog/fl
- U2 pad 35: /PHI2 -> unconnected-(U2-P35-Pad35)
- U7 pad 1: (no net) -> Net-(U29-OEb)
- U7 pad 2: (no net) -> Net-(Port1-P6)
- U7 pad 3: (no net) -> /Joysticks/J_Fire
- U7 pad 4: (no net) -> Net-(U29-OEa)
- U7 pad 5: (no net) -> Net-(Port2-P6)
- U7 pad 6: (no net) -> /Joysticks/J_Fire
- U9 pad 1: Net-(U15-VDD) -> Net-(U15-VSS)
Routing:
- net /~{RESET}: track 312.7 -> 101.8 mm, vias 1 -> 0
- net /CPU_D5: track 180.5 -> 0.00 mm
- net /PHI2: track 192.6 -> 25.6 mm, vias 1 -> 0
- net /CPU_D2: track 166.3 -> 0.00 mm, vias 2 -> 0
- net /CPU_D4: track 165.0 -> 0.00 mm
- net /CPU_D7: track 157.2 -> 0.00 mm
- net /CPU_D3: track 148.5 -> 0.00 mm, vias 1 -> 0
- net /CPU_D0: track 148.1 -> 0.00 mm
- net /CPU_D6: track 146.7 -> 0.00 mm, vias 1 -> 0
- net /CPU_D1: track 145.4 -> 0.00 mm, vias 1 -> 0
- net /~{OE}: track 144.9 -> 0.00 mm, vias 2 -> 0
- net /BUF_D0: track 143.7 -> 0.00 mm, vias 1 -> 0
- net /CPU_A0: track 156.1 -> 15.8 mm, vias 1 -> 0
- net /CPU_RDY: track 131.3 -> 0.00 mm
- net /~{CS_VIA}: track 126.9 -> 0.00 mm, vias 1 -> 0
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Other:
- board size 299.7 x 159.4 mm -> 238.1 x 142.2 mm
- board text added: "BANK0"
- board text added: "BANK1"
- board text added: "EXT"

Commit message: io area relayout
Parts:
- added BT1: BATTERY, Battery:Battery_Panasonic_CR2032-VS1N_Vertical_CircularHoles, F.Cu at (98.0, 99.5)
- added U30: DS1306, Package_DIP:DIP-16_W7.62mm_LongPads, F.Cu at (110.5, 110.5)
- added X4: CRYSTAL_SMD, Crystal:Crystal_Round_D3.0mm_Vertical, F.Cu at (102.9, 105.4)
- P3: footprint Connector_PinHeader_2.54mm:PinHeader_2x03_P2.54mm_Horizontal -> Connector_PinHeader_2.54mm:PinHeader_2x03_P2.54mm_Vertical
- SW1: footprint Button_Switch_THT:Push_E-Switch_KS01Q01 -> Button_Switch_THT:SW_SPST_Omron_B3F-315x_Angled
- moved C3 186.8 mm to (167.6, 154.9)
- moved SW1 123.4 mm to (90.8, 66.7)
- moved J1 121.8 mm to (276.2, 79.0), turned to 90 degrees
- moved Port1 101.5 mm to (79.2, 177.3), turned to -90 degrees
- moved C18 94.9 mm to (262.4, 86.4)
- moved CON1 89.5 mm to (259.1, 77.1)
- moved Port2 84.3 mm to (79.2, 141.8), turned to -90 degrees
- moved RR1 79.2 mm to (86.4, 165.1), turned to -90 degrees
- moved U17 76.8 mm to (161.9, 150.5)
- moved R41 68.5 mm to (83.8, 148.6), turned to -90 degrees
- moved U9 65.7 mm to (106.0, 85.7), turned to -90 degrees
- moved R42 64.7 mm to (86.4, 148.6), turned to -90 degrees
- moved U29 64.7 mm to (130.8, 163.8), turned to -90 degrees
- moved X2 61.6 mm to (164.5, 135.3), turned to 180 degrees
- moved C24 60.3 mm to (83.2, 91.4)
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Connections:
- RR1 pad 2: Net-(U29-I0b) -> Net-(U29-I1a)
- RR1 pad 3: Net-(Port1-P6) -> Net-(U29-I2a)
- RR1 pad 4: Net-(U29-I1b) -> Net-(U29-I3a)
- RR1 pad 5: Net-(U29-I2b) -> Net-(U29-I0b)
- RR1 pad 6: Net-(U29-I3b) -> Net-(Port1-P6)
- RR1 pad 7: Net-(U29-I1a) -> Net-(U29-I1b)
- RR1 pad 8: Net-(U29-I2a) -> Net-(U29-I2b)
- U28 pad 1: /Joysticks/JOYPORT_SELECT -> /PA7
- U28 pad 11: (no net) -> Net-(U30-CE)
- U28 pad 12: (no net) -> /~{SPI_SS1}
- U28 pad 13: (no net) -> /~{SPI_SS1}
- U28 pad 2: /Joysticks/JOYPORT_SELECT -> /PA7
- U28 pad 4: /Joysticks/JOYPORT_SELECT -> /PA7
- U28 pad 5: /Joysticks//JOYPORT_ENABLE -> /~{JOYPORT_ENABLE}
- U28 pad 9: /Joysticks//JOYPORT_ENABLE -> /~{JOYPORT_ENABLE}
- U29 pad 12: /Joysticks/J_Right -> /PA3
- U29 pad 14: /Joysticks/J_Left -> /PA2
- U29 pad 16: /Joysticks/J_Down -> /PA1
- U29 pad 18: /Joysticks/J_Up -> /PA0
- U29 pad 3: /Joysticks/J_Right -> /PA3
- U29 pad 5: /Joysticks/J_Left -> /PA2
- U29 pad 7: /Joysticks/J_Down -> /PA1
- U29 pad 9: /Joysticks/J_Up -> /PA0
- U6 pad 38: unconnected-(U6-~{OUT1}-Pad38) -> /~{JOYPORT_ENABLE}
- U7 pad 3: /Joysticks/J_Fire -> /PA4
- U7 pad 6: /Joysticks/J_Fire -> /PA4
Routing:
- net /~{IRQ}: track 110.6 -> 0.00 mm
- net /~{RESET}: track 101.8 -> 3.74 mm
- net /~{WE}: track 115.1 -> 21.7 mm, vias 1 -> 0
- net /CPU_R~{W}: track 86.9 -> 0.00 mm
- net Net-(U11-PB6): track 73.6 -> 0.00 mm
- net Net-(U11-CA2): track 72.5 -> 0.00 mm
- net Net-(U11-CA1): track 70.0 -> 0.00 mm
- net /SD Card/DAT0: track 69.6 -> 0.00 mm
- net /BUF_A0: track 67.8 -> 0.00 mm
- net Net-(U11-PA6): track 67.5 -> 0.00 mm
- net /SPI_MOSI: track 66.0 -> 0.00 mm
- net Net-(U6-MR): track 65.1 -> 0.00 mm, vias 2 -> 0
- net /SPI_CLK: track 64.6 -> 0.00 mm
- net /~{SPI_SS1}: track 64.0 -> 0.00 mm
- net Net-(U11-PA0): track 62.8 -> 0.00 mm
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
Commit message: pinout expansion slot
Connections:
- SLOT0 pad 12: /BUF_PHI2 -> /~{BUF_WE}
- SLOT0 pad 14: unconnected-(SLOT0-Pin_14-Pad14) -> /~{BUF_OE}
- SLOT0 pad 17: unconnected-(SLOT0-Pin_17-Pad17) -> /~{IRQ}
- SLOT0 pad 18: unconnected-(SLOT0-Pin_18-Pad18) -> /~{NMI}
- SLOT0 pad 19: unconnected-(SLOT0-Pin_19-Pad19) -> /CPU_RDY
- SLOT0 pad 20: unconnected-(SLOT0-Pin_20-Pad20) -> /BUF_PHI2
- SLOT0 pad 21: unconnected-(SLOT0-Pin_21-Pad21) -> /~{RESET}
- SLOT0 pad 22: unconnected-(SLOT0-Pin_22-Pad22) -> /RESET_TRIG
- SLOT1 pad 12: /BUF_PHI2 -> /~{BUF_WE}
- SLOT1 pad 14: unconnected-(SLOT1-Pin_14-Pad14) -> /~{BUF_OE}
- SLOT1 pad 17: unconnected-(SLOT1-Pin_17-Pad17) -> /~{IRQ}
- SLOT1 pad 18: unconnected-(SLOT1-Pin_18-Pad18) -> /~{NMI}
- SLOT1 pad 19: unconnected-(SLOT1-Pin_19-Pad19) -> /CPU_RDY
- SLOT1 pad 20: unconnected-(SLOT1-Pin_20-Pad20) -> /BUF_PHI2
- SLOT1 pad 21: unconnected-(SLOT1-Pin_21-Pad21) -> /~{RESET}
- SLOT1 pad 22: unconnected-(SLOT1-Pin_22-Pad22) -> /RESET_TRIG
