File: kicad/sbc/a_analog.kicad_sch (KiCad schematic)
At the start: 14 parts, among them J1 Audio, U10 Y3014B, U11 LM324

Commit message: routing
Parts:
- removed J1: Audio, Connector_Audio:Jack_3.5mm_Lumberg_1503_07_Horizontal, symbol v9958-rescue:Conn_Coaxial
- added J3: AudioJack3, Connector_Audio:Jack_3.5mm_Lumberg_1503_07_Horizontal, symbol Connector_Audio:AudioJack3
- added U11: LM324, Package_DIP:DIP-14_W7.62mm_LongPads, symbol Amplifier_Operational:LM324
- C11, C14, C32: symbol v9958-rescue:CP -> Device:C_Polarized
- C12, C13: symbol v9958-rescue:C -> Device:C
- R1, R2, R3, R4, R5, R6: symbol v9958-rescue:R-RESCUE-v9958 -> Device:R
- U10: symbol v9958-rescue:Y3014B -> yamaha_opl:Y3014B
- U11: symbol v9958-rescue:LM324 -> Amplifier_Operational:LM324
Connections:
- net AUDIO_OUT: now also J3.R, J3.S
- net GND: now also J3.T; no longer U11.11 (V-), U11.11 (V-), U11.11 (V-), U11.11 (V-)
- net VCC: no longer U11.4 (V+), U11.4 (V+), U11.4 (V+)

Commit message: moved all symbols into custom library
Parts:
- C11, C14: footprint Capacitor_THT:CP_Radial_D5.0mm_P2.50mm -> Capacitor_THT:CP_Radial_D10.0mm_P5.00mm; symbol Device:C_Polarized -> steckschwein:C_Polarized
- C12, C13: footprint Capacitor_THT:C_Disc_D3.0mm_W2.0mm_P2.50mm -> Capacitor_SMD:C_1206_3216Metric_Pad1.33x1.80mm_HandSolder; symbol Device:C -> steckschwein:C
- C32: footprint Capacitor_THT:CP_Radial_D4.0mm_P2.00mm -> Capacitor_THT:CP_Radial_D10.0mm_P5.00mm; symbol Device:C_Polarized -> steckschwein:C_Polarized
- J3: symbol Connector_Audio:AudioJack3 -> steckschwein:AudioJack3
- R1, R2, R3, R4, R5, R6: symbol Device:R -> steckschwein:R
- U10: symbol yamaha_opl:Y3014B -> steckschwein:Y3014B
- U11: symbol Amplifier_Operational:LM324 -> steckschwein:LM324
Changed lines of the file:
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@@
     (effects (font (size 1.524 1.524)) (justify right))
   )
-  (symbol (lib_id "Device:R") (at 168.91 104.14 90) (unit 1)
+  (symbol (lib_id "steckschwein:R") (at 168.91 104.14 90) (unit 1)
     (in_bom yes) (on_board yes) (dnp no)
     (property "Reference" "R4" (at 168.91 102.108 90)
@@
     )
     (property "Footprint" "Resistor_THT:R_Axial_DIN0204_L3.6mm_D1.6mm_P5.08mm_Horizontal" (at 168.91 105.918 90)
-      (effects (font (size 1.27 1.27)) hide)
+      (effects (font (size 0.762 0.762)) hide)
     )
     (property "Datasheet" "~" (at 168.91 104.14 0)
-      (effects (font (size 1.27 1.27)) hide)
+      (effects (font (size 0.762 0.762)))
     )
     (pin "1")
@@
     )
   )
-  (symbol (lib_id "Connector_Audio:AudioJack3") (at 250.19 107.95 180) (unit 1)
+  (symbol (lib_id "steckschwein:AudioJack3") (at 250.19 107.95 180) (unit 1)
     (in_bom yes) (on_board yes) (dnp no) (fields_autoplaced)
     (property "Reference" "J3" (at 257.302 106.6713 0)
@@
     )
   )
-  (symbol (lib_id "Device:R") (at 144.78 73.66 90) (unit 1)
+  (symbol (lib_id "steckschwein:R") (at 144.78 73.66 90) (unit 1)
     (in_bom yes) (on_board yes) (dnp no)
     (property "Reference" "R3" (at 144.78 71.628 90)
@@
     )
     (property "Footprint" "Resistor_THT:R_Axial_DIN0204_L3.6mm_D1.6mm_P5.08mm_Horizontal" (at 144.78 75.438 90)
-      (effects (font (size 1.27 1.27)) hide)
+      (effects (font (size 0.762 0.762)) hide)
     )
     (property "Datasheet" "~" (at 144.78 73.66 0)
-      (effects (font (size 1.27 1.27)) hide)
+      (effects (font (size 0.762 0.762)))
     )
     (pin "1")
@@
     )
   )
-  (symbol (lib_id "Device:R") (at 193.04 115.57 90) (unit 1)
+  (symbol (lib_id "steckschwein:R") (at 193.04 115.57 90) (unit 1)
     (in_bom yes) (on_board yes) (dnp no)
     (property "Reference" "R5" (at 193.04 113.538 90)
@@
     )
     (property "Footprint" "Resistor_THT:R_Axial_DIN0204_L3.6mm_D1.6mm_P5.08mm_Horizontal" (at 193.04 117.348 90)
-      (effects (font (size 1.27 1.27)) hide)
+      (effects (font (size 0.762 0.762)) hide)
     )
     (property "Datasheet" "~" (at 193.04 115.57 0)
-      (effects (font (size 1.27 1.27)) hide)
+      (effects (font (size 0.762 0.762)))
     )
     (pin "1")
@@
     )
   )
-  (symbol (lib_id "Device:C") (at 157.48 60.96 270) (unit 1)
+  (symbol (lib_id "steckschwein:C") (at 157.48 60.96 270) (unit 1)
     (in_bom yes) (on_board yes) (dnp no)
     (property "Reference" "C13" (at 160.02 61.595 0)
@@
       (effects (font (size 1.27 1.27)) (justify left))
     )
-    (property "Footprint" "Capacitor_THT:C_Disc_D3.0mm_W2.0mm_P2.50mm" (at 153.67 61.9252 0)
-      (effects (font (size 1.27 1.27)) hide)
+    (property "Footprint" "Capacitor_SMD:C_1206_3216Metric_Pad1.33x1.80mm_HandSolder" (at 153.67 61.9252 0)
+      (effects (font (size 0.762 0.762)) hide)
     )
     (property "Datasheet" "~" (at 157.48 60.96 0)
-      (effects (font (size 1.27 1.27)) hide)
+      (effects (font (size 1.524 1.524)))
     )
     (pin "1")
@@
     )
   )
-  (symbol (lib_id "Device:R") (at 223.52 123.19 180) (unit 1)
+  (symbol (lib_id "steckschwein:R") (at 223.52 123.19 180) (unit 1)
     (in_bom yes) (on_board yes) (dnp no)
     (property "Reference" "R6" (at 221.488 123.19 90)
@@
     )
     (property "Footprint" "Resistor_THT:R_Axial_DIN0204_L3.6mm_D1.6mm_P5.08mm_Horizontal" (at 225.298 123.19 90)
-      (effects (font (size 1.27 1.27)) hide)
+      (effects (font (size 0.762 0.762)) hide)
     )
     (property "Datasheet" "~" (at 223.52 123.19 0)
-      (effects (font (size 1.27 1.27)) hide)
+      (effects (font (size 0.762 0.762)))
     )
     (pin "1")
@@
     )
   )
-  (symbol (lib_id "Device:C_Polarized") (at 100.33 107.95 0) (unit 1)
+  (symbol (lib_id "steckschwein:C_Polarized") (at 100.33 107.95 0) (unit 1)
     (in_bom yes) (on_board yes) (dnp no)
     (property "Reference" "C11" (at 100.965 105.41 0)
@@
       (effects (font (size 1.27 1.27)) (justify left))
     )
-    (property "Footprint" "Capacitor_THT:CP_Radial_D5.0mm_P2.50mm" (at 101.2952 111.76 0)
+    (property "Footprint" "Capacitor_THT:CP_Radial_D10.0mm_P5.00mm" (at 101.2952 111.76 0)
       (effects (font (size 1.27 1.27)) hide)
     )
@@
     )
   )
-  (symbol (lib_id "Device:C_Polarized") (at 66.04 148.59 0) (unit 1)
+  (symbol (lib_id "steckschwein:C_Polarized") (at 66.04 148.59 0) (unit 1)
     (in_bom yes) (on_board yes) (dnp no)
     (property "Reference" "C32" (at 66.675 146.05 0)
@@
       (effects (font (size 1.27 1.27)) (justify left))
     )
-    (property "Footprint" "Capacitor_THT:CP_Radial_D4.0mm_P2.00mm" (at 67.0052 152.4 0)
+    (property "Footprint" "Capacitor_THT:CP_Radial_D10.0mm_P5.00mm" (at 67.0052 152.4 0)
       (effects (font (size 1.27 1.27)) hide)
     )
@@
     )
   )
-  (symbol (lib_id "Device:C") (at 153.67 82.55 180) (unit 1)
+  (symbol (lib_id "steckschwein:C") (at 153.67 82.55 180) (unit 1)
     (in_bom yes) (on_board yes) (dnp no)
     (property "Reference" "C12" (at 153.035 85.09 0)
@@
       (effects (font (size 1.27 1.27)) (justify left))
     )
-    (property "Footprint" "Capacitor_THT:C_Disc_D3.0mm_W2.0mm_P2.50mm" (at 152.7048 78.74 0)
-      (effects (font (size 1.27 1.27)) hide)
+    (property "Footprint" "Capacitor_SMD:C_1206_3216Metric_Pad1.33x1.80mm_HandSolder" (at 152.7048 78.74 0)
+      (effects (font (size 0.762 0.762)) hide)
     )
     (property "Datasheet" "~" (at 153.67 82.55 0)
-      (effects (font (size 1.27 1.27)) hide)
+      (effects (font (size 1.524 1.524)))
     )
     (pin "1")
@@
     )
   )
-  (symbol (lib_id "Amplifier_Operational:LM324") (at 111.76 73.66 0) (unit 1)
+  (symbol (lib_id "steckschwein:LM324") (at 111.76 73.66 0) (unit 1)
     (in_bom yes) (on_board yes) (dnp no)
     (property "Reference" "U11" (at 111.76 68.58 0)
@@
     )
   )
-  (symbol (lib_id "Device:R") (at 129.54 113.03 180) (unit 1)
+  (symbol (lib_id "steckschwein:R") (at 129.54 113.03 180) (unit 1)
     (in_bom yes) (on_board yes) (dnp no)
     (property "Reference" "R2" (at 127.508 113.03 90)
@@
     )
     (property "Footprint" "Resistor_THT:R_Axial_DIN0204_L3.6mm_D1.6mm_P5.08mm_Horizontal" (at 131.318 113.03 90)
-      (effects (font (size 1.27 1.27)) hide)
+      (effects (font (size 0.762 0.762)) hide)
     )
     (property "Datasheet" "~" (at 129.54 113.03 0)
-      (effects (font (size 1.27 1.27)) hide)
+      (effects (font (size 0.762 0.762)))
     )
     (pin "1")
@@
     )
   )
-  (symbol (lib_id "yamaha_opl:Y3014B") (at 80.01 88.9 0) (unit 1)
+  (symbol (lib_id "steckschwein:Y3014B") (at 80.01 88.9 0) (unit 1)
     (in_bom yes) (on_board yes) (dnp no)
     (property "Reference" "U10" (at 80.01 87.63 0)
@@
     )
   )
-  (symbol (lib_id "Device:R") (at 129.54 73.66 90) (unit 1)
+  (symbol (lib_id "steckschwein:R") (at 129.54 73.66 90) (unit 1)
     (in_bom yes) (on_board yes) (dnp no)
     (property "Reference" "R1" (at 129.54 71.628 90)
@@
     )
     (property "Footprint" "Resistor_THT:R_Axial_DIN0204_L3.6mm_D1.6mm_P5.08mm_Horizontal" (at 129.54 75.438 90)
-      (effects (font (size 1.27 1.27)) hide)
+      (effects (font (size 0.762 0.762)) hide)
     )
     (property "Datasheet" "~" (at 129.54 73.66 0)
-      (effects (font (size 1.27 1.27)) hide)
+      (effects (font (size 0.762 0.762)))
     )
     (pin "1")
@@
     )
   )
-  (symbol (lib_id "Device:C_Polarized") (at 233.68 101.6 90) (unit 1)
+  (symbol (lib_id "steckschwein:C_Polarized") (at 233.68 101.6 90) (unit 1)
     (in_bom yes) (on_board yes) (dnp no)
     (property "Reference" "C14" (at 231.14 100.965 0)
@@
       (effects (font (size 1.27 1.27)) (justify left))
     )
-    (property "Footprint" "Capacitor_THT:CP_Radial_D5.0mm_P2.50mm" (at 237.49 100.6348 0)
-      (effects (font (size 1.27 1.27)) hide)
-    )
+    (property "Footprint" "Capacitor_THT:CP_Radial_D10.0mm_P5.00mm" (at 237.49 100.6348 0)
+      (effects (font (size 1.27 1.27)) hide)
+    )

Commit message: moved all footprints into local library
Parts:
- C11, C14: footprint Capacitor_THT:CP_Radial_D10.0mm_P5.00mm -> steckschwein:CP_Radial_D5.0mm_P2.50mm
- C12, C13: footprint Capacitor_SMD:C_1206_3216Metric_Pad1.33x1.80mm_HandSolder -> steckschwein:C_Disc_D3.0mm_W2.0mm_P2.50mm
- C32: footprint Capacitor_THT:CP_Radial_D10.0mm_P5.00mm -> steckschwein:CP_Radial_D4.0mm_P2.00mm
- J3: footprint Connector_Audio:Jack_3.5mm_Lumberg_1503_07_Horizontal -> steckschwein:Jack_3.5mm_Lumberg_1503_07_Horizontal
- R1, R2, R3, R4, R5, R6: footprint Resistor_THT:R_Axial_DIN0204_L3.6mm_D1.6mm_P5.08mm_Horizontal -> steckschwein:R_Axial_DIN0204_L3.6mm_D1.6mm_P7.62mm_Horizontal
- U10: footprint Package_DIP:DIP-8_W7.62mm_LongPads -> steckschwein:DIP-8_W7.62mm_LongPads
- U11: footprint Package_DIP:DIP-14_W7.62mm_LongPads -> steckschwein:DIP-14_W7.62mm_LongPads
Changed lines of the file:
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@@
       (effects (font (size 1.016 1.016)))
     )
-    (property "Footprint" "Resistor_THT:R_Axial_DIN0204_L3.6mm_D1.6mm_P5.08mm_Horizontal" (at 168.91 105.918 90)
+    (property "Footprint" "steckschwein:R_Axial_DIN0204_L3.6mm_D1.6mm_P7.62mm_Horizontal" (at 168.91 105.918 90)
       (effects (font (size 0.762 0.762)) hide)
     )
@@
       (effects (font (size 1.27 1.27)) (justify right))
     )
-    (property "Footprint" "Connector_Audio:Jack_3.5mm_Lumberg_1503_07_Horizontal" (at 250.19 107.95 0)
+    (property "Footprint" "steckschwein:Jack_3.5mm_Lumberg_1503_07_Horizontal" (at 250.19 107.95 0)
       (effects (font (size 1.27 1.27)) hide)
     )
@@
       (effects (font (size 1.27 1.27)) (justify left))
     )
-    (property "Footprint" "Package_DIP:DIP-14_W7.62mm_LongPads" (at 203.2 99.06 0)
+    (property "Footprint" "steckschwein:DIP-14_W7.62mm_LongPads" (at 203.2 99.06 0)
       (effects (font (size 1.27 1.27)) hide)
     )
@@
       (effects (font (size 1.016 1.016)))
     )
-    (property "Footprint" "Resistor_THT:R_Axial_DIN0204_L3.6mm_D1.6mm_P5.08mm_Horizontal" (at 144.78 75.438 90)
+    (property "Footprint" "steckschwein:R_Axial_DIN0204_L3.6mm_D1.6mm_P7.62mm_Horizontal" (at 144.78 75.438 90)
       (effects (font (size 0.762 0.762)) hide)
     )
@@
       (effects (font (size 1.016 1.016)))
     )
-    (property "Footprint" "Resistor_THT:R_Axial_DIN0204_L3.6mm_D1.6mm_P5.08mm_Horizontal" (at 193.04 117.348 90)
+    (property "Footprint" "steckschwein:R_Axial_DIN0204_L3.6mm_D1.6mm_P7.62mm_Horizontal" (at 193.04 117.348 90)
       (effects (font (size 0.762 0.762)) hide)
     )
@@
       (effects (font (size 1.27 1.27)) (justify left))
     )
-    (property "Footprint" "Package_DIP:DIP-14_W7.62mm_LongPads" (at 81.28 146.05 0)
+    (property "Footprint" "steckschwein:DIP-14_W7.62mm_LongPads" (at 81.28 146.05 0)
       (effects (font (size 1.27 1.27)) hide)
     )
@@
       (effects (font (size 1.27 1.27)) (justify left))
     )
-    (property "Footprint" "Capacitor_SMD:C_1206_3216Metric_Pad1.33x1.80mm_HandSolder" (at 153.67 61.9252 0)
+    (property "Footprint" "steckschwein:C_Disc_D3.0mm_W2.0mm_P2.50mm" (at 153.67 61.9252 0)
       (effects (font (size 0.762 0.762)) hide)
     )
@@
       (effects (font (size 1.016 1.016)))
     )
-    (property "Footprint" "Resistor_THT:R_Axial_DIN0204_L3.6mm_D1.6mm_P5.08mm_Horizontal" (at 225.298 123.19 90)
+    (property "Footprint" "steckschwein:R_Axial_DIN0204_L3.6mm_D1.6mm_P7.62mm_Horizontal" (at 225.298 123.19 90)
       (effects (font (size 0.762 0.762)) hide)
     )
@@
       (effects (font (size 1.27 1.27)) (justify left))
     )
-    (property "Footprint" "Capacitor_THT:CP_Radial_D10.0mm_P5.00mm" (at 101.2952 111.76 0)
+    (property "Footprint" "steckschwein:CP_Radial_D5.0mm_P2.50mm" (at 101.2952 111.76 0)
       (effects (font (size 1.27 1.27)) hide)
     )
@@
       (effects (font (size 1.27 1.27)) (justify left))
     )
-    (property "Footprint" "Package_DIP:DIP-14_W7.62mm_LongPads" (at 167.64 73.66 0)
+    (property "Footprint" "steckschwein:DIP-14_W7.62mm_LongPads" (at 167.64 73.66 0)
       (effects (font (size 1.27 1.27)) hide)
     )
@@
       (effects (font (size 1.27 1.27)) (justify left))
     )
-    (property "Footprint" "Package_DIP:DIP-14_W7.62mm_LongPads" (at 113.03 101.6 0)
+    (property "Footprint" "steckschwein:DIP-14_W7.62mm_LongPads" (at 113.03 101.6 0)
       (effects (font (size 1.27 1.27)) hide)
     )
@@
       (effects (font (size 1.27 1.27)) (justify left))
     )
-    (property "Footprint" "Capacitor_THT:CP_Radial_D10.0mm_P5.00mm" (at 67.0052 152.4 0)
+    (property "Footprint" "steckschwein:CP_Radial_D4.0mm_P2.00mm" (at 67.0052 152.4 0)
       (effects (font (size 1.27 1.27)) hide)
     )
@@
       (effects (font (size 1.27 1.27)) (justify left))
     )
-    (property "Footprint" "Capacitor_SMD:C_1206_3216Metric_Pad1.33x1.80mm_HandSolder" (at 152.7048 78.74 0)
+    (property "Footprint" "steckschwein:C_Disc_D3.0mm_W2.0mm_P2.50mm" (at 152.7048 78.74 0)
       (effects (font (size 0.762 0.762)) hide)
     )
@@
       (effects (font (size 1.27 1.27)) (justify left))
     )
-    (property "Footprint" "Package_DIP:DIP-14_W7.62mm_LongPads" (at 110.49 71.12 0)
+    (property "Footprint" "steckschwein:DIP-14_W7.62mm_LongPads" (at 110.49 71.12 0)
       (effects (font (size 1.27 1.27)) hide)
     )
@@
       (effects (font (size 1.016 1.016)))
     )
-    (property "Footprint" "Resistor_THT:R_Axial_DIN0204_L3.6mm_D1.6mm_P5.08mm_Horizontal" (at 131.318 113.03 90)
+    (property "Footprint" "steckschwein:R_Axial_DIN0204_L3.6mm_D1.6mm_P7.62mm_Horizontal" (at 131.318 113.03 90)
       (effects (font (size 0.762 0.762)) hide)
     )
@@
       (effects (font (size 1.524 1.524)))
     )
-    (property "Footprint" "Package_DIP:DIP-8_W7.62mm_LongPads" (at 80.01 88.9 0)
+    (property "Footprint" "steckschwein:DIP-8_W7.62mm_LongPads" (at 80.01 88.9 0)
       (effects (font (size 1.524 1.524)) hide)
     )
@@
       (effects (font (size 1.016 1.016)))
     )
-    (property "Footprint" "Resistor_THT:R_Axial_DIN0204_L3.6mm_D1.6mm_P5.08mm_Horizontal" (at 129.54 75.438 90)
+    (property "Footprint" "steckschwein:R_Axial_DIN0204_L3.6mm_D1.6mm_P7.62mm_Horizontal" (at 129.54 75.438 90)
       (effects (font (size 0.762 0.762)) hide)
     )
@@
       (effects (font (size 1.27 1.27)) (justify left))
     )
-    (property "Footprint" "Capacitor_THT:CP_Radial_D10.0mm_P5.00mm" (at 237.49 100.6348 0)
-      (effects (font (size 1.27 1.27)) hide)
-    )
+    (property "Footprint" "steckschwein:CP_Radial_D5.0mm_P2.50mm" (at 237.49 100.6348 0)
+      (effects (font (size 1.27 1.27)) hide)
+    )
