File: kicad/sbc/rtc.kicad_sch (KiCad schematic)
At the start: 4 parts, among them U28 7400, U30 DS1306, X4 CRYSTAL_SMD

Commit message: routing
Parts:
- BT1: footprint Battery:Battery_Panasonic_CR2032-VS1N_Vertical_CircularHoles -> Battery:BatteryHolder_Keystone_103_1x20mm; symbol io-rescue:Battery -> Device:Battery_Cell
- U28: symbol io-rescue:7400 -> 74xx:7400
- U30: symbol io-rescue:DS1306-RESCUE-io -> dallas-rtc:DS1306
- X4: symbol io-rescue:Crystal -> Device:Crystal_Small
Connections:
- net GND: no longer U28.7 (GND)
- net VCC: no longer U28.14 (VCC)
Changed lines of the file:
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@@
     (stroke (width 0) (type default))
   )
-  (wire (pts (xy 107.95 85.09) (xy 110.49 85.09))
-    (stroke (width 0) (type default))
-  )
-  (wire (pts (xy 149.86 105.41) (xy 161.29 105.41))
+  (wire (pts (xy 107.95 85.09) (xy 111.76 85.09))
+    (stroke (width 0) (type default))
+  )
+  (wire (pts (xy 149.86 105.41) (xy 176.53 105.41))
     (stroke (width 0) (type default))
   )
@@
     (stroke (width 0) (type default))
   )
-  (wire (pts (xy 118.11 85.09) (xy 119.38 85.09))
+  (wire (pts (xy 116.84 85.09) (xy 119.38 85.09))
     (stroke (width 0) (type default))
   )
@@
     (effects (font (size 1.524 1.524)) (justify left))
   )
-  (symbol (lib_id "io-rescue:DS1306-RESCUE-io") (at 134.62 92.71 0) (unit 1)
+  (symbol (lib_id "dallas-rtc:DS1306") (at 134.62 92.71 0) (unit 1)
     (in_bom yes) (on_board yes) (dnp no)
     (property "Reference" "U30" (at 124.46 72.39 0)
@@
     )
   )
-  (symbol (lib_id "io-rescue:GND") (at 100.33 115.57 0) (unit 1)
+  (symbol (lib_id "power:GND") (at 100.33 115.57 0) (unit 1)
     (in_bom yes) (on_board yes) (dnp no)
     (property "Reference" "#PWR072" (at 100.33 115.57 0)
@@
     )
     (property "Footprint" "" (at 100.33 115.57 0)
-      (effects (font (size 1.524 1.524)))
+      (effects (font (size 1.27 1.27)) hide)
     )
     (property "Datasheet" "" (at 100.33 115.57 0)
-      (effects (font (size 1.524 1.524)))
+      (effects (font (size 1.27 1.27)) hide)
     )
     (pin "1")
@@
     )
   )
-  (symbol (lib_id "io-rescue:VCC") (at 154.94 69.85 0) (unit 1)
+  (symbol (lib_id "power:VCC") (at 154.94 69.85 0) (unit 1)
     (in_bom yes) (on_board yes) (dnp no)
     (property "Reference" "#PWR073" (at 154.94 67.31 0)
@@
     )
     (property "Footprint" "" (at 154.94 69.85 0)
+      (effects (font (size 1.27 1.27)) hide)
+    )
+    (property "Datasheet" "" (at 154.94 69.85 0)
+      (effects (font (size 1.27 1.27)) hide)
+    )
+    (pin "1")
+    (instances
+      (project "sbc"
+        (path "/896d5dab-44ec-47d0-8232-7ef57773545e/fe2f3103-6209-4021-9455-fda781985721"
+          (reference "#PWR073") (unit 1)
+        )
+      )
+      (project "io"
+        (path "/dd492dee-3ed3-48c7-8a89-2dc679fadc05/00000000-0000-0000-0000-000058e79100"
+          (reference "#PWR039") (unit 1)
+        )
+      )
+    )
+  )
+  (symbol (lib_id "Device:Battery_Cell") (at 109.22 80.01 270) (unit 1)
+    (in_bom yes) (on_board yes) (dnp no)
+    (property "Reference" "BT1" (at 114.3 80.01 0)
+      (effects (font (size 1.27 1.27)))
+    )
+    (property "Value" "BATTERY" (at 104.394 80.01 0)
+      (effects (font (size 1.27 1.27)))
+    )
+    (property "Footprint" "Battery:BatteryHolder_Keystone_103_1x20mm" (at 110.744 80.01 90)
+      (effects (font (size 1.27 1.27)) hide)
+    )
+    (property "Datasheet" "~" (at 110.744 80.01 90)
+      (effects (font (size 1.27 1.27)) hide)
+    )
+    (pin "1")
+    (pin "2")
+    (instances
+      (project "sbc"
+        (path "/896d5dab-44ec-47d0-8232-7ef57773545e/fe2f3103-6209-4021-9455-fda781985721"
+          (reference "BT1") (unit 1)
+        )
+      )
+      (project "io"
+        (path "/dd492dee-3ed3-48c7-8a89-2dc679fadc05/00000000-0000-0000-0000-000058e79100"
+          (reference "BT1") (unit 1)
+        )
+      )
+    )
+  )
+  (symbol (lib_id "74xx:7400") (at 184.15 105.41 180) (unit 4)
+    (in_bom yes) (on_board yes) (dnp no)
+    (property "Reference" "U28" (at 184.15 106.68 0)
       (effects (font (size 1.524 1.524)))
     )
-    (property "Datasheet" "" (at 154.94 69.85 0)
+    (property "Value" "7400" (at 184.15 102.87 0)
       (effects (font (size 1.524 1.524)))
     )
-    (pin "1")
-    (instances
-      (project "sbc"
-        (path "/896d5dab-44ec-47d0-8232-7ef57773545e/fe2f3103-6209-4021-9455-fda781985721"
-          (reference "#PWR073") (unit 1)
-        )
-      )
-      (project "io"
-        (path "/dd492dee-3ed3-48c7-8a89-2dc679fadc05/00000000-0000-0000-0000-000058e79100"
-          (reference "#PWR039") (unit 1)
-        )
-      )
-    )
-  )
-  (symbol (lib_id "io-rescue:Battery") (at 110.49 80.01 270) (unit 1)
-    (in_bom yes) (on_board yes) (dnp no)
-    (property "Reference" "BT1" (at 115.57 80.01 0)
-      (effects (font (size 1.27 1.27)))
-    )
-    (property "Value" "BATTERY" (at 105.664 80.01 0)
-      (effects (font (size 1.27 1.27)))
-    )
-    (property "Footprint" "Battery:Battery_Panasonic_CR2032-VS1N_Vertical_CircularHoles" (at 110.49 80.01 0)
-      (effects (font (size 1.524 1.524)) hide)
-    )
-    (property "Datasheet" "" (at 110.49 80.01 0)
-      (effects (font (size 1.524 1.524)))
-    )
-    (pin "1")
-    (pin "2")
-    (instances
-      (project "sbc"
-        (path "/896d5dab-44ec-47d0-8232-7ef57773545e/fe2f3103-6209-4021-9455-fda781985721"
-          (reference "BT1") (unit 1)
-        )
-      )
-      (project "io"
-        (path "/dd492dee-3ed3-48c7-8a89-2dc679fadc05/00000000-0000-0000-0000-000058e79100"
-          (reference "BT1") (unit 1)
-        )
-      )
-    )
-  )
-  (symbol (lib_id "io-rescue:7400") (at 176.53 105.41 180) (unit 4)
-    (in_bom yes) (on_board yes) (dnp no)
-    (property "Reference" "U28" (at 176.53 106.68 0)
-      (effects (font (size 1.524 1.524)))
-    )
-    (property "Value" "7400" (at 176.53 102.87 0)
-      (effects (font (size 1.524 1.524)))
-    )
-    (property "Footprint" "Package_DIP:DIP-14_W7.62mm_LongPads" (at 176.53 105.41 0)
-      (effects (font (size 1.524 1.524)) hide)
-    )
-    (property "Datasheet" "" (at 176.53 105.41 0)
-      (effects (font (size 1.524 1.524)))
-    )
-    (pin "14")
-    (pin "7")
+    (property "Footprint" "Package_DIP:DIP-14_W7.62mm_LongPads" (at 184.15 105.41 0)
+      (effects (font (size 1.27 1.27)) hide)
+    )
+    (property "Datasheet" "http://www.ti.com/lit/gpn/sn7400" (at 184.15 105.41 0)
+      (effects (font (size 1.27 1.27)) hide)
+    )
     (pin "1")
     (pin "2")
@@
     (pin "12")
     (pin "13")
+    (pin "14")
+    (pin "7")
     (instances
       (project "sbc"
@@
     )
   )
-  (symbol (lib_id "io-rescue:Crystal") (at 114.3 85.09 0) (unit 1)
+  (symbol (lib_id "Device:Crystal_Small") (at 114.3 85.09 0) (unit 1)
     (in_bom yes) (on_board yes) (dnp no)
     (property "Reference" "X4" (at 114.3 82.804 0)
@@
     )
     (property "Footprint" "Crystal:Crystal_Round_D3.0mm_Vertical" (at 114.3 85.09 0)
-      (effects (font (size 1.524 1.524)) hide)
-    )
-    (property "Datasheet" "" (at 114.3 85.09 0)
-      (effects (font (size 1.524 1.524)))
-    )
-    (pin "1")
+      (effects (font (size 1.27 1.27)) hide)
+    )
+    (property "Datasheet" "~" (at 114.3 85.09 0)
+      (effects (font (size 1.27 1.27)) hide)
+    )
+    (pin "1")

Commit message: moved all symbols into custom library
Parts:
- BT1: symbol Device:Battery_Cell -> steckschwein:Battery_Cell
- U28: symbol 74xx:7400 -> steckschwein:7400
- U30: symbol dallas-rtc:DS1306 -> steckschwein:DS1306
- X4: footprint Crystal:Crystal_Round_D3.0mm_Vertical -> Crystal:Crystal_HC49-U_Vertical; symbol Device:Crystal_Small -> steckschwein:Crystal_Small
Changed lines of the file:
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@@
     (effects (font (size 1.524 1.524)) (justify left))
   )
-  (symbol (lib_id "dallas-rtc:DS1306") (at 134.62 92.71 0) (unit 1)
+  (symbol (lib_id "steckschwein:DS1306") (at 134.62 92.71 0) (unit 1)
     (in_bom yes) (on_board yes) (dnp no)
     (property "Reference" "U30" (at 124.46 72.39 0)
@@
     )
   )
-  (symbol (lib_id "Device:Battery_Cell") (at 109.22 80.01 270) (unit 1)
+  (symbol (lib_id "steckschwein:Battery_Cell") (at 109.22 80.01 270) (unit 1)
     (in_bom yes) (on_board yes) (dnp no)
     (property "Reference" "BT1" (at 114.3 80.01 0)
@@
     )
   )
-  (symbol (lib_id "74xx:7400") (at 184.15 105.41 180) (unit 4)
+  (symbol (lib_id "steckschwein:7400") (at 184.15 105.41 180) (unit 4)
     (in_bom yes) (on_board yes) (dnp no)
     (property "Reference" "U28" (at 184.15 106.68 0)
@@
     )
   )
-  (symbol (lib_id "Device:Crystal_Small") (at 114.3 85.09 0) (unit 1)
+  (symbol (lib_id "steckschwein:Crystal_Small") (at 114.3 85.09 0) (unit 1)
     (in_bom yes) (on_board yes) (dnp no)
     (property "Reference" "X4" (at 114.3 82.804 0)
@@
       (effects (font (size 0.762 0.762)) (justify left))
     )
-    (property "Footprint" "Crystal:Crystal_Round_D3.0mm_Vertical" (at 114.3 85.09 0)
+    (property "Footprint" "Crystal:Crystal_HC49-U_Vertical" (at 114.3 85.09 0)
       (effects (font (size 1.27 1.27)) hide)
     )

Commit message: moved all footprints into local library
Parts:
- BT1: footprint Battery:BatteryHolder_Keystone_103_1x20mm -> steckschwein:BatteryHolder_Keystone_103_1x20mm
- U28: footprint Package_DIP:DIP-14_W7.62mm_LongPads -> steckschwein:DIP-14_W7.62mm_LongPads
- U30: footprint Package_DIP:DIP-16_W7.62mm_LongPads -> steckschwein:DIP-16_W7.62mm_LongPads
- X4: footprint Crystal:Crystal_HC49-U_Vertical -> steckschwein:Crystal_Round_D3.0mm_Vertical
Changed lines of the file:
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@@
       (effects (font (size 1.27 1.27)) (justify left bottom))
     )
-    (property "Footprint" "Package_DIP:DIP-16_W7.62mm_LongPads" (at 134.62 88.9 0)
+    (property "Footprint" "steckschwein:DIP-16_W7.62mm_LongPads" (at 134.62 88.9 0)
       (effects (font (size 1.27 1.27)) hide)
     )
@@
       (effects (font (size 1.27 1.27)))
     )
-    (property "Footprint" "Battery:BatteryHolder_Keystone_103_1x20mm" (at 110.744 80.01 90)
+    (property "Footprint" "steckschwein:BatteryHolder_Keystone_103_1x20mm" (at 110.744 80.01 90)
       (effects (font (size 1.27 1.27)) hide)
     )
@@
       (effects (font (size 1.524 1.524)))
     )
-    (property "Footprint" "Package_DIP:DIP-14_W7.62mm_LongPads" (at 184.15 105.41 0)
+    (property "Footprint" "steckschwein:DIP-14_W7.62mm_LongPads" (at 184.15 105.41 0)
       (effects (font (size 1.27 1.27)) hide)
     )
@@
       (effects (font (size 0.762 0.762)) (justify left))
     )
-    (property "Footprint" "Crystal:Crystal_HC49-U_Vertical" (at 114.3 85.09 0)
+    (property "Footprint" "steckschwein:Crystal_Round_D3.0mm_Vertical" (at 114.3 85.09 0)
       (effects (font (size 1.27 1.27)) hide)
     )
