File: kicad/io_uart/50pin_connector.sch (KiCad schematic (older format))
At the start: 1 part, among them P5 CONN_02X25

Commit message: io board release candidate
Connections:
- no-connect marks 8 -> 13
Changed lines of the file:
@@
 Wire Wire Line
 	5800 4350 5900 4350
+Text GLabel 8000 2450 0    60   Input ~ 0
+/CS_IO2
+Text GLabel 8000 2600 0    60   Input ~ 0
+/CS_IO1
+Text GLabel 8000 2750 0    60   Input ~ 0
+/CS_IO0
+Wire Wire Line
+	8000 2450 8100 2450
+Wire Wire Line
+	8000 2600 8100 2600
+Wire Wire Line
+	8000 2750 8100 2750
+NoConn ~ 8100 2450
+NoConn ~ 8100 2600
+NoConn ~ 8100 2750
+Text GLabel 8000 2900 0    60   Input ~ 0
+/CS_VDP
+Wire Wire Line
+	8000 2900 8100 2900
+NoConn ~ 8100 2900
+Text GLabel 8000 3050 0    60   Input ~ 0
+RDY
+Wire Wire Line
+	8000 3050 8100 3050
+NoConn ~ 8100 3050
 $EndSCHEMATC

Commit message: cleanup
Parts:
- P5: symbol CONN_02X25 -> io-rescue:CONN_02X25
Changed lines of the file:
@@
-EESchema Schematic File Version 2
-LIBS:io-rescue
-LIBS:power
-LIBS:device
-LIBS:transistors
-LIBS:conn
-LIBS:linear
-LIBS:regul
-LIBS:74xx
-LIBS:cmos4000
-LIBS:adc-dac
-LIBS:memory
-LIBS:xilinx
-LIBS:microcontrollers
-LIBS:dsp
-LIBS:microchip
-LIBS:analog_switches
-LIBS:motorola
-LIBS:texas
-LIBS:intel
-LIBS:audio
-LIBS:interface
-LIBS:digital-audio
-LIBS:philips
-LIBS:display
-LIBS:cypress
-LIBS:siliconi
-LIBS:opto
-LIBS:atmel
-LIBS:contrib
-LIBS:valves
-LIBS:65xxx
-LIBS:ttl_ieee
-LIBS:mini_din
-LIBS:dallas-rtc
-LIBS:lp2950l
-LIBS:osc
-LIBS:io-cache
-EELAYER 25 0
+EESchema Schematic File Version 4
+EELAYER 30 0
 EELAYER END
 $Descr A4 11693 8268
@@
 $EndDescr
 $Comp
-L CONN_02X25 P5
+L io-rescue:CONN_02X25 P5
 U 1 1 542071FB
 P 5550 3750
@@
 $EndComp
 $Comp
-L VCC #PWR010
+L io-rescue:VCC #PWR010
 U 1 1 54207202
 P 5200 2400
@@
 	4750 3950 5300 3950
 $Comp
-L GND #PWR011
+L io-rescue:GND #PWR011
 U 1 1 54207240
 P 4700 4100
@@
 	4700 4050 5300 4050
 $Comp
-L GND #PWR012
+L io-rescue:GND #PWR012
 U 1 1 54207248
 P 6350 4100
@@
 A5
 $Comp
-L GND #PWR013
+L io-rescue:GND #PWR013
 U 1 1 5436D639
 P 5250 5150
@@
 Connection ~ 5250 4950
 $Comp
-L VCC #PWR014
+L io-rescue:VCC #PWR014
 U 1 1 5436D6BC
 P 5950 4550
@@
 Connection ~ 5950 4650
 $Comp
-L VCC #PWR015
+L io-rescue:VCC #PWR015
 U 1 1 5436D806
 P 5150 4550
@@
 RESET_TRIG
 $Comp
-L GND #PWR016
+L io-rescue:GND #PWR016
 U 1 1 54BC2AE5
 P 4700 4300
