File: kicad/io_uart/io.sch (KiCad schematic (older format))
At the start: 18 parts, among them P2 SPI4, U1 G65SC22P

Commit message: cleanup
Parts:
- added R14, R15: 1k, symbol R
- gave numbers to parts that had none: 11
Connections:
- net labels removed: CA1', CA2', PA0', PA1', PA2', PA3', PA4', PA5', PA6', PA7'
- wire segments 136 -> 128
Other:
- moved on the sheet: R10, R11, R12, R13, R18, R19, R6, R7, R8, R9

Commit message: new joystick interface
Connections:
- wire segments 128 -> 129
Changed lines of the file:
@@
 L GND #PWR08
 U 1 1 58E66B3D
-P 10700 6250
-F 0 "#PWR08" H 10700 6000 50  0001 C CNN
-F 1 "GND" H 10700 6100 50  0000 C CNN
-F 2 "" H 10700 6250 50  0000 C CNN
-F 3 "" H 10700 6250 50  0000 C CNN
-	1    10700 6250
+P 10100 6200
+F 0 "#PWR08" H 10100 5950 50  0001 C CNN
+F 1 "GND" H 10100 6050 50  0000 C CNN
+F 2 "" H 10100 6200 50  0000 C CNN
+F 3 "" H 10100 6200 50  0000 C CNN
+	1    10100 6200
 	1    0    0    -1
 $EndComp
-Wire Wire Line
-	10700 6050 10700 6250
 Text Label 7500 6000 0    60   ~ 0
 /JOYPORT_ENABLE
@@
 L VCC #PWR09
 U 1 1 58E539E2
-P 9750 5450
-F 0 "#PWR09" H 9750 5550 30  0001 C CNN
-F 1 "VCC" H 9750 5550 30  0000 C CNN
-F 2 "" H 9750 5450 60  0000 C CNN
-F 3 "" H 9750 5450 60  0000 C CNN
-	1    9750 5450
+P 11100 5450
+F 0 "#PWR09" H 11100 5550 30  0001 C CNN
+F 1 "VCC" H 11100 5550 30  0000 C CNN
+F 2 "" H 11100 5450 60  0000 C CNN
+F 3 "" H 11100 5450 60  0000 C CNN
+	1    11100 5450
 	1    0    0    -1
 $EndComp
 Wire Wire Line
-	9750 5450 9750 6050
-Wire Wire Line
-	9750 6050 10200 6050
-Wire Wire Line
 	6700 2950 7100 2950
 Wire Wire Line
 	6700 2550 7100 2550
-Text Label 9950 5550 0    60   ~ 0
+Text Label 10750 5950 0    60   ~ 0
 PA0
+Text Label 10000 5950 0    60   ~ 0
+PA1
+Text Label 10750 5850 0    60   ~ 0
+PA2
+Text Label 10000 5850 0    60   ~ 0
+PA3
+Text Label 10750 5750 0    60   ~ 0
+PA4
+Text Label 10000 5750 0    60   ~ 0
+PA5
+Text Label 10750 5650 0    60   ~ 0
+PA6
+Text Label 10000 5650 0    60   ~ 0
+PA7
 Text Label 10750 5550 0    60   ~ 0
-PA1
-Text Label 9950 5650 0    60   ~ 0
-PA2
-Text Label 10750 5650 0    60   ~ 0
-PA3
-Text Label 9950 5750 0    60   ~ 0
-PA4
-Text Label 10750 5750 0    60   ~ 0
-PA5
-Text Label 9950 5850 0    60   ~ 0
-PA6
-Text Label 10750 5850 0    60   ~ 0
-PA7
-Text Label 9950 5950 0    60   ~ 0
 CA1
-Text Label 10750 5950 0    60   ~ 0
+Text Label 10000 5550 0    60   ~ 0
 CA2
 Wire Wire Line
@@
 Text Label 7850 5450 0    60   ~ 0
 PA2
+Wire Wire Line
+	10100 6200 10100 6050
+Wire Wire Line
+	10100 6050 10200 6050
+Wire Wire Line
+	10700 6050 11100 6050
+Wire Wire Line
+	11100 6050 11100 5450
 $EndSCHEMATC

Commit message: xmodem
Parts:
- P1: footprint (none) -> Pin_Headers:Pin_Header_Angled_2x06
- P2: footprint Pin_Headers:Pin_Header_Straight_2x03 -> Pin_Headers:Pin_Header_Angled_2x03
- R10, R11, R12, R13, R14, R15, R18, R19, R6, R7, R8, R9: footprint (none) -> Discret:R3-LARGE_PADS

Commit message: io board release candidate
Parts:
- C1, C2, C3, C5: footprint Capacitors_ThroughHole:C_Rect_L4_W2.5_P2.5 -> Capacitors_ThroughHole:C_Disc_D3_P2.5
- C4: footprint Capacitors_ThroughHole:C_Radial_D8_L11.5_P3.5 -> Capacitors_ThroughHole:C_Disc_D3_P2.5
- P1: footprint Pin_Headers:Pin_Header_Angled_2x06 -> Pin_Headers:Pin_Header_Angled_2x08; symbol CONN_02X06 -> CONN_02X08
- R10, R11, R12, R13, R14, R15, R18, R19, R6, R7, R8, R9: footprint Discret:R3-LARGE_PADS -> Resistors_ThroughHole:Resistor_Horizontal_RM7mm
Connections:
- wire segments 129 -> 131
- no-connect marks 2 -> 4
Changed lines of the file:
@@
 F 0 "C1" H 4350 7250 40  0000 L CNN
 F 1 "100nF" H 4356 7065 40  0000 L CNN
-F 2 "Capacitors_ThroughHole:C_Rect_L4_W2.5_P2.5" H 4388 7000 30  0001 C CNN
+F 2 "Capacitors_ThroughHole:C_Disc_D3_P2.5" H 4388 7000 30  0001 C CNN
 F 3 "" H 4350 7150 60  0000 C CNN
 	1    4350 7150
@@
 F 0 "C2" H 4650 7250 40  0000 L CNN
 F 1 "100nF" H 4656 7065 40  0000 L CNN
-F 2 "Capacitors_ThroughHole:C_Rect_L4_W2.5_P2.5" H 4688 7000 30  0001 C CNN
+F 2 "Capacitors_ThroughHole:C_Disc_D3_P2.5" H 4688 7000 30  0001 C CNN
 F 3 "" H 4650 7150 60  0000 C CNN
 	1    4650 7150
@@
 F 0 "C3" H 4950 7250 40  0000 L CNN
 F 1 "100nF" H 4956 7065 40  0000 L CNN
-F 2 "Capacitors_ThroughHole:C_Rect_L4_W2.5_P2.5" H 4988 7000 30  0001 C CNN
+F 2 "Capacitors_ThroughHole:C_Disc_D3_P2.5" H 4988 7000 30  0001 C CNN
 F 3 "" H 4950 7150 60  0000 C CNN
 	1    4950 7150
@@
 F 0 "C4" H 5250 7250 40  0000 L CNN
 F 1 "100µF" H 5256 7065 40  0000 L CNN
-F 2 "Capacitors_ThroughHole:C_Radial_D8_L11.5_P3.5" H 5288 7000 30  0001 C CNN
+F 2 "Capacitors_ThroughHole:C_Disc_D3_P2.5" H 5288 7000 30  0001 C CNN
 F 3 "" H 5250 7150 60  0000 C CNN
 	1    5250 7150
@@
 F 0 "C5" H 5550 7250 40  0000 L CNN
 F 1 "100nF" H 5556 7065 40  0000 L CNN
-F 2 "Capacitors_ThroughHole:C_Rect_L4_W2.5_P2.5" H 5588 7000 30  0001 C CNN
+F 2 "Capacitors_ThroughHole:C_Disc_D3_P2.5" H 5588 7000 30  0001 C CNN
 F 3 "" H 5550 7150 60  0000 C CNN
 	1    5550 7150
@@
 $EndSheet
 $Comp
-L CONN_02X06 P1
-U 1 1 58E669F2
-P 10450 5800
-F 0 "P1" H 10450 6150 50  0000 C CNN
-F 1 "USERPORT" H 10450 5450 50  0000 C CNN
-F 2 "Pin_Headers:Pin_Header_Angled_2x06" H 10450 4600 50  0001 C CNN
-F 3 "" H 10450 4600 50  0000 C CNN
-	1    10450 5800
-	1    0    0    -1
-$EndComp
-$Comp
 L GND #PWR08
 U 1 1 58E66B3D
-P 10100 6200
-F 0 "#PWR08" H 10100 5950 50  0001 C CNN
-F 1 "GND" H 10100 6050 50  0000 C CNN
-F 2 "" H 10100 6200 50  0000 C CNN
-F 3 "" H 10100 6200 50  0000 C CNN
-	1    10100 6200
+P 9600 6250
+F 0 "#PWR08" H 9600 6000 50  0001 C CNN
+F 1 "GND" H 9600 6100 50  0000 C CNN
+F 2 "" H 9600 6250 50  0000 C CNN
+F 3 "" H 9600 6250 50  0000 C CNN
+	1    9600 6250
 	1    0    0    -1
 $EndComp
@@
 	1    0    0    -1
 $EndComp
-Text Label 10750 5950 0    60   ~ 0
-PA0
-Text Label 10000 5950 0    60   ~ 0
-PA1
-Text Label 10750 5850 0    60   ~ 0
-PA2
-Text Label 10000 5850 0    60   ~ 0
-PA3
-Text Label 10750 5750 0    60   ~ 0
-PA4
-Text Label 10000 5750 0    60   ~ 0
-PA5
-Text Label 10750 5650 0    60   ~ 0
-PA6
-Text Label 10000 5650 0    60   ~ 0
-PA7
-Text Label 10750 5550 0    60   ~ 0
-CA1
-Text Label 10000 5550 0    60   ~ 0
-CA2
 Text Label 7850 6200 0    60   ~ 0
 PA7
@@
 F 0 "R19" V 6550 4400 50  0000 C CNN
 F 1 "1k" V 6550 4500 50  0000 C CNN
-F 2 "Discret:R3-LARGE_PADS" V 6480 4450 50  0001 C CNN
+F 2 "Resistors_ThroughHole:Resistor_Horizontal_RM7mm" V 6480 4450 50  0001 C CNN
 F 3 "" H 6550 4450 50  0000 C CNN
 	1    6550 4450
@@
 F 0 "R18" V 6550 4300 50  0000 C CNN
 F 1 "1k" V 6550 4400 50  0000 C CNN
-F 2 "Discret:R3-LARGE_PADS" V 6480 4350 50  0001 C CNN
+F 2 "Resistors_ThroughHole:Resistor_Horizontal_RM7mm" V 6480 4350 50  0001 C CNN
 F 3 "" H 6550 4350 50  0000 C CNN
 	1    6550 4350
@@
 F 0 "R15" V 6550 4000 50  0000 C CNN
 F 1 "1k" V 6550 4100 50  0000 C CNN
-F 2 "Discret:R3-LARGE_PADS" V 6480 4050 50  0001 C CNN
+F 2 "Resistors_ThroughHole:Resistor_Horizontal_RM7mm" V 6480 4050 50  0001 C CNN
 F 3 "" H 6550 4050 50  0000 C CNN
 	1    6550 4050
@@
 F 0 "R14" V 6550 3900 50  0000 C CNN
 F 1 "1k" V 6550 4000 50  0000 C CNN
-F 2 "Discret:R3-LARGE_PADS" V 6480 3950 50  0001 C CNN
+F 2 "Resistors_ThroughHole:Resistor_Horizontal_RM7mm" V 6480 3950 50  0001 C CNN
 F 3 "" H 6550 3950 50  0000 C CNN
 	1    6550 3950
@@
 	6700 4450 7100 4450
 Wire Wire Line
-	10200 5550 9850 5550
-Wire Wire Line
-	10700 5550 11000 5550
-Wire Wire Line
-	10200 5650 9850 5650
-Wire Wire Line
-	10700 5650 11000 5650
-Wire Wire Line
-	10200 5750 9850 5750
-Wire Wire Line
-	10700 5750 11000 5750
-Wire Wire Line
-	10200 5850 9850 5850
-Wire Wire Line
-	10700 5850 11000 5850
-Wire Wire Line
-	10200 5950 9850 5950
-Wire Wire Line
-	10700 5950 11000 5950
-Wire Wire Line
 	6400 2550 6100 2550
 Wire Wire Line
@@
 	6700 4050 6900 4050
 Wire Wire Line
-	10100 6200 10100 6050
-Wire Wire Line
-	10100 6050 10200 6050
-Wire Wire Line
-	10700 6050 11100 6050
-Wire Wire Line
-	11100 6050 11100 5450
+	9600 6250 9600 5850
+Wire Wire Line
+	11100 5850 11100 5450
 $Comp
 L R R13
@@
 F 0 "R13" V 6550 3200 50  0000 C CNN
 F 1 "1k" V 6550 3300 50  0000 C CNN
-F 2 "Discret:R3-LARGE_PADS" V 6480 3250 50  0001 C CNN
+F 2 "Resistors_ThroughHole:Resistor_Horizontal_RM7mm" V 6480 3250 50  0001 C CNN
 F 3 "" H 6550 3250 50  0000 C CNN
 	1    6550 3250
@@
 F 0 "R12" V 6550 3100 50  0000 C CNN
 F 1 "1k" V 6550 3200 50  0000 C CNN
-F 2 "Discret:R3-LARGE_PADS" V 6480 3150 50  0001 C CNN
+F 2 "Resistors_ThroughHole:Resistor_Horizontal_RM7mm" V 6480 3150 50  0001 C CNN
 F 3 "" H 6550 3150 50  0000 C CNN
 	1    6550 3150
@@
 F 0 "R11" V 6550 3000 50  0000 C CNN
 F 1 "1k" V 6550 3100 50  0000 C CNN
-F 2 "Discret:R3-LARGE_PADS" V 6480 3050 50  0001 C CNN
+F 2 "Resistors_ThroughHole:Resistor_Horizontal_RM7mm" V 6480 3050 50  0001 C CNN
 F 3 "" H 6550 3050 50  0000 C CNN
 	1    6550 3050
@@
 F 0 "R10" V 6550 2900 50  0000 C CNN
 F 1 "1k" V 6550 3000 50  0000 C CNN
-F 2 "Discret:R3-LARGE_PADS" V 6480 2950 50  0001 C CNN
+F 2 "Resistors_ThroughHole:Resistor_Horizontal_RM7mm" V 6480 2950 50  0001 C CNN
 F 3 "" H 6550 2950 50  0000 C CNN
 	1    6550 2950
@@
 F 0 "R9" V 6550 2800 50  0000 C CNN
 F 1 "1k" V 6550 2900 50  0000 C CNN
-F 2 "Discret:R3-LARGE_PADS" V 6480 2850 50  0001 C CNN
+F 2 "Resistors_ThroughHole:Resistor_Horizontal_RM7mm" V 6480 2850 50  0001 C CNN
 F 3 "" H 6550 2850 50  0000 C CNN
 	1    6550 2850
@@
 F 0 "R8" V 6550 2700 50  0000 C CNN
 F 1 "1k" V 6550 2800 50  0000 C CNN
-F 2 "Discret:R3-LARGE_PADS" V 6480 2750 50  0001 C CNN
+F 2 "Resistors_ThroughHole:Resistor_Horizontal_RM7mm" V 6480 2750 50  0001 C CNN
 F 3 "" H 6550 2750 50  0000 C CNN
 	1    6550 2750
@@
 F 0 "R7" V 6550 2600 50  0000 C CNN
 F 1 "1k" V 6550 2700 50  0000 C CNN
-F 2 "Discret:R3-LARGE_PADS" V 6480 2650 50  0001 C CNN
+F 2 "Resistors_ThroughHole:Resistor_Horizontal_RM7mm" V 6480 2650 50  0001 C CNN
 F 3 "" H 6550 2650 50  0000 C CNN
 	1    6550 2650
@@
 F 0 "R6" V 6550 2500 50  0000 C CNN
 F 1 "1k" V 6550 2600 50  0000 C CNN
-F 2 "Discret:R3-LARGE_PADS" V 6480 2550 50  0001 C CNN
+F 2 "Resistors_ThroughHole:Resistor_Horizontal_RM7mm" V 6480 2550 50  0001 C CNN
 F 3 "" H 6550 2550 50  0000 C CNN
 	1    6550 2550
 	0    1    1    0
 $EndComp
+$Comp
+L CONN_02X08 P1
+U 1 1 58E669F2
+P 10450 5800
+F 0 "P1" H 10450 6150 50  0000 C CNN
+F 1 "USERPORT" H 10450 5350 50  0000 C CNN
+F 2 "Pin_Headers:Pin_Header_Angled_2x08" H 10450 4600 50  0001 C CNN
+F 3 "" H 10450 4600 50  0000 C CNN
+	1    10450 5800
+	1    0    0    -1
+$EndComp
+Wire Wire Line
+	9600 5850 10200 5850
+Wire Wire Line
+	11100 5850 10700 5850
+NoConn ~ 10700 5950
+NoConn ~ 10200 5950
+Wire Wire Line
+	10200 6050 10100 6050
+Wire Wire Line
+	10200 6150 9950 6150
+Wire Wire Line
+	10200 5750 9950 5750
+Wire Wire Line
+	10200 5650 9950 5650
+Wire Wire Line
+	10200 5550 9950 5550
+Wire Wire Line
+	10200 5450 9950 5450
+Wire Wire Line
+	10700 5450 11000 5450
+Wire Wire Line
+	10700 5550 11000 5550
+Wire Wire Line
+	10700 5650 11000 5650
+Wire Wire Line
+	10700 5750 11000 5750
+Text Label 10050 5450 0    60   ~ 0
+PA0
+Text Label 10750 5450 0    60   ~ 0
+PA1
+Text Label 10050 5550 0    60   ~ 0
+PA2
+Text Label 10750 5550 0    60   ~ 0
+PA3
+Text Label 10050 5650 0    60   ~ 0
+PA4
+Text Label 10750 5650 0    60   ~ 0
+PA5
+Text Label 10050 5750 0    60   ~ 0
+PA6
+Text Label 10750 5750 0    60   ~ 0
+PA7
+Wire Wire Line
+	10700 6050 10900 6050
+Wire Wire Line
+	10700 6150 11000 6150
+Text Label 10050 6150 0    60   ~ 0
+CA2
+Text Label 10750 6150 0    60   ~ 0
+CA1
+Text GLabel 10100 6050 0    60   Input ~ 0
+/RESET
+Text GLabel 10900 6050 2    60   Input ~ 0
+/IRQ
 $EndSCHEMATC

Commit message: C8 fix footprint
Parts:
- U1: symbol G65SC22P -> G65SC22P-RESCUE-io
Changed lines of the file:
@@
 $EndComp
 $Comp
-L G65SC22P U1
+L G65SC22P-RESCUE-io U1
 U 1 1 542879F7
 P 5500 3550

Commit message: cleanup
Parts:
- C1, C2, C3, C5: symbol C -> io-rescue:C
- C4: symbol CP -> io-rescue:CP
- P1: symbol CONN_02X08 -> io-rescue:CONN_02X08
- P2: symbol CONN_02X03 -> io-rescue:CONN_02X03
- R10, R11, R12, R13, R14, R15, R18, R19, R6, R7, R8, R9: symbol R -> io-rescue:R
- U1: symbol G65SC22P-RESCUE-io -> io-rescue:G65SC22P-RESCUE-io
Connections:
- wire segments 131 -> 138
Changed lines of the file:
@@
-EESchema Schematic File Version 2
-LIBS:io-rescue
-LIBS:power
-LIBS:device
-LIBS:transistors
-LIBS:conn
-LIBS:linear
-LIBS:regul
-LIBS:74xx
-LIBS:cmos4000
-LIBS:adc-dac
-LIBS:memory
-LIBS:xilinx
-LIBS:microcontrollers
-LIBS:dsp
-LIBS:microchip
-LIBS:analog_switches
-LIBS:motorola
-LIBS:texas
-LIBS:intel
-LIBS:audio
-LIBS:interface
-LIBS:digital-audio
-LIBS:philips
-LIBS:display
-LIBS:cypress
-LIBS:siliconi
-LIBS:opto
-LIBS:atmel
-LIBS:contrib
-LIBS:valves
-LIBS:65xxx
-LIBS:ttl_ieee
-LIBS:mini_din
-LIBS:dallas-rtc
-LIBS:lp2950l
-LIBS:osc
-LIBS:io-cache
-EELAYER 25 0
+EESchema Schematic File Version 4
+EELAYER 30 0
 EELAYER END
 $Descr A4 11693 8268
@@
 PHI2
 $Comp
-L VCC #PWR01
+L io-rescue:VCC #PWR01
 U 1 1 5428C2B0
 P 4850 4550
@@
 $EndComp
 $Comp
-L GND #PWR02
+L io-rescue:GND #PWR02
 U 1 1 5428C330
 P 4850 5150
@@
 $EndComp
 $Comp
-L VCC #PWR03
+L io-rescue:VCC #PWR03
 U 1 1 5428C3FC
 P 4350 6950
@@
 $EndComp
 $Comp
-L GND #PWR04
+L io-rescue:GND #PWR04
 U 1 1 5428C42D
 P 4350 7400
@@
 $EndComp
 $Comp
-L C C1
+L io-rescue:C C1
 U 1 1 5428C484
 P 4350 7150
@@
 $EndComp
 $Comp
-L VCC #PWR05
+L io-rescue:VCC #PWR05
 U 1 1 5428D273
 P 6250 4900
@@
 SPI_MISO
 $Comp
-L C C2
+L io-rescue:C C2
 U 1 1 545C1C49
 P 4650 7150
@@
 ~SPI_SS3
 $Comp
-L C C3
+L io-rescue:C C3
 U 1 1 548DF92D
 P 4950 7150
@@
 ~SD_CARD_DETECT
 $Comp
-L CP C4
+L io-rescue:CP C4
 U 1 1 54B14D65
 P 5250 7150
@@
 $EndComp
 $Comp
-L CONN_02X03 P2
+L io-rescue:CONN_02X03 P2
 U 1 1 54B176A0
 P 1600 4950
@@
 $EndComp
 $Comp
-L VCC #PWR06
+L io-rescue:VCC #PWR06
 U 1 1 54B17C97
 P 1950 4700
@@
 $EndComp
 $Comp
-L GND #PWR07
+L io-rescue:GND #PWR07
 U 1 1 54B17DD5
 P 1950 5150
@@
 ~SPI_SS4
 $Comp
-L C C5
+L io-rescue:C C5
 U 1 1 54B17E82
 P 5550 7150
@@
 $EndComp
 $Comp
-L G65SC22P-RESCUE-io U1
+L io-rescue:G65SC22P-RESCUE-io U1
 U 1 1 542879F7
 P 5500 3550
@@
 $EndSheet
 $Comp
-L GND #PWR08
+L io-rescue:GND #PWR08
 U 1 1 58E66B3D
 P 9600 6250
@@
 CA2
 $Comp
-L VCC #PWR09
+L io-rescue:VCC #PWR09
 U 1 1 58E539E2
 P 11100 5450
@@
 PA2
 $Comp
-L R R19
+L io-rescue:R R19
 U 1 1 58E602B4
 P 6550 4450
@@
 $EndComp
 $Comp
-L R R18
+L io-rescue:R R18
 U 1 1 58E60166
 P 6550 4350
@@
 $EndComp
 $Comp
-L R R15
+L io-rescue:R R15
 U 1 1 58E6A856
 P 6550 4050
@@
 $EndComp
 $Comp
-L R R14
+L io-rescue:R R14
 U 1 1 58E69E9D
 P 6550 3950
@@
 	6100 3550 6900 3550
 Wire Wire Line
-	6100 3450 6900 3450
+	6100 3450 6250 3450
 Connection ~ 4350 7300
 Connection ~ 4650 7300
@@
 Connection ~ 4350 7000
 Wire Wire Line
-	4350 7300 5550 7300
-Wire Wire Line
-	4350 7000 5550 7000
+	4350 7300 4650 7300
+Wire Wire Line
+	4350 7000 4650 7000
 Wire Wire Line
 	6100 5050 6350 5050
@@
 Wire Wire Line
 	4800 3450 4900 3450
-Wire Bus Line
-	4700 3250 4700 3750
 Wire Wire Line
 	4900 3250 4800 3250
@@
 Wire Wire Line
 	4800 2550 4900 2550
-Wire Bus Line
-	4700 2350 4700 3150
 Wire Wire Line
 	10300 2500 10200 2500
@@
 Wire Wire Line
 	10200 1800 10300 1800
-Wire Bus Line
-	10100 1600 10100 2400
 Wire Wire Line
 	10200 1050 10300 1050
@@
 Wire Wire Line
 	10200 750  10300 750
-Wire Bus Line
-	10100 550  10100 1050
 Wire Wire Line
 	6250 4650 6250 3450
@@
 Connection ~ 5250 7000
 Connection ~ 5250 7300
-Connection ~ 4900 2550
-Connection ~ 4900 2650
-Connection ~ 4900 2750
-Connection ~ 4900 2850
-Connection ~ 4900 2950
-Connection ~ 4900 3050
-Connection ~ 4900 3150
-Connection ~ 4900 3250
-Connection ~ 4900 3450
-Connection ~ 4900 3550
-Connection ~ 4900 3650
-Connection ~ 4900 3750
-Connection ~ 4900 3950
-Connection ~ 4900 4050
-Connection ~ 4900 4150
-Connection ~ 4900 4250
-Connection ~ 4900 4650
 Wire Wire Line
 	8050 2300 7950 2300
@@
 Wire Wire Line
 	7950 1600 8050 1600
-Wire Bus Line
-	7850 1400 7850 2200
 Wire Wire Line
 	8050 1000 7950 1000
@@
 Wire Wire Line
 	7950 800  8050 800
-Wire Bus Line
-	7850 600  7850 1100
 Wire Wire Line
 	8050 1250 7200 1250
@@
 	11100 5850 11100 5450
 $Comp
-L R R13
+L io-rescue:R R13
 U 1 1 58E6001B
 P 6550 3250
@@
 $EndComp
 $Comp
-L R R12
+L io-rescue:R R12
 U 1 1 58E5FED7
 P 6550 3150
@@
 $EndComp
 $Comp
-L R R11
+L io-rescue:R R11
 U 1 1 58E5FD96
 P 6550 3050
@@
 $EndComp
 $Comp
-L R R10
+L io-rescue:R R10
 U 1 1 58E5FA24
 P 6550 2950
@@
 $EndComp
 $Comp
-L R R9
+L io-rescue:R R9
 U 1 1 58E5F8E9
 P 6550 2850
@@
 $EndComp
 $Comp
-L R R8
+L io-rescue:R R8
 U 1 1 58E5F7AD
 P 6550 2750
@@
 $EndComp
 $Comp
-L R R7
+L io-rescue:R R7
 U 1 1 58E5F674
 P 6550 2650
@@
 $EndComp
 $Comp
-L R R6
+L io-rescue:R R6
 U 1 1 58E669F9
 P 6550 2550
@@
 $EndComp
 $Comp
-L CONN_02X08 P1
+L io-rescue:CONN_02X08 P1
 U 1 1 58E669F2
 P 10450 5800
@@
 Text GLabel 10900 6050 2    60   Input ~ 0
 /IRQ
+Wire Wire Line
+	4650 7300 4950 7300
+Wire Wire Line
+	4950 7300 5250 7300
+Wire Wire Line
+	4950 7000 5250 7000
+Wire Wire Line
+	4650 7000 4950 7000
+Wire Wire Line
+	6250 3450 6900 3450
+Wire Wire Line
+	5250 7000 5550 7000
+Wire Wire Line
+	5250 7300 5550 7300
+Wire Bus Line
+	4700 3250 4700 3750
+Wire Bus Line
+	10100 550  10100 1050
+Wire Bus Line
+	7850 600  7850 1100
+Wire Bus Line
+	4700 2350 4700 3150
+Wire Bus Line
+	10100 1600 10100 2400
+Wire Bus Line
+	7850 1400 7850 2200
 $EndSCHEMATC
