File: kicad/io_uart/rtc.sch (KiCad schematic (older format))
At the start: 4 parts

Commit message: cleanup
Parts:
- gave numbers to parts that had none: 4
Connections:
- wire segments 25 -> 22
Changed lines of the file:
@@
 $EndDescr
 $Comp
-L DS1306 U?
+L DS1306 U7
 U 1 1 58E7934B
 P 4850 3400
-F 0 "U?" H 4450 4200 50  0000 L BNN
+F 0 "U7" H 4450 4200 50  0000 L BNN
 F 1 "DS1306" H 4450 2500 50  0000 L BNN
 F 2 "Housings_DIP:DIP-16_W7.62mm_LongPads" H 4850 3550 50  0001 C CNN
@@
 $EndComp
 $Comp
-L Crystal X?
+L Crystal X1
 U 1 1 58E79352
 P 3750 3100
-F 0 "X?" H 3750 3190 30  0000 C CNN
+F 0 "X1" H 3750 3190 30  0000 C CNN
 F 1 "CRYSTAL_SMD" H 3780 2990 30  0000 L CNN
 F 2 "Crystals:Crystal_Round_Vertical_3mm_BigPad" H 3750 3100 60  0001 C CNN
@@
 $EndComp
 $Comp
-L GND #PWR?
+L GND #PWR037
 U 1 1 58E79359
 P 4200 4300
-F 0 "#PWR?" H 4200 4300 30  0001 C CNN
+F 0 "#PWR037" H 4200 4300 30  0001 C CNN
 F 1 "GND" H 4200 4230 30  0001 C CNN
 F 2 "" H 4200 4300 60  0000 C CNN
@@
 $EndComp
 $Comp
-L GND #PWR?
+L GND #PWR038
 U 1 1 58E7935F
 P 4150 2750
-F 0 "#PWR?" H 4150 2750 30  0001 C CNN
+F 0 "#PWR038" H 4150 2750 30  0001 C CNN
 F 1 "GND" H 4150 2680 30  0001 C CNN
 F 2 "" H 4150 2750 60  0000 C CNN
@@
 $EndComp
 $Comp
-L VCC #PWR?
+L VCC #PWR039
 U 1 1 58E79365
 P 5650 2500
-F 0 "#PWR?" H 5650 2600 30  0001 C CNN
+F 0 "#PWR039" H 5650 2600 30  0001 C CNN
 F 1 "VCC" H 5650 2600 30  0000 C CNN
 F 2 "" H 5650 2500 60  0000 C CNN
@@
 $EndComp
 $Comp
-L Battery BT?
+L Battery BT1
 U 1 1 58E7936D
 P 3900 2900
-F 0 "BT?" H 3900 3100 50  0000 C CNN
+F 0 "BT1" H 3900 3100 50  0000 C CNN
 F 1 "BATTERY" H 3900 2710 50  0000 C CNN
 F 2 "Connect:CR2032H" H 3900 2900 60  0001 C CNN
@@
 $EndComp
 $Comp
-L GND #PWR?
+L GND #PWR040
 U 1 1 58E79374
 P 3500 2950
-F 0 "#PWR?" H 3500 2950 30  0001 C CNN
+F 0 "#PWR040" H 3500 2950 30  0001 C CNN
 F 1 "GND" H 3500 2880 30  0001 C CNN
 F 2 "" H 3500 2950 60  0000 C CNN
@@
 NoConn ~ 5450 2900
 $Comp
-L 7400 U?
-U 1 1 58E7937F
+L 7400 U2
+U 4 1 58E7937F
 P 6500 3900
-F 0 "U?" H 6500 3950 60  0000 C CNN
+F 0 "U2" H 6500 3950 60  0000 C CNN
 F 1 "7400" H 6500 3800 60  0000 C CNN
 F 2 "Housings_DIP:DIP-14_W7.62mm_LongPads" H 6500 3900 60  0001 C CNN
 F 3 "" H 6500 3900 60  0000 C CNN
-	1    6500 3900
+	4    6500 3900
 	-1   0    0    1
 $EndComp
@@
 	5450 2700 5650 2700
 Wire Wire Line
-	5650 2500 5650 2700
-Wire Wire Line
-	5650 2700 5650 3100
-Wire Wire Line
-	5650 3100 5650 4100
+	5650 2500 5650 4100
 Wire Wire Line
 	5650 3100 5450 3100
@@
 	5450 3300 5950 3300
 Wire Wire Line
-	7100 3800 7100 3900
-Wire Wire Line
-	7100 3900 7100 4000
+	7100 3800 7100 4000
 Connection ~ 7100 3900
 Text GLabel 3950 3500 0    60   Input ~ 0

Commit message: C8 fix footprint
Parts:
- U7: symbol DS1306 -> DS1306-RESCUE-io
Changed lines of the file:
@@
 $EndDescr
 $Comp
-L DS1306 U7
+L DS1306-RESCUE-io U7
 U 1 1 58E7934B
 P 4850 3400
+AR Path="/58E7934B" Ref="U7"  Part="1"
+AR Path="/58E79100/58E7934B" Ref="U7"  Part="1"
 F 0 "U7" H 4450 4200 50  0000 L BNN
 F 1 "DS1306" H 4450 2500 50  0000 L BNN

Commit message: cleanup
Parts:
- BT1: symbol Battery -> io-rescue:Battery
- U2: symbol 7400 -> io-rescue:7400
- U7: symbol DS1306-RESCUE-io -> io-rescue:DS1306-RESCUE-io
- X1: symbol Crystal -> io-rescue:Crystal
Changed lines of the file:
@@
-EESchema Schematic File Version 2
-LIBS:io-rescue
-LIBS:power
-LIBS:device
-LIBS:transistors
-LIBS:conn
-LIBS:linear
-LIBS:regul
-LIBS:74xx
-LIBS:cmos4000
-LIBS:adc-dac
-LIBS:memory
-LIBS:xilinx
-LIBS:microcontrollers
-LIBS:dsp
-LIBS:microchip
-LIBS:analog_switches
-LIBS:motorola
-LIBS:texas
-LIBS:intel
-LIBS:audio
-LIBS:interface
-LIBS:digital-audio
-LIBS:philips
-LIBS:display
-LIBS:cypress
-LIBS:siliconi
-LIBS:opto
-LIBS:atmel
-LIBS:contrib
-LIBS:valves
-LIBS:65xxx
-LIBS:ttl_ieee
-LIBS:mini_din
-LIBS:dallas-rtc
-LIBS:lp2950l
-LIBS:osc
-LIBS:io-cache
-EELAYER 25 0
+EESchema Schematic File Version 4
+EELAYER 30 0
 EELAYER END
 $Descr A4 11693 8268
@@
 $EndDescr
 $Comp
-L DS1306-RESCUE-io U7
+L io-rescue:DS1306-RESCUE-io U7
 U 1 1 58E7934B
 P 4850 3400
@@
 $EndComp
 $Comp
-L Crystal X1
+L io-rescue:Crystal X1
 U 1 1 58E79352
 P 3750 3100
@@
 $EndComp
 $Comp
-L GND #PWR037
+L io-rescue:GND #PWR037
 U 1 1 58E79359
 P 4200 4300
@@
 $EndComp
 $Comp
-L GND #PWR038
+L io-rescue:GND #PWR038
 U 1 1 58E7935F
 P 4150 2750
@@
 $EndComp
 $Comp
-L VCC #PWR039
+L io-rescue:VCC #PWR039
 U 1 1 58E79365
 P 5650 2500
@@
 $EndComp
 $Comp
-L Battery BT1
+L io-rescue:Battery BT1
 U 1 1 58E7936D
 P 3900 2900
@@
 $EndComp
 $Comp
-L GND #PWR040
+L io-rescue:GND #PWR040
 U 1 1 58E79374
 P 3500 2950
@@
 NoConn ~ 5450 2900
 $Comp
-L 7400 U2
+L io-rescue:7400 U2
 U 4 1 58E7937F
 P 6500 3900
