File: kicad/io_uart/sd_card.sch (KiCad schematic (older format))
At the start: 14 parts, among them U4 74125, U5 LP2950, U6 7407

Commit message: xmodem
Parts:
- R1, R2, R3, R4, R5: footprint Discret:R3-LARGE_PADS -> Discret:R1
Changed lines of the file:
@@
 $Comp
 L 7407 U6
-U 3 1 542928D0
+U 4 1 542928D0
 P 1900 3600
 F 0 "U6" H 2050 3950 60  0000 C CNN
@@
 F 2 "Housings_DIP:DIP-14_W7.62mm_LongPads" H 1900 3600 60  0001 C CNN
 F 3 "" H 1900 3600 60  0000 C CNN
-	3    1900 3600
+	4    1900 3600
 	1    0    0    -1
 $EndComp
 $Comp
 L 7407 U6
-U 1 1 542928D7
+U 6 1 542928D7
 P 1900 2200
 F 0 "U6" H 2050 2550 60  0000 C CNN
@@
 F 2 "Housings_DIP:DIP-14_W7.62mm_LongPads" H 1900 2200 60  0001 C CNN
 F 3 "" H 1900 2200 60  0000 C CNN
-	1    1900 2200
+	6    1900 2200
 	1    0    0    -1
 $EndComp
 $Comp
 L 7407 U6
-U 2 1 542928DE
+U 5 1 542928DE
 P 1900 2900
 F 0 "U6" H 2050 3250 60  0000 C CNN
@@
 F 2 "Housings_DIP:DIP-14_W7.62mm_LongPads" H 1900 2900 60  0001 C CNN
 F 3 "" H 1900 2900 60  0000 C CNN
-	2    1900 2900
+	5    1900 2900
 	1    0    0    -1
 $EndComp
@@
 F 0 "R1" V 2780 1700 40  0000 C CNN
 F 1 "1k" V 2707 1701 40  0000 C CNN
-F 2 "Discret:R3-LARGE_PADS" V 2630 1700 30  0001 C CNN
+F 2 "Discret:R1" V 2630 1700 30  0001 C CNN
 F 3 "" H 2700 1700 30  0000 C CNN
 	1    2700 1700
@@
 F 0 "R2" V 2980 1700 40  0000 C CNN
 F 1 "10k" V 2907 1701 40  0000 C CNN
-F 2 "Discret:R3-LARGE_PADS" V 2830 1700 30  0001 C CNN
+F 2 "Discret:R1" V 2830 1700 30  0001 C CNN
 F 3 "" H 2900 1700 30  0000 C CNN
 	1    2900 1700
@@
 F 0 "R3" V 3180 1700 40  0000 C CNN
 F 1 "10k" V 3107 1701 40  0000 C CNN
-F 2 "Discret:R3-LARGE_PADS" V 3030 1700 30  0001 C CNN
+F 2 "Discret:R1" V 3030 1700 30  0001 C CNN
 F 3 "" H 3100 1700 30  0000 C CNN
 	1    3100 1700
@@
 F 0 "R5" V 4380 1700 40  0000 C CNN
 F 1 "47k" V 4307 1701 40  0000 C CNN
-F 2 "Discret:R3-LARGE_PADS" V 4230 1700 30  0001 C CNN
+F 2 "Discret:R1" V 4230 1700 30  0001 C CNN
 F 3 "" H 4300 1700 30  0000 C CNN
 	1    4300 1700
@@
 F 0 "R4" V 4180 1700 40  0000 C CNN
 F 1 "47k" V 4107 1701 40  0000 C CNN
-F 2 "Discret:R3-LARGE_PADS" V 4030 1700 30  0001 C CNN
+F 2 "Discret:R1" V 4030 1700 30  0001 C CNN
 F 3 "" H 4100 1700 30  0000 C CNN
 	1    4100 1700

Commit message: io board release candidate
Parts:
- C10, C7, C9: footprint Capacitors_ThroughHole:C_Rect_L4_W2.5_P2.5 -> Capacitors_ThroughHole:C_Disc_D3_P2.5
- C6: footprint Capacitors_ThroughHole:C_Radial_D6.3_L11.2_P2.5 -> Capacitors_ThroughHole:C_Radial_D5_L6_P2.5
- C8: footprint Capacitors_ThroughHole:C_Rect_L4_W2.5_P2.5 -> Capacitors_ThroughHole:C_Radial_D8_L11.5_P3.5
- R1, R2, R3, R4, R5: footprint Discret:R1 -> Resistors_ThroughHole:Resistor_Horizontal_RM7mm
- U5: footprint TO_SOT_Packages_THT:TO-92_Inline_Wide -> TO_SOT_Packages_THT:TO-92_Inline_Narrow_Oval
Changed lines of the file:
@@
 F 0 "R1" V 2780 1700 40  0000 C CNN
 F 1 "1k" V 2707 1701 40  0000 C CNN
-F 2 "Discret:R1" V 2630 1700 30  0001 C CNN
+F 2 "Resistors_ThroughHole:Resistor_Horizontal_RM7mm" V 2630 1700 30  0001 C CNN
 F 3 "" H 2700 1700 30  0000 C CNN
 	1    2700 1700
@@
 F 0 "U5" H 2050 1204 60  0000 C CNN
 F 1 "LP2950" H 1900 1600 60  0000 C CNN
-F 2 "TO_SOT_Packages_THT:TO-92_Inline_Wide" H 1900 1400 60  0001 C CNN
+F 2 "TO_SOT_Packages_THT:TO-92_Inline_Narrow_Oval" H 1900 1400 60  0001 C CNN
 F 3 "" H 1900 1400 60  0000 C CNN
 	1    1900 1400
@@
 F 0 "R2" V 2980 1700 40  0000 C CNN
 F 1 "10k" V 2907 1701 40  0000 C CNN
-F 2 "Discret:R1" V 2830 1700 30  0001 C CNN
+F 2 "Resistors_ThroughHole:Resistor_Horizontal_RM7mm" V 2830 1700 30  0001 C CNN
 F 3 "" H 2900 1700 30  0000 C CNN
 	1    2900 1700
@@
 F 0 "R3" V 3180 1700 40  0000 C CNN
 F 1 "10k" V 3107 1701 40  0000 C CNN
-F 2 "Discret:R1" V 3030 1700 30  0001 C CNN
+F 2 "Resistors_ThroughHole:Resistor_Horizontal_RM7mm" V 3030 1700 30  0001 C CNN
 F 3 "" H 3100 1700 30  0000 C CNN
 	1    3100 1700
@@
 F 0 "C7" H 2400 1650 40  0000 L CNN
 F 1 "100nF" H 2406 1465 40  0000 L CNN
-F 2 "Capacitors_ThroughHole:C_Rect_L4_W2.5_P2.5" H 2438 1400 30  0001 C CNN
+F 2 "Capacitors_ThroughHole:C_Disc_D3_P2.5" H 2438 1400 30  0001 C CNN
 F 3 "" H 2400 1550 60  0000 C CNN
 	1    2400 1550
@@
 F 0 "C6" H 1450 1650 40  0000 L CNN
 F 1 "10µF" H 1456 1465 40  0000 L CNN
-F 2 "Capacitors_ThroughHole:C_Radial_D6.3_L11.2_P2.5" H 1488 1400 30  0001 C CNN
+F 2 "Capacitors_ThroughHole:C_Radial_D5_L6_P2.5" H 1488 1400 30  0001 C CNN
 F 3 "" H 1450 1550 60  0000 C CNN
 	1    1450 1550
@@
 F 0 "C9" H 5750 7150 40  0000 L CNN
 F 1 "100nF" H 5756 6965 40  0000 L CNN
-F 2 "Capacitors_ThroughHole:C_Rect_L4_W2.5_P2.5" H 5788 6900 30  0001 C CNN
+F 2 "Capacitors_ThroughHole:C_Disc_D3_P2.5" H 5788 6900 30  0001 C CNN
 F 3 "" H 5750 7050 60  0000 C CNN
 	1    5750 7050
@@
 F 0 "C10" H 6050 7150 40  0000 L CNN
 F 1 "100nF" H 6056 6965 40  0000 L CNN
-F 2 "Capacitors_ThroughHole:C_Rect_L4_W2.5_P2.5" H 6088 6900 30  0001 C CNN
+F 2 "Capacitors_ThroughHole:C_Disc_D3_P2.5" H 6088 6900 30  0001 C CNN
 F 3 "" H 6050 7050 60  0000 C CNN
 	1    6050 7050
@@
 F 0 "R5" V 4380 1700 40  0000 C CNN
 F 1 "47k" V 4307 1701 40  0000 C CNN
-F 2 "Discret:R1" V 4230 1700 30  0001 C CNN
+F 2 "Resistors_ThroughHole:Resistor_Horizontal_RM7mm" V 4230 1700 30  0001 C CNN
 F 3 "" H 4300 1700 30  0000 C CNN
 	1    4300 1700
@@
 F 0 "R4" V 4180 1700 40  0000 C CNN
 F 1 "47k" V 4107 1701 40  0000 C CNN
-F 2 "Discret:R1" V 4030 1700 30  0001 C CNN
+F 2 "Resistors_ThroughHole:Resistor_Horizontal_RM7mm" V 4030 1700 30  0001 C CNN
 F 3 "" H 4100 1700 30  0000 C CNN
 	1    4100 1700
@@
 F 0 "C8" H 5050 1750 40  0000 L CNN
 F 1 "100nF" H 5056 1565 40  0000 L CNN
-F 2 "Capacitors_ThroughHole:C_Rect_L4_W2.5_P2.5" H 5088 1500 30  0001 C CNN
+F 2 "Capacitors_ThroughHole:C_Radial_D8_L11.5_P3.5" H 5088 1500 30  0001 C CNN
 F 3 "" H 5050 1650 60  0000 C CNN
 	1    5050 1650

Commit message: C8 fix footprint
Parts:
- C8: footprint Capacitors_ThroughHole:C_Radial_D8_L11.5_P3.5 -> Capacitors_ThroughHole:C_Disc_D3_P2.5
Changed lines of the file:
@@
 F 0 "C8" H 5050 1750 40  0000 L CNN
 F 1 "100nF" H 5056 1565 40  0000 L CNN
-F 2 "Capacitors_ThroughHole:C_Radial_D8_L11.5_P3.5" H 5088 1500 30  0001 C CNN
+F 2 "Capacitors_ThroughHole:C_Disc_D3_P2.5" H 5088 1500 30  0001 C CNN
 F 3 "" H 5050 1650 60  0000 C CNN
 	1    5050 1650

Commit message: cleanup
Parts:
- C10, C7, C8, C9: symbol C -> io-rescue:C
- C6: symbol CP -> io-rescue:CP
- R1, R2, R3, R4, R5: symbol R -> io-rescue:R
- SDCARD1: symbol SD_Card -> io-rescue:SD_Card
- U4: symbol 74125 -> io-rescue:74125
- U5: symbol LP2950 -> io-rescue:LP2950
- U6: symbol 7407 -> io-rescue:7407
Changed lines of the file:
@@
-EESchema Schematic File Version 2
-LIBS:io-rescue
-LIBS:power
-LIBS:device
-LIBS:transistors
-LIBS:conn
-LIBS:linear
-LIBS:regul
-LIBS:74xx
-LIBS:cmos4000
-LIBS:adc-dac
-LIBS:memory
-LIBS:xilinx
-LIBS:microcontrollers
-LIBS:dsp
-LIBS:microchip
-LIBS:analog_switches
-LIBS:motorola
-LIBS:texas
-LIBS:intel
-LIBS:audio
-LIBS:interface
-LIBS:digital-audio
-LIBS:philips
-LIBS:display
-LIBS:cypress
-LIBS:siliconi
-LIBS:opto
-LIBS:atmel
-LIBS:contrib
-LIBS:valves
-LIBS:65xxx
-LIBS:ttl_ieee
-LIBS:mini_din
-LIBS:dallas-rtc
-LIBS:lp2950l
-LIBS:osc
-LIBS:io-cache
-EELAYER 25 0
+EESchema Schematic File Version 4
+EELAYER 30 0
 EELAYER END
 $Descr A4 11693 8268
@@
 $EndDescr
 $Comp
-L 7407 U6
+L io-rescue:7407 U6
 U 4 1 542928D0
 P 1900 3600
@@
 $EndComp
 $Comp
-L 7407 U6
+L io-rescue:7407 U6
 U 6 1 542928D7
 P 1900 2200
@@
 $EndComp
 $Comp
-L 7407 U6
+L io-rescue:7407 U6
 U 5 1 542928DE
 P 1900 2900
@@
 $EndComp
 $Comp
-L R R1
+L io-rescue:R R1
 U 1 1 542928E5
 P 2700 1700
@@
 $EndComp
 $Comp
-L 74125 U4
+L io-rescue:74125 U4
 U 3 1 54292908
 P 1850 4400
@@
 $EndComp
 $Comp
-L LP2950 U5
+L io-rescue:LP2950 U5
 U 1 1 54292916
 P 1900 1400
@@
 SPI_CLK
 $Comp
-L GND #PWR017
+L io-rescue:GND #PWR017
 U 1 1 54292A1E
 P 1450 1900
@@
 $EndComp
 $Comp
-L VCC #PWR018
+L io-rescue:VCC #PWR018
 U 1 1 54292A61
 P 1450 1200
@@
 SPI_SS1
 $Comp
-L R R2
+L io-rescue:R R2
 U 1 1 542931DC
 P 2900 1700
@@
 $EndComp
 $Comp
-L R R3
+L io-rescue:R R3
 U 1 1 54293212
 P 3100 1700
@@
 $EndComp
 $Comp
-L GND #PWR019
+L io-rescue:GND #PWR019
 U 1 1 54293655
 P 5050 3250
@@
 $EndComp
 $Comp
-L C C7
+L io-rescue:C C7
 U 1 1 542937DA
 P 2400 1550
@@
 $EndComp
 $Comp
-L CP C6
+L io-rescue:CP C6
 U 1 1 542939AF
 P 1450 1550
@@
 $EndComp
 $Comp
-L C C9
+L io-rescue:C C9
 U 1 1 5429B6F0
 P 5750 7050
@@
 $EndComp
 $Comp
-L C C10
+L io-rescue:C C10
 U 1 1 5429B734
 P 6050 7050
@@
 $EndComp
 $Comp
-L VCC #PWR020
+L io-rescue:VCC #PWR020
 U 1 1 5429B75D
 P 5500 6800
@@
 $EndComp
 $Comp
-L GND #PWR021
+L io-rescue:GND #PWR021
 U 1 1 5429B775
 P 5500 7400
@@
 $EndComp
 $Comp
-L R R5
+L io-rescue:R R5
 U 1 1 54B01F31
 P 4300 1700
@@
 $EndComp
 $Comp
-L R R4
+L io-rescue:R R4
 U 1 1 54B02039
 P 4100 1700
@@
 	4300 2100 4300 1850
 $Comp
-L C C8
+L io-rescue:C C8
 U 1 1 54B2DE3A
 P 5050 1650
@@
 Connection ~ 5050 2400
 $Comp
-L SD_Card SDCARD1
+L io-rescue:SD_Card SDCARD1
 U 1 1 54C3AF89
 P 6200 2500
